File: old.kicad_sch (KiCad schematic)
At the start: 114 parts, among them CON1 I2S, CON2 Display, CON3 OUT, CON4 IN, Q1 BC850, Q2 BC850

Commit message: HW Version 1.8
Parts:
- removed C18, C19, C20, C21, C22: 1u, Capacitor_THT:Medved_CP_Radial_D5.0mm_P2.50mm, symbol Device:C_Polarized_Small
- removed JP3: GP18 Jumper, LIBS:Medved_PinHeader_1x02_P2.54mm_Vertical_R, symbol Jumper:Jumper_2_Small_Bridged
- removed JP4: GP19 Jumper, LIBS:Medved_PinHeader_1x02_P2.54mm_Vertical_R, symbol Jumper:Jumper_2_Small_Bridged
- removed JP6: RS232 Jumpers, LIBS:Medved_PinHeader_2x04_P2.54mm_Vertical, symbol Connector_Generic:Conn_02x04_Odd_Even
- removed JP7: RP ZERO +5V Jumper, LIBS:Medved_PinHeader_1x02_P2.54mm_Vertical_R, symbol Jumper:Jumper_2_Bridged
- removed L4, L5: LED, LED_SMD:LED_0805_2012Metric_Pad1.15x1.40mm_HandSolder, symbol Device:LED
- added C12, C13, C14, C15, C17: 1u, Capacitor_THT:CP_Radial_D5.0mm_P2.50mm, symbol Device:C_Polarized_Small
- added JP3: JRX, Connector_PinHeader_2.54mm:PinHeader_1x02_P2.54mm_Vertical, symbol Jumper:SolderJumper_2_Open
- added JP4: JTX, Connector_PinHeader_2.54mm:PinHeader_1x02_P2.54mm_Vertical, symbol Jumper:SolderJumper_2_Open
- added JP5: JCTS, Connector_PinHeader_2.54mm:PinHeader_1x02_P2.54mm_Vertical, symbol Jumper:SolderJumper_2_Open
- added JP6: JRTS, Connector_PinHeader_2.54mm:PinHeader_1x02_P2.54mm_Vertical, symbol Jumper:SolderJumper_2_Open
- added L2, L3: LED, LIBS:R_0805_PLUS, symbol Device:LED
- AIN1: renamed from CON4; footprint LIBS:Medved_Pins_1x03_P2.54mm_Vertical_GM -> Connector_PinHeader_2.54mm:PinHeader_1x03_P2.54mm_Vertical
- AOUT1: renamed from CON3; footprint LIBS:Medved_Pins_1x03_P2.54mm_Vertical_GM -> Connector_PinHeader_2.54mm:PinHeader_1x03_P2.54mm_Vertical
- C3: footprint LIBS:Medved_CP_Radial_D5.0mm_P2.50mm -> LIBS:R_0805_PLUS
- C6, C7, C9: footprint LIBS:Medved_CP_Radial_D5.0mm_P2.50mm -> Capacitor_THT:CP_Radial_D5.0mm_P2.50mm
- CON1: renamed from JP5; value Main Jumpers -> JMP; footprint LIBS:Medved_PinHeader_2x07_P2.54mm_Vertical -> Connector_PinHeader_2.54mm:PinHeader_2x07_P2.54mm_Vertical
- I2S1: renamed from CON1; footprint LIBS:Medved_PinHeader_1x02_P2.54mm_Vertical_NoLB -> Connector_PinHeader_2.54mm:PinHeader_1x02_P2.54mm_Vertical
- J1: renamed from PWR2; value 3V3 -> Conn_01x02; footprint LIBS:Medved_PinHeader_1x02_P2.54mm_Vertical -> Connector_PinHeader_2.54mm:PinHeader_1x02_P2.54mm_Vertical
- JOY1: renamed from DB93; value Joystick -> JOY-1
- JOY2: renamed from DB92; value Joystick -> JOY-2
- L1: footprint LED_SMD:LED_0805_2012Metric_Pad1.15x1.40mm_HandSolder -> LIBS:R_0805_PLUS
- MICROSD1: renamed from SD1; footprint LIBS:Medved_SD_Card -> LIBS:GCT-MEM2055-00-190-01-A
- PWR1: value 5V -> PWR; footprint LIBS:Medved_Pins_1x03_P2.54mm_Vertical -> Connector_PinHeader_2.54mm:PinHeader_1x03_P2.54mm_Vertical
- UART1: footprint LIBS:Medved_Pins_1x03_P2.54mm_Vertical -> Connector_PinHeader_2.54mm:PinHeader_1x03_P2.54mm_Vertical
- VIDEO1: renamed from SC1; value VIDEO (Soft Composite) -> VIDEO
- renumbered AU2 to A_IN1, AU1 to A_OUT1, CON2 to DISP1, KB1 to MINI_DIN_1, PSR1 to PSRAM1, RP2 to RP2040Z1, DB91 to RS232_1, TDA1 to TDA1387T1
Connections:
- net +5V: now also RP2040Z1.23 (5V), C12.2, C14.1
- net C1+: now also C13.1
- net C1-: now also C13.2
- net C2+: now also C15.1
- net C2-: now also C15.2
- net CTS_IN: now also RS232_1.8; no longer RS232_1.7
- net GND: now also R56.2, R57.1, C14.2, C17.1
- net GP_16: now also JP4.2 (B)
- net GP_17: now also JP3.2 (B)
- net GP_18: now also PSRAM1.1 (~{CE}), JP5.2 (B)
- net GP_19: now also PSRAM1.6 (SCLK), JP6.2 (B)
- net RTS_IN: now also RS232_1.7; no longer RS232_1.8
- net RX_IN: now also RS232_1.2; no longer RS232_1.3
- net TX_IN: now also RS232_1.3; no longer RS232_1.2
- net V+: now also C12.1
- net V-: now also C17.2
- net at R57.2: now also L3.1 (K)
- net CTS_OUT: no longer names the net of MAX1.10 (T2IN)
- net CTS_OUT: now also JP5.1 (A)
- net RTS_OUT: no longer names the net of MAX1.9 (R2OUT)
- net RTS_OUT: now also JP6.1 (A)
- net RX_OUT: no longer names the net of R56.1
- net RX_OUT: now also L2.1 (K); no longer MAX1.12 (R1OUT)
- net TX_OUT: no longer names the net of MAX1.11 (T1IN)
- net TX_OUT: now also JP4.1 (A), L2.2 (A); no longer R57.1
- new net: JP3.1 (A), L3.2 (A), MAX1.12 (R1OUT)
Other:
- note added: "CTS_OUT"
- note added: "RTS_OUT"
- note added: "RX_OUT"
- note added: "TX_OUT"
- moved on the sheet: C2, C3, J1, L1, PSRAM1, R49, RS232_1, TDA1387T1
