File: _autosave-CMZJ2.kicad_sch (KiCad schematic)
At the start: 114 parts, among them CON1 I2S, CON2 Display, CON3 OUT, CON4 IN, Q1 BC850, Q2 BC850

Commit message: HW Revision 1.8
Other:
- moved on the sheet: JP2
Changed lines of the file:
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@@
 	(wire
 		(pts
-			(xy 71.12 96.52) (xy 83.82 96.52)
+			(xy 71.12 96.52) (xy 101.6 96.52)
 		)
 		(stroke
@@
 	(wire
 		(pts
+			(xy 82.55 99.06) (xy 71.12 99.06)
+		)
+		(stroke
+			(width 0)
+			(type default)
+		)
+	)
+	(wire
+		(pts
 			(xy 118.11 67.31) (xy 130.81 67.31)
 		)
@@
 	(wire
 		(pts
-			(xy 88.9 86.36) (xy 99.06 86.36)
+			(xy 88.9 86.36) (xy 101.6 86.36)
 		)
 		(stroke
@@
 	(wire
 		(pts
+			(xy 82.55 102.87) (xy 82.55 99.06)
+		)
+		(stroke
+			(width 0)
+			(type default)
+		)
+	)
+	(wire
+		(pts
 			(xy 189.23 156.21) (xy 189.23 151.13)
 		)
@@
 	(wire
 		(pts
-			(xy 91.44 99.06) (xy 101.6 99.06)
+			(xy 91.44 102.87) (xy 93.98 102.87)
 		)
 		(stroke
@@
 	(wire
 		(pts
+			(xy 93.98 102.87) (xy 93.98 99.06)
+		)
+		(stroke
+			(width 0)
+			(type default)
+		)
+	)
+	(wire
+		(pts
 			(xy 332.74 165.1) (xy 340.36 165.1)
 		)
@@
 	(wire
 		(pts
-			(xy 71.12 99.06) (xy 83.82 99.06)
+			(xy 82.55 102.87) (xy 83.82 102.87)
 		)
 		(stroke
@@
 	(wire
 		(pts
+			(xy 93.98 99.06) (xy 101.6 99.06)
+		)
+		(stroke
+			(width 0)
+			(type default)
+		)
+	)
+	(wire
+		(pts
 			(xy 270.51 21.59) (xy 280.67 21.59)
 		)
@@
 	(wire
 		(pts
-			(xy 88.9 88.9) (xy 99.06 88.9)
+			(xy 88.9 88.9) (xy 101.6 88.9)
 		)
 		(stroke
@@
 	)
 	(label "GP_18"
-		(at 99.06 86.36 0)
+		(at 101.6 86.36 0)
 		(fields_autoplaced yes)
 		(effects
@@
 	)
 	(label "GP_21"
-		(at 95.25 99.06 0)
+		(at 101.6 99.06 0)
 		(fields_autoplaced yes)
 		(effects
@@
 	)
 	(label "GP_20"
-		(at 77.47 96.52 0)
+		(at 101.6 96.52 0)
 		(fields_autoplaced yes)
 		(effects
@@
 	)
 	(label "GP_19"
-		(at 99.06 88.9 0)
+		(at 101.6 88.9 0)
 		(fields_autoplaced yes)
 		(effects
@@
 	(symbol
 		(lib_id "Jumper:SolderJumper_2_Open")
-		(at 87.63 99.06 0)
+		(at 87.63 102.87 0)
 		(unit 1)
 		(exclude_from_sim no)
@@
 		(dnp no)
 		(property "Reference" "JP2"
-			(at 83.82 97.79 0)
+			(at 87.63 105.41 0)
 			(effects
 				(font
@@
 		)
 		(property "Value" "JMP PSRAM"
-			(at 88.138 101.6 0)
+			(at 88.138 105.41 0)
 			(effects
 				(font
@@
 		)
 		(property "Footprint" "Jumper:SolderJumper-2_P1.3mm_Open_RoundedPad1.0x1.5mm"
-			(at 87.63 99.06 0)
+			(at 87.63 102.87 0)
 			(effects
 				(font
@@
 		)
 		(property "Datasheet" "~"
-			(at 87.63 99.06 0)
+			(at 87.63 102.87 0)
 			(effects
 				(font
@@
 		)
 		(property "Description" ""
-			(at 87.63 99.06 0)
+			(at 87.63 102.87 0)
 			(effects
 				(font
