File: minifrank.kicad_pcb (KiCad board)
At the start: 2 copper layers, 66.5 x 48.3 mm, 94 parts, among them Q1 BC850, Q2 BC850, SW1 Flash Button, SW2 Reset Button, U1 NCP1117-3.3_SOT223, Y1 12 MHz

Commit message: Minor updates
Other:
- board text added: "HW REV 2.0"
- board text removed: "HW REV 1.0"
Changed lines of the file:
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@@
 		)
 	)
-	(gr_text "HW REV 1.0"
+	(gr_text "HW REV 2.0"
 		(at 149.7 94.9 90)
 		(layer "B.SilkS")
@@
 			(justify left bottom mirror)
 		)
-		(render_cache "HW REV 1.0" 90
+		(render_cache "HW REV 2.0" 90
 			(polygon
 				(pts
@@
 			(polygon
 				(pts
-					(xy 149.53 99.849825) (xy 148.871765 99.849825) (xy 148.894642 99.805054) (xy 148.895212 99.803175)
-					(xy 148.902812 99.754122) (xy 148.904738 99.705478) (xy 148.748667 99.705478) (xy 148.743734 99.758376)
-					(xy 148.729629 99.807561) (xy 148.711053 99.836636) (xy 148.668224 99.866349) (xy 148.622347 99.883393)
-					(xy 148.576475 99.894521) (xy 148.576475 100.050348) (xy 149.53 100.050348)
+					(xy 149.342421 100.29972) (xy 149.53 100.29972) (xy 149.53 99.703279) (xy 149.480959 99.705269)
+					(xy 149.426439 99.710489) (xy 149.376642 99.718801) (xy 149.324515 99.732405) (xy 149.278816 99.750217)
+					(xy 149.272812 99.753105) (xy 149.228173 99.777949) (xy 149.188411 99.807052) (xy 149.164612 99.82882)
+					(xy 149.128849 99.86859) (xy 149.097147 99.908028) (xy 149.065475 99.949799) (xy 149.035408 99.990997)
+					(xy 149.002703 100.032058) (xy 148.967882 100.066714) (xy 148.942351 100.085764) (xy 148.89779 100.106275)
+					(xy 148.848828 100.114228) (xy 148.841967 100.11434) (xy 148.792328 100.105762) (xy 148.762588 100.087229)
+					(xy 148.736312 100.044288) (xy 148.732791 100.015666) (xy 148.747096 99.968653) (xy 148.766008 99.949232)
+					(xy 148.811365 99.927774) (xy 148.859631 99.919179) (xy 148.868101 99.918457) (xy 148.868101 99.720132)
+					(xy 148.814924 99.726523) (xy 148.766094 99.738431) (xy 148.715612 99.758795) (xy 148.670808 99.786364)
+					(xy 148.660495 99.794382) (xy 148.621666 99.833139) (xy 148.592374 99.877389) (xy 148.572619 99.927132)
+					(xy 148.562401 99.982369) (xy 148.560844 100.016399) (xy 148.563703 100.065391) (xy 148.574267 100.117666)
+					(xy 148.592615 100.164681) (xy 148.618746 100.206437) (xy 148.642177 100.233042) (xy 148.68237 100.265526)
+					(xy 148.727967 100.288729) (xy 148.778968 100.302651) (xy 148.828027 100.307219) (xy 148.835373 100.307292)
+					(xy 148.885076 100.304101) (xy 148.936321 100.292885) (xy 148.982621 100.273593) (xy 149.010739 100.256245)
+					(xy 149.052947 100.220559) (xy 149.088286 100.182972) (xy 149.120326 100.143909) (xy 149.15398 100.098525)
+					(xy 149.177313 100.064759) (xy 149.208609 100.020744) (xy 149.24156 99.979121) (xy 149.270858 99.948988)
+					(xy 149.312583 99.92259) (xy 149.342421 99.914549)
 				)
 			)
 			(polygon
 				(pts
-					(xy 149.311158 100.436985) (xy 149.53 100.436985) (xy 149.53 100.215212) (xy 149.311158 100.215212)
+					(xy 149.311158 100.648011) (xy 149.53 100.648011) (xy 149.53 100.426238) (xy 149.311158 100.426238)
 				)
 			)
 			(polygon
 				(pts
-					(xy 149.06463 100.556237) (xy 149.115291 100.557708) (xy 149.174689 100.562305) (xy 149.229722 100.569968)
-					(xy 149.280391 100.580695) (xy 149.335431 100.597614) (xy 149.384187 100.618946) (xy 149.422025 100.640771)
-					(xy 149.462229 100.671563) (xy 149.500067 100.71366) (xy 149.526554 100.761373) (xy 149.54169 100.814702)
-					(xy 149.545631 100.863433) (xy 149.545087 100.88109) (xy 149.53693 100.931256) (xy 149.518984 100.977215)
-					(xy 149.491249 101.018966) (xy 149.453725 101.05651) (xy 149.406413 101.089846) (xy 149.373715 101.107535)
-					(xy 149.328463 101.126329) (xy 149.278345 101.141438) (xy 149.223362 101.152861) (xy 149.163513 101.1606)
-					(xy 149.112131 101.164138) (xy 149.057634 101.165317) (xy 149.037523 101.165182) (xy 148.979678 101.163157)
-					(xy 148.925565 101.158702) (xy 148.875182 101.151817) (xy 148.813808 101.138857) (xy 148.759067 101.121577)
-					(xy 148.710959 101.099976) (xy 148.660151 101.066901) (xy 148.619706 101.027076) (xy 148.602749 101.004181)
-					(xy 148.579468 100.960297) (xy 148.5655 100.912974) (xy 148.560844 100.862212) (xy 148.560932 100.859281)
-					(xy 148.732791 100.859281) (xy 148.733993 100.872058) (xy 148.762844 100.914922) (xy 148.809727 100.938415)
-					(xy 148.841833 100.94738) (xy 148.894765 100.956447) (xy 148.950572 100.961677) (xy 149.005458 100.96415)
-					(xy 149.056168 100.964794) (xy 149.075703 100.964693) (xy 149.130586 100.963187) (xy 149.195081 100.958367)
-					(xy 149.249655 100.950334) (xy 149.303917 100.935773) (xy 149.353839 100.906954) (xy 149.373684 100.861967)
-					(xy 149.372482 100.849355) (xy 149.343631 100.806765) (xy 149.296748 100.783077) (xy 149.264737 100.774029)
-					(xy 149.212224 100.764878) (xy 149.15706 100.7596) (xy 149.102929 100.757104) (xy 149.052993 100.756454)
-					(xy 149.033293 100.756555) (xy 148.977946 100.758061) (xy 148.912905 100.762881) (xy 148.85787 100.770914)
-					(xy 148.803148 100.785475) (xy 148.752803 100.814294) (xy 148.732791 100.859281) (xy 148.560932 100.859281)
-					(xy 148.56138 100.844284) (xy 148.569423 100.79335) (xy 148.587117 100.746693) (xy 148.614463 100.704312)
-					(xy 148.65146 100.666208) (xy 148.698108 100.632379) (xy 148.739516 100.610426) (xy 148.786041 100.592194)
-					(xy 148.837681 100.577682) (xy 148.894438 100.566892) (xy 148.943527 100.560938) (xy 148.99589 100.557366)
-					(xy 149.051528 100.556175)
+					(xy 149.06463 100.767262) (xy 149.115291 100.768734) (xy 149.174689 100.773331) (xy 149.229722 100.780994)
+					(xy 149.280391 100.791721) (xy 149.335431 100.808639) (xy 149.384187 100.829972) (xy 149.422025 100.851797)
+					(xy 149.462229 100.882589) (xy 149.500067 100.924686) (xy 149.526554 100.972399) (xy 149.54169 101.025728)
+					(xy 149.545631 101.074459) (xy 149.545087 101.092116) (xy 149.53693 101.142282) (xy 149.518984 101.188241)
+					(xy 149.491249 101.229992) (xy 149.453725 101.267536) (xy 149.406413 101.300872) (xy 149.373715 101.31856)
+					(xy 149.328463 101.337354) (xy 149.278345 101.352463) (xy 149.223362 101.363887) (xy 149.163513 101.371626)
+					(xy 149.112131 101.375164) (xy 149.057634 101.376343) (xy 149.037523 101.376208) (xy 148.979678 101.374183)
+					(xy 148.925565 101.369728) (xy 148.875182 101.362843) (xy 148.813808 101.349883) (xy 148.759067 101.332602)
+					(xy 148.710959 101.311002) (xy 148.660151 101.277927) (xy 148.619706 101.238101) (xy 148.602749 101.215207)
+					(xy 148.579468 101.171323) (xy 148.5655 101.124) (xy 148.560844 101.073237) (xy 148.560932 101.070307)
+					(xy 148.732791 101.070307) (xy 148.733993 101.083084) (xy 148.762844 101.125948) (xy 148.809727 101.149441)
+					(xy 148.841833 101.158406) (xy 148.894765 101.167473) (xy 148.950572 101.172702) (xy 149.005458 101.175175)
+					(xy 149.056168 101.175819) (xy 149.075703 101.175719) (xy 149.130586 101.174213) (xy 149.195081 101.169393)
+					(xy 149.249655 101.16136) (xy 149.303917 101.146799) (xy 149.353839 101.11798) (xy 149.373684 101.072993)
+					(xy 149.372482 101.06038) (xy 149.343631 101.017791) (xy 149.296748 100.994103) (xy 149.264737 100.985055)
+					(xy 149.212224 100.975904) (xy 149.15706 100.970626) (xy 149.102929 100.96813) (xy 149.052993 100.96748)
+					(xy 149.033293 100.967581) (xy 148.977946 100.969087) (xy 148.912905 100.973907) (xy 148.85787 100.98194)
+					(xy 148.803148 100.996501) (xy 148.752803 101.02532) (xy 148.732791 101.070307) (xy 148.560932 101.070307)
+					(xy 148.56138 101.055309) (xy 148.569423 101.004376) (xy 148.587117 100.957719) (xy 148.614463 100.915338)
+					(xy 148.65146 100.877234) (xy 148.698108 100.843405) (xy 148.739516 100.821452) (xy 148.786041 100.803219)
+					(xy 148.837681 100.788708) (xy 148.894438 100.777917) (xy 148.943527 100.771964) (xy 148.99589 100.768392)
+					(xy 149.051528 100.767201)
 				)
 			)
@@
 	)
 	(gr_text "HDMI"
-		(at 208.4 62.5 90)
+		(at 208.1 62.9 90)
 		(layer "F.SilkS")
 		(effects

Commit message: Minor updates
Parts:
- C24, C26, C27: value 10u -> 10u (tantal)
- D5: value 4148 -> 1N4148
- FL1: value W25Q128JVS -> W25Q128JVSIQ
- JP2: value I2S -> TAPE IN
Routing:
- net VBUS: track 153.8 -> 151.5 mm
- net Net-(C24-Pad1): track 52.4 -> 50.1 mm
- net +3V3: track 260.0 -> 258.0 mm
- net GND: track 10.9 -> 9.74 mm
- net /LOAD_IN_D: track 108.6 -> 107.4 mm
- net Net-(D5-K): track 33.4 -> 32.8 mm
- net /Audio Out/L: track 42.8 -> 42.2 mm
- net Net-(L1-A): track 7.90 -> 7.33 mm
- net /AUDIO_B: track 122.1 -> 121.6 mm
- net /Audio Out/R: track 32.9 -> 32.4 mm
Other:
- board text added: "Gamepad 1"
- board text added: "Gamepad 2"

Commit message: Minor updates
Parts:
- removed JOY1, JOY2: Joystick, LIBS:DSUB-9
- added GP1: Gamepad, FRANK:D-SUB (9 pin, male), F.Cu at (163.2, 99.9)
- added GP2: Gamepad, FRANK:D-SUB (9 pin, male), F.Cu at (198.2, 99.9)
- AJ1, AJ2: footprint LIBS:Jack_3.5mm -> FRANK:Jack (3.5mm)
- C1, C10, C11, C12, C13, C14, C15, C16, C17, C18, C19, C2, C20, C21, C22, C23, C25, C28, C3, C4, C5, C6, C7, C8, C9: footprint LIBS:C_0805 -> FRANK:Capacitor (0805)
- C24, C26, C27: value 10u (tantal) -> 10u*; footprint LIBS:CT_3528 -> FRANK:Capacitor (3528, tantalum, polar)
- D1, D2, D3, D4, D5: footprint LIBS:D_0805 -> FRANK:Diode (0805)
- FL1, TDA1: footprint LIBS:SO_4x4 -> FRANK:SOIC-8
- H1, H2, H3, H4: footprint LIBS:MountingHole_2.7 -> FRANK:Mounting Hole (2.7mm)
- HDMI1: value HDMI -> HDMI Female; footprint LIBS:HDMI -> FRANK:HDMI (female)
- JP1: footprint LIBS:Jumper_S -> FRANK:Jumper (solder)
- JP2: value TAPE IN -> Tape In Jumper; footprint LIBS:PinHeader_1x02 -> FRANK:Pin Header (1x02)
- JP3: value I2S -> I2S Jumper; footprint LIBS:PinHeader_1x02 -> FRANK:Pin Header (1x02)
- JP4: footprint LIBS:PinHeader_2x03 -> FRANK:Pin Header (2x03)
- KB1: value PS/2 -> PS/2 Keyboard; footprint LIBS:Connector_Mini-DIN_Female_6Pin_2rows -> FRANK:MiniDIN (6 Pin, female)
- L1: value LED -> BLUE; footprint LIBS:L_0805 -> FRANK:LED (0805)
- L2: footprint LIBS:L_0805 -> FRANK:LED (0805)
- PSR1: value PSRAM -> ESP-PSRAM32; footprint LIBS:SO_4x4 -> FRANK:SOIC-8
- Q1, Q2: footprint LIBS:Q_SOT-23 -> FRANK:SOT-23
- R1, R10, R11, R12, R13, R14, R15, R16, R17, R18, R19, R2, R20, R21, R22, R23, R24, R25, R26, R27, R28, R29, R3, R30, R31, R32, R33, R4, R5, R6, R7, R8, R9: footprint LIBS:R_0805 -> FRANK:Resistor (0805)
- RP1: footprint LIBS:RP2040-QFN-56 -> FRANK:QFN 56
- SD1: footprint LIBS:microsd -> FRANK:MicroSD (SMD, short)
- SW1, SW2: footprint LIBS:Button_SMD_3x3x2 -> FRANK:Button (SMD, 3x3mm)
- U1: value NCP1117-3.3_SOT223 -> NCP1117 3.3; footprint LIBS:SOT-223 -> FRANK:SOT-223
- USB1: footprint LIBS:USB-TYPE-C-31-M-12_lib2 -> FRANK:USB Type C
- Y1: footprint LIBS:CR_3225 -> FRANK:Crystal (3225)
- moved SW2 0.62 mm to (172.3, 91.3)
- moved C2 0.19 mm to (184.4, 90.0)
- moved C9 0.15 mm to (184.4, 87.9)
- moved R4 0.15 mm to (184.4, 85.9)
- moved R11 0.11 mm to (179.7, 73.6)
Routing:
- net /RP2040/QSPI_SS: track 87.2 -> 88.5 mm
- net /Audio Out/R: track 32.4 -> 33.2 mm
- net /LOAD_IN_D: track 107.4 -> 106.8 mm
- net /PS2_DATA: track 30.2 -> 30.7 mm
- net GND: vias 115 -> 117
Other:
- board text added: "BOOT"
- board text added: "RESET"

Commit message: HW Rev 2.0
Parts:
- AJ1: value Audio IN -> Audio In
- D1, D2, D3, D4, D5: footprint FRANK:Diode (0805) -> FRANK:Diode (SOD-323)
- JP1: value JMP PSRAM -> Jumper PSRAM (2.54)
- JP2: value Tape In Jumper -> Jumper Tape In(2.54)
- JP3: value I2S Jumper -> Jumper I2S(2.54)
- JP4: value Audio Jumpers -> Jumpers Audio(2.54)
Other:
- board text added: "USB"
