File: power.kicad_sch (KiCad schematic)
At the start: 8 parts, among them U1 NCP1117-3.3_SOT223

Commit message: Initial commit
Other:
- title: FRANK -> MiniFRANK
Changed lines of the file:
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@@
 	(paper "A4")
 	(title_block
-		(title "FRANK")
-		(date "2024-12-15")
+		(title "MiniFRANK")
+		(date "2025-01-12")
 		(rev "2.0")
 		(company "Mikhail Matveev")
-		(comment 1 "https://github.com/xtremespb/frank2")
+		(comment 1 "https://github.com/xtremespb/frank")
 	)
 	(junction

Commit message: Minor updates
Other:
- moved on the sheet: C16, C17, L2, R6, R7, R8, U1

Commit message: Minor updates
Parts:
- C16, C17: footprint LIBS:C_0805 -> FRANK:Capacitor (0805)
- L2: footprint LIBS:L_0805 -> FRANK:LED (0805)
- R6, R7, R8: footprint LIBS:R_0805 -> FRANK:Resistor (0805)
- U1: value NCP1117-3.3_SOT223 -> NCP1117 3.3; footprint LIBS:SOT-223 -> FRANK:SOT-223
- USB1: footprint LIBS:USB-TYPE-C-31-M-12_lib2 -> FRANK:USB Type C; symbol Type-C:HRO-TYPE-C-31-M-12 -> FRANK:USB-C
Other:
- note added: "The LED indicates +3V power availability. Usually it's green, but you decide ;-)"
- note added: "The power source is USB-C connector. The NCP1117 transforms +5V to +3V3."
Changed lines of the file:
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@@
+		)
+	)
+	(text "The LED indicates +3V power availability.\nUsually it's green, but you decide ;-)"
+		(exclude_from_sim no)
+		(at 87.884 102.108 0)
+		(effects
+			(font
+				(size 1.27 1.27)
+			)
+			(justify left)
+		)
+	)
+	(text "The power source is USB-C connector.\nThe NCP1117 transforms +5V to +3V3."
+		(exclude_from_sim no)
+		(at 44.45 33.274 0)
+		(effects
+			(font
+				(size 1.27 1.27)
+			)
+			(justify left)
 		)
 	)
@@
 	)
 	(symbol
+		(lib_name "GND_3")
 		(lib_id "power:GND")
 		(at 96.52 66.04 0)
@@
 			)
 		)
-		(property "Description" ""
+		(property "Description" "Power symbol creates a global label with name \"GND\" , ground"
 			(at 96.52 66.04 0)
 			(effects
@@
 	)
 	(symbol
+		(lib_name "GND_5")
 		(lib_id "power:GND")
 		(at 63.5 69.85 90)
@@
 			)
 		)
-		(property "Description" ""
+		(property "Description" "Power symbol creates a global label with name \"GND\" , ground"
 			(at 63.5 69.85 0)
 			(effects
@@
 			)
 		)
-		(property "Footprint" "LIBS:L_0805"
+		(property "Footprint" "FRANK:LED (0805)"
 			(at 57.15 105.41 0)
 			(effects
@@
 			)
 		)
-		(property "Value" "NCP1117-3.3_SOT223"
+		(property "Value" "NCP1117 3.3"
 			(at 110.49 46.9646 0)
 			(effects
@@
 			)
 		)
-		(property "Footprint" "LIBS:SOT-223"
+		(property "Footprint" "FRANK:SOT-223"
 			(at 110.49 45.72 0)
 			(effects
@@
 			)
 		)
-		(property "Footprint" "LIBS:C_0805"
+		(property "Footprint" "FRANK:Capacitor (0805)"
 			(at 129.2352 59.69 0)
 			(effects
@@
 			)
 		)
-		(property "Datasheet" "~"
+		(property "Datasheet" "https://eu.mouser.com/datasheet/2/40/KGM_X7R-3223212.pdf"
 			(at 128.27 55.88 0)
 			(effects
@@
 	)
 	(symbol
-		(lib_id "Type-C:HRO-TYPE-C-31-M-12")
+		(lib_id "FRANK:USB-C")
 		(at 55.88 60.96 0)
 		(unit 1)
@@
 			)
 		)
-		(property "Footprint" "LIBS:USB-TYPE-C-31-M-12_lib2"
+		(property "Footprint" "FRANK:USB Type C"
 			(at 59.69 62.23 0)
 			(effects
@@
 			)
 		)
-		(property "Footprint" "LIBS:C_0805"
+		(property "Footprint" "FRANK:Capacitor (0805)"
 			(at 93.6752 59.69 0)
 			(effects
@@
 			)
 		)
-		(property "Datasheet" "~"
+		(property "Datasheet" "https://eu.mouser.com/datasheet/2/40/KGM_X7R-3223212.pdf"
 			(at 92.71 55.88 0)
 			(effects
@@
 			)
 		)
-		(property "Footprint" "LIBS:R_0805"
+		(property "Footprint" "FRANK:Resistor (0805)"
 			(at 64.77 107.188 90)
 			(effects
@@
 			)
 		)
-		(property "Footprint" "LIBS:R_0805"
+		(property "Footprint" "FRANK:Resistor (0805)"
 			(at 60.96 69.85 0)
 			(effects
@@
 	)
 	(symbol
+		(lib_name "GND_6")
 		(lib_id "power:GND")
 		(at 63.5 54.61 90)
@@
 			)
 		)
-		(property "Description" ""
+		(property "Description" "Power symbol creates a global label with name \"GND\" , ground"
 			(at 63.5 54.61 0)
 			(effects
@@
 	)
 	(symbol
+		(lib_name "GND_1")
 		(lib_id "power:GND")
 		(at 128.27 60.96 0)
@@
 			)
 		)
-		(property "Description" ""
+		(property "Description" "Power symbol creates a global label with name \"GND\" , ground"
 			(at 128.27 60.96 0)
 			(effects
@@
 			)
 		)
-		(property "Description" ""
+		(property "Description" "Power symbol creates a global label with name \"+3V3\""
 			(at 128.27 49.53 0)
 			(effects
@@
 			)
 		)
-		(property "Footprint" "LIBS:R_0805"
+		(property "Footprint" "FRANK:Resistor (0805)"
 			(at 60.96 54.61 0)
 			(effects
@@
 			)
 		)
-		(property "Description" ""
+		(property "Description" "Power symbol creates a global label with name \"GND\" , ground"
 			(at 63.5 46.99 0)
 			(effects
@@
 	)
 	(symbol
+		(lib_name "GND_7")
 		(lib_id "power:GND")
 		(at 66.04 77.47 90)
@@
 			)
 		)
-		(property "Description" ""
+		(property "Description" "Power symbol creates a global label with name \"GND\" , ground"
 			(at 66.04 77.47 0)
 			(effects
@@
 	)
 	(symbol
+		(lib_name "GND_4")
 		(lib_id "power:GND")
 		(at 110.49 59.69 0)
@@
 			)
 		)
-		(property "Description" ""
+		(property "Description" "Power symbol creates a global label with name \"GND\" , ground"
 			(at 110.49 59.69 0)
 			(effects

Commit message: HW Rev 2.0
Parts:
- C16, C17: AliExpress (none) -> https://www.aliexpress.com/item/33008008276.html
- L2: AliExpress (none) -> https://www.aliexpress.com/item/1005007252088951.html
- R6, R7, R8: AliExpress (none) -> https://www.aliexpress.com/item/1005005945735199.html
- U1: AliExpress (none) -> https://www.aliexpress.com/item/1005005802338707.html
- USB1: AliExpress (none) -> https://www.aliexpress.com/item/1005005500797563.html
Changed lines of the file:
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@@
 	(title_block
 		(title "MiniFRANK")
-		(date "2025-01-13")
+		(date "2025-01-14")
 		(rev "2.0")
 		(company "Mikhail Matveev")
@@
 			)
 		)
-		(property "Datasheet" "~"
+		(property "Datasheet" "https://www.we-online.com/components/products/datasheet/15408085BA400.pdf"
 			(at 57.15 105.41 0)
 			(effects
@@
 		)
 		(property "Description" "Light emitting diode"
+			(at 57.15 105.41 0)
+			(effects
+				(font
+					(size 1.27 1.27)
+				)
+				(hide yes)
+			)
+		)
+		(property "AliExpress" "https://www.aliexpress.com/item/1005007252088951.html"
 			(at 57.15 105.41 0)
 			(effects
@@
 			)
 		)
+		(property "AliExpress" "https://www.aliexpress.com/item/1005005802338707.html"
+			(at 110.49 50.8 0)
+			(effects
+				(font
+					(size 1.27 1.27)
+				)
+				(hide yes)
+			)
+		)
 		(pin "1"
 		)
@@
 			)
 		)
+		(property "AliExpress" "https://www.aliexpress.com/item/33008008276.html"
+			(at 128.27 55.88 0)
+			(effects
+				(font
+					(size 1.27 1.27)
+				)
+				(hide yes)
+			)
+		)
 		(pin "1"
 		)
@@
 			)
 		)
-		(property "Datasheet" ""
+		(property "Datasheet" "https://eu.mouser.com/datasheet/2/837/usb4215-3472997.pdf"
 			(at 59.69 62.23 0)
 			(effects
@@
 		)
 		(property "LCSC" "C165948"
+			(at 55.88 60.96 0)
+			(effects
+				(font
+					(size 1.27 1.27)
+				)
+				(hide yes)
+			)
+		)
+		(property "AliExpress" "https://www.aliexpress.com/item/1005005500797563.html"
 			(at 55.88 60.96 0)
 			(effects
@@
 		)
 		(property "Description" ""
+			(at 92.71 55.88 0)
+			(effects
+				(font
+					(size 1.27 1.27)
+				)
+				(hide yes)
+			)
+		)
+		(property "AliExpress" "https://www.aliexpress.com/item/33008008276.html"
 			(at 92.71 55.88 0)
 			(effects
@@
 			)
 		)
-		(property "Datasheet" "~"
+		(property "Datasheet" "https://www.vishay.com/docs/28952/mcs0402at-mct0603at-mcu0805at-mca1206at.pdf"
 			(at 64.77 105.41 0)
 			(effects
@@
 		)
 		(property "Description" "Resistor"
+			(at 64.77 105.41 0)
+			(effects
+				(font
+					(size 1.27 1.27)
+				)
+				(hide yes)
+			)
+		)
+		(property "AliExpress" "https://www.aliexpress.com/item/1005005945735199.html"
 			(at 64.77 105.41 0)
 			(effects
@@
 			)
 		)
-		(property "Datasheet" ""
+		(property "Datasheet" "https://www.vishay.com/docs/28952/mcs0402at-mct0603at-mcu0805at-mca1206at.pdf"
 			(at 60.96 69.85 0)
 			(effects
@@
 		)
 		(property "LCSC" " "
+			(at 60.96 69.85 0)
+			(effects
+				(font
+					(size 1.27 1.27)
+				)
+				(hide yes)
+			)
+		)
+		(property "AliExpress" "https://www.aliexpress.com/item/1005005945735199.html"
 			(at 60.96 69.85 0)
 			(effects
@@
 			)
 		)
-		(property "Datasheet" ""
+		(property "Datasheet" "https://www.vishay.com/docs/28952/mcs0402at-mct0603at-mcu0805at-mca1206at.pdf"
 			(at 60.96 54.61 0)
 			(effects
@@
 			(at 60.96 54.61 0)
 			(effects
+				(font
+					(size 1.27 1.27)
+				)
+				(hide yes)
+			)
+		)
+		(property "AliExpress" "https://www.aliexpress.com/item/1005005945735199.html"
+			(at 60.96 54.61 0)
+			(effects
