File: rp2040.kicad_sch (KiCad schematic)
At the start: 25 parts, among them SW1 Flash Button, Y1 12 MHz

Commit message: Initial commit
Other:
- title: FRANK -> MiniFRANK
Changed lines of the file:
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@@
 	(paper "A4")
 	(title_block
-		(title "FRANK")
-		(date "2024-12-15")
+		(title "MiniFRANK")
+		(date "2025-01-12")
 		(rev "2.0")
 		(company "Mikhail Matveev")
-		(comment 1 "https://github.com/xtremespb/frank2")
+		(comment 1 "https://github.com/xtremespb/frank")
 	)
 	(junction

Commit message: Minor updates
Parts:
- FL1: value W25Q128JVS -> W25Q128JVSIQ
- Y1: footprint CR_3225 -> LIBS:CR_3225
Changed lines of the file:
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@@
 	(title_block
 		(title "MiniFRANK")
-		(date "2025-01-12")
+		(date "2025-01-13")
 		(rev "2.0")
 		(company "Mikhail Matveev")
@@
 			)
 		)
-		(property "Footprint" "CR_3225"
+		(property "Footprint" "LIBS:CR_3225"
 			(at 227.33 111.76 0)
 			(effects
@@
 			)
 		)
-		(property "Value" "W25Q128JVS"
+		(property "Value" "W25Q128JVSIQ"
 			(at 264.16 75.565 0)
 			(effects

Commit message: Minor updates
Parts:
- C1, C10, C11, C12, C13, C14, C15, C2, C3, C4, C5, C6, C7, C8, C9: footprint LIBS:C_0805 -> FRANK:Capacitor (0805)
- FL1: footprint LIBS:SO_4x4 -> FRANK:SOIC-8; symbol Memory_Flash:W25Q128JVS -> FRANK:Flash_W25Q128JVS
- L1: value LED -> BLUE; footprint LIBS:L_0805 -> FRANK:LED (0805)
- R1, R2, R3, R4, R5: footprint LIBS:R_0805 -> FRANK:Resistor (0805)
- RP1: footprint LIBS:RP2040-QFN-56 -> FRANK:QFN 56; symbol MCU_RaspberryPi_RP2040:RP2040 -> FRANK:RP2040
- SW1: footprint LIBS:Button_SMD_3x3x2 -> FRANK:Button (SMD, 3x3mm)
- Y1: footprint LIBS:CR_3225 -> FRANK:Crystal (3225)
Other:
- note added: "Flash memory is required as RP2040 doesn't have it's own. You may save some money buying a cheaper flash (4MB is OK)."
- note added: "This is the 12Mhz external crystal. RP2040 has it's own, but the external crystal is more robust and is recommended."
- note added: "This is the main schematics of RP2040. Note that all 3V3 capacitors shall be kept close to the RP2040, especially pins 45 and 44."
- moved on the sheet: C1, C14, C15, FL1, L1, R1, R4, R5, SW1, Y1

Commit message: HW Rev 2.0
Parts:
- C1, C10, C11, C12, C13, C14, C15, C2, C3, C4, C5, C6, C7, C8, C9: AliExpress (none) -> https://www.aliexpress.com/item/33008008276.html
- FL1: AliExpress (none) -> https://www.aliexpress.com/item/1005007820627233.html
- L1: AliExpress (none) -> https://www.aliexpress.com/item/1005007252088951.html
- R1, R2, R3, R4, R5: AliExpress (none) -> https://www.aliexpress.com/item/1005005945735199.html
- RP1: AliExpress (none) -> https://www.aliexpress.com/item/1005007275652762.html
- SW1: AliExpress (none) -> https://www.aliexpress.com/item/1005001629293584.html
- Y1: AliExpress (none) -> https://www.aliexpress.com/item/1005004661413307.html
