File: tape.kicad_sch (KiCad schematic)
At the start: 12 parts, among them Q1 BC850, Q2 BC850

Commit message: Initial commit
Other:
- title: FRANK -> MiniFRANK
Changed lines of the file:
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@@
 	(paper "A4")
 	(title_block
-		(title "FRANK")
-		(date "2024-12-15")
+		(title "MiniFRANK")
+		(date "2025-01-12")
 		(rev "2.0")
 		(company "Mikhail Matveev")
-		(comment 1 "https://github.com/xtremespb/frank2")
+		(comment 1 "https://github.com/xtremespb/frank")
 	)
 	(junction

Commit message: Minor updates
Parts:
- D1: value 4148 -> 1N4148
- JP2: value I2S -> TAPE IN
Other:
- moved on the sheet: AJ1, C1, C2, D1, JP2, Q1, Q2, R1, R2, R3, R4, R5

Commit message: Minor updates
Parts:
- AJ1: footprint LIBS:Jack_3.5mm -> FRANK:Jack (3.5mm); symbol Connector_Audio:AudioJack3_SwitchTR -> FRANK:AudioJack_3.5mm
- C1, C2: footprint LIBS:C_0805 -> FRANK:Capacitor (0805)
- D1: footprint LIBS:D_0805 -> FRANK:Diode (0805)
- JP2: value TAPE IN -> Tape In Jumper; footprint LIBS:PinHeader_1x02 -> FRANK:Pin Header (1x02)
- Q1, Q2: footprint LIBS:Q_SOT-23 -> FRANK:SOT-23
- R1, R2, R3, R4, R5: footprint LIBS:R_0805 -> FRANK:Resistor (0805)
Other:
- note added: "This schematics is used to load data from external audio source, e.g. tape."
Changed lines of the file:
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@@
 		)
 	)
-	(label "LOAD_IN_D"
-		(at 138.43 81.28 0)
-		(fields_autoplaced yes)
+	(text "This schematics is used to load data from\nexternal audio source, e.g. tape."
+		(exclude_from_sim no)
+		(at 38.1 27.178 0)
 		(effects
 			(font
 				(size 1.27 1.27)
 			)
-			(justify left bottom)
+			(justify left)
 		)
 	)
 	(label "LOAD_IN_D"
-		(at 138.43 66.04 0)
+		(at 138.43 81.28 0)
 		(fields_autoplaced yes)
 		(effects
@@
 		)
 	)
-	(label "LOAD_IN"
-		(at 49.53 72.39 0)
+	(label "LOAD_IN_D"
+		(at 138.43 66.04 0)
 		(fields_autoplaced yes)
 		(effects
@@
 		)
 	)
+	(label "LOAD_IN"
+		(at 49.53 72.39 0)
+		(fields_autoplaced yes)
+		(effects
+			(font
+				(size 1.27 1.27)
+			)
+			(justify left bottom)
+		)
+	)
 	(hierarchical_label "LOAD_IN"
 		(shape input)
@@
 			)
 		)
-		(property "Footprint" "LIBS:D_0805"
+		(property "Footprint" "FRANK:Diode (0805)"
 			(at 93.98 64.77 0)
 			(effects
@@
 			)
 		)
-		(property "Footprint" "LIBS:R_0805"
+		(property "Footprint" "FRANK:Resistor (0805)"
 			(at 105.41 66.548 90)
 			(effects
@@
 			)
 		)
-		(property "Footprint" "LIBS:R_0805"
+		(property "Footprint" "FRANK:Resistor (0805)"
 			(at 115.062 53.34 90)
 			(effects
@@
 	)
 	(symbol
-		(lib_id "Connector_Audio:AudioJack3_SwitchTR")
+		(lib_id "FRANK:AudioJack_3.5mm")
 		(at 44.45 77.47 0)
 		(mirror x)
@@
 			)
 		)
-		(property "Footprint" "LIBS:Jack_3.5mm"
+		(property "Footprint" "FRANK:Jack (3.5mm)"
 			(at 44.45 77.47 0)
 			(effects
@@
 			)
 		)
-		(property "Datasheet" "~"
+		(property "Datasheet" "https://eu.mouser.com/datasheet/2/1628/sj1_353xng-3511142.pdf"
 			(at 44.45 77.47 0)
 			(effects
@@
 			)
 		)
-		(property "Footprint" "LIBS:C_0805"
+		(property "Footprint" "FRANK:Capacitor (0805)"
 			(at 73.66 71.4248 0)
 			(effects
@@
 			)
 		)
-		(property "Datasheet" "~"
+		(property "Datasheet" "https://eu.mouser.com/datasheet/2/447/KEM_C1075_X7R_HT_SMD-3316221.pdf"
 			(at 69.85 72.39 0)
 			(effects
@@
 			)
 		)
-		(property "Footprint" "LIBS:R_0805"
+		(property "Footprint" "FRANK:Resistor (0805)"
 			(at 81.28 74.168 90)
 			(effects
@@
 			)
 		)
-		(property "Value" "TAPE IN"
+		(property "Value" "Tape In Jumper"
 			(at 162.56 83.8199 0)
 			(effects
@@
 			)
 		)
-		(property "Footprint" "LIBS:PinHeader_1x02"
+		(property "Footprint" "FRANK:Pin Header (1x02)"
 			(at 160.02 81.28 0)
 			(effects
@@
 			)
 		)
-		(property "Footprint" "LIBS:C_0805"
+		(property "Footprint" "FRANK:Capacitor (0805)"
 			(at 133.0452 54.61 0)
 			(effects
@@
 			)
 		)
-		(property "Datasheet" "~"
+		(property "Datasheet" "https://eu.mouser.com/datasheet/2/447/KEM_C1075_X7R_HT_SMD-3316221.pdf"
 			(at 132.08 50.8 0)
 			(effects
@@
 			)
 		)
-		(property "Footprint" "LIBS:R_0805"
+		(property "Footprint" "FRANK:Resistor (0805)"
 			(at 64.262 83.82 90)
 			(effects
@@
 			)
 		)
-		(property "Footprint" "LIBS:Q_SOT-23"
+		(property "Footprint" "FRANK:SOT-23"
 			(at 101.6 74.295 0)
 			(effects
@@
 			)
 		)
-		(property "Footprint" "LIBS:R_0805"
+		(property "Footprint" "FRANK:Resistor (0805)"
 			(at 97.282 53.34 90)
 			(effects
@@
 			)
 		)
-		(property "Footprint" "LIBS:Q_SOT-23"
+		(property "Footprint" "FRANK:SOT-23"
 			(at 119.38 66.675 0)
 			(effects

Commit message: HW Rev 2.0
Parts:
- AJ1: value Audio IN -> Audio In; AliExpress (none) -> https://www.aliexpress.com/item/1005006710837751.html
- C1, C2: AliExpress (none) -> https://www.aliexpress.com/item/33008008276.html
- D1: footprint FRANK:Diode (0805) -> FRANK:Diode (SOD-323); AliExpress (none) -> https://www.aliexpress.com/item/1005005707644429.html
- JP2: value Tape In Jumper -> Jumper Tape In(2.54); AliExpress (none) -> https://www.aliexpress.com/item/1005006454399822.html
- Q1, Q2: AliExpress (none) -> https://www.aliexpress.com/item/33017911878.html
- R1, R2, R3, R4, R5: AliExpress (none) -> https://www.aliexpress.com/item/1005005945735199.html
Changed lines of the file:
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@@
 	(title_block
 		(title "MiniFRANK")
-		(date "2025-01-13")
+		(date "2025-01-14")
 		(rev "2.0")
 		(company "Mikhail Matveev")
@@
 			)
 		)
-		(property "Footprint" "FRANK:Diode (0805)"
+		(property "Footprint" "FRANK:Diode (SOD-323)"
 			(at 93.98 64.77 0)
 			(effects
@@
 			)
 		)
-		(property "Datasheet" "~"
+		(property "Datasheet" "https://www.vishay.com/docs/40002/293d.pdf"
 			(at 93.98 64.77 0)
 			(effects
@@
 		)
 		(property "Sim.Pins" "1=K 2=A"
+			(at 93.98 64.77 0)
+			(effects
+				(font
+					(size 1.27 1.27)
+				)
+				(hide yes)
+			)
+		)
+		(property "AliExpress" "https://www.aliexpress.com/item/1005005707644429.html"
 			(at 93.98 64.77 0)
 			(effects
@@
 			)
 		)
-		(property "Datasheet" "~"
+		(property "Datasheet" "https://www.vishay.com/docs/28952/mcs0402at-mct0603at-mcu0805at-mca1206at.pdf"
 			(at 105.41 64.77 0)
 			(effects
@@
 		)
 		(property "Description" ""
+			(at 105.41 64.77 0)
+			(effects
+				(font
+					(size 1.27 1.27)
+				)
+				(hide yes)
+			)
+		)
+		(property "AliExpress" "https://www.aliexpress.com/item/1005005945735199.html"
 			(at 105.41 64.77 0)
 			(effects
@@
 			)
 		)
-		(property "Datasheet" "~"
+		(property "Datasheet" "https://www.vishay.com/docs/28952/mcs0402at-mct0603at-mcu0805at-mca1206at.pdf"
 			(at 116.84 53.34 0)
 			(effects
@@
 		)
 		(property "Description" ""
+			(at 116.84 53.34 0)
+			(effects
+				(font
+					(size 1.27 1.27)
+				)
+				(hide yes)
+			)
+		)
+		(property "AliExpress" "https://www.aliexpress.com/item/1005005945735199.html"
 			(at 116.84 53.34 0)
 			(effects
@@
 			)
 		)
-		(property "Value" "Audio IN"
+		(property "Value" "Audio In"
 			(at 46.99 66.04 0)
 			(effects
@@
 		)
 		(property "Description" "Audio Jack, 3 Poles (Stereo / TRS), Switched TR Poles (Normalling)"
+			(at 44.45 77.47 0)
+			(effects
+				(font
+					(size 1.27 1.27)
+				)
+				(hide yes)
+			)
+		)
+		(property "AliExpress" "https://www.aliexpress.com/item/1005006710837751.html"
 			(at 44.45 77.47 0)
 			(effects
@@
 			)
 		)
+		(property "AliExpress" "https://www.aliexpress.com/item/33008008276.html"
+			(at 69.85 72.39 0)
+			(effects
+				(font
+					(size 1.27 1.27)
+				)
+				(hide yes)
+			)
+		)
 		(pin "1"
 		)
@@
 			)
 		)
-		(property "Datasheet" "~"
+		(property "Datasheet" "https://www.vishay.com/docs/28952/mcs0402at-mct0603at-mcu0805at-mca1206at.pdf"
 			(at 81.28 72.39 0)
 			(effects
@@
 		)
 		(property "Description" ""
+			(at 81.28 72.39 0)
+			(effects
+				(font
+					(size 1.27 1.27)
+				)
+				(hide yes)
+			)
+		)
+		(property "AliExpress" "https://www.aliexpress.com/item/1005005945735199.html"
 			(at 81.28 72.39 0)
 			(effects
@@
 			)
 		)
-		(property "Value" "Tape In Jumper"
+		(property "Value" "Jumper Tape In(2.54)"
 			(at 162.56 83.8199 0)
 			(effects
@@
 		)
 		(property "Description" "Generic connector, single row, 01x02, script generated (kicad-library-utils/schlib/autogen/connector/)"
+			(at 160.02 81.28 0)
+			(effects
+				(font
+					(size 1.27 1.27)
+				)
+				(hide yes)
+			)
+		)
+		(property "AliExpress" "https://www.aliexpress.com/item/1005006454399822.html"
 			(at 160.02 81.28 0)
 			(effects
@@
 			)
 		)
+		(property "AliExpress" "https://www.aliexpress.com/item/33008008276.html"
+			(at 132.08 50.8 0)
+			(effects
+				(font
+					(size 1.27 1.27)
+				)
+				(hide yes)
+			)
+		)
 		(pin "1"
 		)
@@
 			)
 		)
-		(property "Datasheet" "~"
+		(property "Datasheet" "https://www.vishay.com/docs/28952/mcs0402at-mct0603at-mcu0805at-mca1206at.pdf"
 			(at 66.04 83.82 0)
 			(effects
@@
 		)
 		(property "Description" ""
+			(at 66.04 83.82 0)
+			(effects
+				(font
+					(size 1.27 1.27)
+				)
+				(hide yes)
+			)
+		)
+		(property "AliExpress" "https://www.aliexpress.com/item/1005005945735199.html"
 			(at 66.04 83.82 0)
 			(effects
@@
 			)
 		)
+		(property "AliExpress" "https://www.aliexpress.com/item/33017911878.html"
+			(at 96.52 72.39 0)
+			(effects
+				(font
+					(size 1.27 1.27)
+				)
+				(hide yes)
+			)
+		)
 		(pin "1"
 		)
@@
 			)
 		)
-		(property "Datasheet" "~"
+		(property "Datasheet" "https://www.vishay.com/docs/28952/mcs0402at-mct0603at-mcu0805at-mca1206at.pdf"
 			(at 99.06 53.34 0)
 			(effects
@@
 		)
 		(property "Description" ""
+			(at 99.06 53.34 0)
+			(effects
+				(font
+					(size 1.27 1.27)
+				)
+				(hide yes)
+			)
+		)
+		(property "AliExpress" "https://www.aliexpress.com/item/1005005945735199.html"
 			(at 99.06 53.34 0)
 			(effects
@@
 			(at 114.3 64.77 0)
 			(effects
+				(font
+					(size 1.27 1.27)
+				)
+				(hide yes)
+			)
+		)
+		(property "AliExpress" "https://www.aliexpress.com/item/33017911878.html"
+			(at 114.3 64.77 0)
+			(effects
