File: hardware/frank_m2/rp2040.kicad_sch (KiCad schematic)
At the start: 25 parts, among them SW1 Flash Button, Y1 12 MHz

Commit message: Names changed
Other:
- title: Valera-2350A -> MiniFRANK
Changed lines of the file:
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@@
 	(paper "A4")
 	(title_block
-		(title "Valera-2350A")
-		(date "2025-01-30")
-		(rev "1.0")
+		(title "MiniFRANK")
+		(date "2025-01-14")
+		(rev "2.0")
 		(company "Mikhail Matveev")
 		(comment 1 "https://github.com/xtremespb/frank")
