File: hardware/frank_m2/rs232.kicad_sch (KiCad schematic)
At the start: 0 parts

Commit message: Names changed
Parts:
- added C17, C18, C19, C20: 1u, FRANK:Capacitor (0805), symbol Device:C_Small
- added COM1: D-SUB 9 Male, FRANK:D-SUB (9 pin, male, top mount), symbol FRANK:DB9_Male_Small
- added D8, D9: 1N4148, FRANK:Diode (SOD-323), symbol Diode:1N4148
- added MAX1: MAX232CSE+, FRANK:SOIC127P600X175-16N, symbol FRANK:MAX232CSE+
- added R59, R60: 1K, FRANK:Resistor (0805), symbol Device:R
Connections:
- new net: COM1.1, COM1.4, COM1.6
- new net +3V3: R59.2, R60.2
- new net C1+: C18.2, MAX1.1 (C1+)
- new net C1-: C18.1, MAX1.3 (C1-)
- new net C2+: C19.2, MAX1.4 (C2+)
- new net C2-: C19.1, MAX1.5 (C2-)
- new net CTS_IN: COM1.7, MAX1.7 (T2OUT)
- new net CTS_MAX: D8.1 (K), MAX1.9 (R2OUT)
- new net GND: C20.2, COM1.5, MAX1.15 (GND)
- new net RS232_CTS: D8.2 (A), R59.1
- new net RS232_RTS: MAX1.10 (T2IN)
- new net RS232_RX: D9.2 (A), R60.1
- new net RS232_TX: MAX1.11 (T1IN)
- new net RTS_IN: COM1.8, MAX1.8 (R2IN)
- new net RX_IN: COM1.3, MAX1.14 (T1OUT)
- new net RX_MAX: D9.1 (K), MAX1.12 (R1OUT)
- new net TX_IN: COM1.2, MAX1.13 (R1IN)
- new net V+: C17.1, MAX1.2 (V+)
- new net V-: C20.1, MAX1.6 (V-)
- new net VBUS: C17.2, MAX1.16 (VCC)
- no-connect marks 0 -> 1
Other:
- company: (none) -> Mikhail Matveev
- title: (none) -> FRANK
