File: hardware/frank_m2/HR3FQ.kicad_pcb (KiCad board)
At the start: 2 copper layers, 99 x 80.1 mm, 108 parts, among them CON1 Pin Header 1x03, CON2 Pin Header 1x03, CON3 Pin Header 1x08, J1 Pin Header 2x18, Q1 BC850, Q2 BC850, U1 NCP1117 3.3

Commit message: FRANK M1 & M2 HW Revisions
Routing:
- net VBUS: track 485.1 -> 489.5 mm
- net /GPIO9: track 67.9 -> 70.6 mm
- net /GPIO19: track 92.5 -> 94.3 mm
- net /GPIO21: track 66.6 -> 68.2 mm
- net /GPIO1: track 118.5 -> 120.0 mm
- net /GPIO20: track 64.8 -> 66.1 mm
- net Net-(C7-Pad1): track 11.0 -> 12.2 mm
- net /MS_CLK: track 26.1 -> 27.2 mm
- net /MS_DATA: track 31.9 -> 33.0 mm
- net Net-(R45-Pad2): track 38.8 -> 39.7 mm
- net /A_OUTR: track 41.1 -> 42.0 mm
- net /GPIO11: track 65.1 -> 65.7 mm
- net /GPIO14: track 64.9 -> 65.4 mm
- net GND: vias 73 -> 81

Commit message: HW Rev 1.02 (M2)
Connections:
- net /Zero/ZGPIO0 renamed /Zero/ZGPIO0_1
- net /Zero/ZGPIO10 renamed /Zero/ZGPIO10_1
- net /Zero/ZGPIO13_1 renamed /Zero/ZGPIO13
- net /Zero/ZGPIO1_1 renamed /Zero/ZGPIO1
- net /Zero/ZGPIO26 renamed /Zero/ZGPIO26_1
- net /Zero/ZGPIO27 renamed /Zero/ZGPIO27_1
- net /Zero/ZGPIO28_1 renamed /Zero/ZGPIO28
- net /Zero/ZGPIO29_1 renamed /Zero/ZGPIO29
- net /Zero/ZGPIO6_1 renamed /Zero/ZGPIO6
- net /Zero/ZGPIO7_1 renamed /Zero/ZGPIO7
- net /Zero/ZGPIO8 renamed /Zero/ZGPIO8_1
- net /Zero/ZGPIO9 renamed /Zero/ZGPIO9_1
Routing:
- net Net-(USB2-D1+): track 22.3 -> 23.0 mm
Other:
- board text added: "HW Revision 1.02 (M2)"
- board text added: "rh1.tech"
- board text removed: "HW REV 2.1"
- board text removed: "M2"
- board text removed: "RH1.DEV"
