File: hardware/frank_m2/hdmi.kicad_sch (KiCad schematic)
At the start: 10 parts

Commit message: Names changed
Parts:
- HDMI1: renamed from HDMI2; value HDMI Female -> DC3RX19JA2
- renumbered C42 to C5, R68 to R14, R69 to R15, R70 to R16, R71 to R17, R72 to R18, R73 to R19, R74 to R20, R75 to R21
Other:
- note added: "HDMI video output requires the resistors to be close to the HDMI socket in order to work properly."
- title: Frank M2 -> FRANK
Changed lines of the file:
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@@
 	(paper "A4")
 	(title_block
-		(title "Frank M2")
-		(date "2025-02-02")
-		(rev "1.02")
+		(title "FRANK")
+		(date "2025-02-18")
+		(rev "1.13")
 		(company "Mikhail Matveev")
 		(comment 1 "https://github.com/xtremespb/frank")
@@
 			(width 0)
 			(type default)
+		)
+	)
+	(text "HDMI video output requires the resistors to\nbe close to the HDMI socket in order to\nwork properly."
+		(exclude_from_sim no)
+		(at 43.18 27.432 0)
+		(effects
+			(font
+				(size 1.27 1.27)
+			)
+			(justify left)
 		)
 	)
@@
 		(on_board yes)
 		(dnp no)
-		(property "Reference" "R71"
+		(property "Reference" "R17"
 			(at 90.17 104.14 90)
 			(effects
@@
 		(instances
 			(project "frank2"
-				(path "/8c0b3d8b-46d3-4173-ab1e-a61765f77d61/1ea0e9ac-8f42-4d3d-8b47-067d751f5a51"
-					(reference "R71")
+				(path "/8c0b3d8b-46d3-4173-ab1e-a61765f77d61/db853a64-9343-4a36-b5b8-71001392b936"
+					(reference "R17")
 					(unit 1)
 				)
@@
 		(on_board yes)
 		(dnp no)
-		(property "Reference" "R73"
+		(property "Reference" "R19"
 			(at 100.33 111.76 90)
 			(effects
@@
 		(instances
 			(project "frank2"
-				(path "/8c0b3d8b-46d3-4173-ab1e-a61765f77d61/1ea0e9ac-8f42-4d3d-8b47-067d751f5a51"
-					(reference "R73")
+				(path "/8c0b3d8b-46d3-4173-ab1e-a61765f77d61/db853a64-9343-4a36-b5b8-71001392b936"
+					(reference "R19")
 					(unit 1)
 				)
@@
 		(on_board yes)
 		(dnp no)
-		(property "Reference" "R68"
+		(property "Reference" "R14"
 			(at 90.17 91.44 90)
 			(effects
@@
 		(instances
 			(project "frank2"
-				(path "/8c0b3d8b-46d3-4173-ab1e-a61765f77d61/1ea0e9ac-8f42-4d3d-8b47-067d751f5a51"
-					(reference "R68")
+				(path "/8c0b3d8b-46d3-4173-ab1e-a61765f77d61/db853a64-9343-4a36-b5b8-71001392b936"
+					(reference "R14")
 					(unit 1)
 				)
@@
 		(dnp no)
 		(fields_autoplaced yes)
-		(property "Reference" "#PWR087"
+		(property "Reference" "#PWR038"
 			(at 71.12 81.28 0)
 			(effects
@@
 		(instances
 			(project ""
-				(path "/8c0b3d8b-46d3-4173-ab1e-a61765f77d61/1ea0e9ac-8f42-4d3d-8b47-067d751f5a51"
-					(reference "#PWR087")
+				(path "/8c0b3d8b-46d3-4173-ab1e-a61765f77d61/db853a64-9343-4a36-b5b8-71001392b936"
+					(reference "#PWR038")
 					(unit 1)
 				)
@@
 		(on_board yes)
 		(dnp no)
-		(property "Reference" "R72"
+		(property "Reference" "R18"
 			(at 90.17 106.68 90)
 			(effects
@@
 		(instances
 			(project "frank2"
-				(path "/8c0b3d8b-46d3-4173-ab1e-a61765f77d61/1ea0e9ac-8f42-4d3d-8b47-067d751f5a51"
-					(reference "R72")
+				(path "/8c0b3d8b-46d3-4173-ab1e-a61765f77d61/db853a64-9343-4a36-b5b8-71001392b936"
+					(reference "R18")
 					(unit 1)
 				)
@@
 		(on_board yes)
 		(dnp no)
-		(property "Reference" "C42"
+		(property "Reference" "C5"
 			(at 76.3016 74.549 0)
 			(effects
@@
 			)
 		)
-		(property "Datasheet" "https://eu.mouser.com/datasheet/2/447/KEM_C1075_X7R_HT_SMD-3316221.pdf"
+		(property "Datasheet" "https://eu.mouser.com/datasheet/2/40/KGM_X7R-3223212.pdf"
 			(at 77.47 77.47 0)
 			(effects
@@
 		(instances
 			(project "frank2"
-				(path "/8c0b3d8b-46d3-4173-ab1e-a61765f77d61/1ea0e9ac-8f42-4d3d-8b47-067d751f5a51"
-					(reference "C42")
+				(path "/8c0b3d8b-46d3-4173-ab1e-a61765f77d61/db853a64-9343-4a36-b5b8-71001392b936"
+					(reference "C5")
 					(unit 1)
 				)
@@
 		(on_board yes)
 		(dnp no)
-		(property "Reference" "R70"
+		(property "Reference" "R16"
 			(at 80.01 99.06 90)
 			(effects
@@
 		(instances
 			(project "frank2"
-				(path "/8c0b3d8b-46d3-4173-ab1e-a61765f77d61/1ea0e9ac-8f42-4d3d-8b47-067d751f5a51"
-					(reference "R70")
+				(path "/8c0b3d8b-46d3-4173-ab1e-a61765f77d61/db853a64-9343-4a36-b5b8-71001392b936"
+					(reference "R16")
 					(unit 1)
 				)
@@
 		(dnp no)
 		(fields_autoplaced yes)
-		(property "Reference" "#PWR089"
+		(property "Reference" "#PWR040"
 			(at 67.31 137.16 0)
 			(effects
@@
 		(instances
 			(project "frank2"
-				(path "/8c0b3d8b-46d3-4173-ab1e-a61765f77d61/1ea0e9ac-8f42-4d3d-8b47-067d751f5a51"
-					(reference "#PWR089")
+				(path "/8c0b3d8b-46d3-4173-ab1e-a61765f77d61/db853a64-9343-4a36-b5b8-71001392b936"
+					(reference "#PWR040")
 					(unit 1)
 				)
@@
 		(dnp no)
 		(fields_autoplaced yes)
-		(property "Reference" "#PWR088"
+		(property "Reference" "#PWR039"
 			(at 87.63 77.47 0)
 			(effects
@@
 		(instances
 			(project ""
-				(path "/8c0b3d8b-46d3-4173-ab1e-a61765f77d61/1ea0e9ac-8f42-4d3d-8b47-067d751f5a51"
-					(reference "#PWR088")
+				(path "/8c0b3d8b-46d3-4173-ab1e-a61765f77d61/db853a64-9343-4a36-b5b8-71001392b936"
+					(reference "#PWR039")
 					(unit 1)
 				)
@@
 		(on_board yes)
 		(dnp no)
-		(property "Reference" "R69"
+		(property "Reference" "R15"
 			(at 100.33 96.52 90)
 			(effects
@@
 		(instances
 			(project "frank2"
-				(path "/8c0b3d8b-46d3-4173-ab1e-a61765f77d61/1ea0e9ac-8f42-4d3d-8b47-067d751f5a51"
-					(reference "R69")
+				(path "/8c0b3d8b-46d3-4173-ab1e-a61765f77d61/db853a64-9343-4a36-b5b8-71001392b936"
+					(reference "R15")
 					(unit 1)
 				)
@@
 		(dnp no)
 		(fields_autoplaced yes)
-		(property "Reference" "HDMI2"
+		(property "Reference" "HDMI1"
 			(at 43.18 91.4399 0)
 			(effects
@@
 			)
 		)
-		(property "Value" "HDMI Female"
+		(property "Value" "DC3RX19JA2"
 			(at 43.18 93.9799 0)
 			(effects
@@
 			)
 		)
-		(property "Datasheet" "https://eu.mouser.com/datasheet/2/418/8/ENG_CD_1747981_G-2018509.pdf"
+		(property "Datasheet" "https://www.mouser.com/datasheet/2/206/B_0233_2E_DC3-784461.pdf?srsltid=AfmBOopfNOwkdmYR2Zf10LYIa6wS_lfZGGRTVzb0297kvAyc-1zmhqWc"
 			(at 55.88 107.95 0)
 			(effects
@@
 		(instances
 			(project "frank2"
-				(path "/8c0b3d8b-46d3-4173-ab1e-a61765f77d61/1ea0e9ac-8f42-4d3d-8b47-067d751f5a51"
-					(reference "HDMI2")
+				(path "/8c0b3d8b-46d3-4173-ab1e-a61765f77d61/db853a64-9343-4a36-b5b8-71001392b936"
+					(reference "HDMI1")
 					(unit 1)
 				)
@@
 		(on_board yes)
 		(dnp no)
-		(property "Reference" "R75"
+		(property "Reference" "R21"
 			(at 90.17 119.38 90)
 			(effects
@@
 		(instances
 			(project "frank2"
-				(path "/8c0b3d8b-46d3-4173-ab1e-a61765f77d61/1ea0e9ac-8f42-4d3d-8b47-067d751f5a51"
-					(reference "R75")
+				(path "/8c0b3d8b-46d3-4173-ab1e-a61765f77d61/db853a64-9343-4a36-b5b8-71001392b936"
+					(reference "R21")
 					(unit 1)
 				)
@@
 		(on_board yes)
 		(dnp no)
-		(property "Reference" "R74"
+		(property "Reference" "R20"
 			(at 80.01 114.3 90)
 			(effects
@@
 		(instances
 			(project "frank2"
-				(path "/8c0b3d8b-46d3-4173-ab1e-a61765f77d61/1ea0e9ac-8f42-4d3d-8b47-067d751f5a51"
-					(reference "R74")
+				(path "/8c0b3d8b-46d3-4173-ab1e-a61765f77d61/db853a64-9343-4a36-b5b8-71001392b936"
+					(reference "R20")
 					(unit 1)
 				)

Commit message: FRANK M1 & M2 HW Revisions
Other:
- title: FRANK -> FRANK M2
Changed lines of the file:
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@@
 	(paper "A4")
 	(title_block
-		(title "FRANK")
-		(date "2025-02-18")
-		(rev "1.13")
+		(title "FRANK M2")
+		(date "2025-02-19")
+		(rev "2.1")
 		(company "Mikhail Matveev")
 		(comment 1 "https://github.com/xtremespb/frank")
