File: hardware/frank_m2/pico.kicad_sch (KiCad schematic)
At the start: 0 parts

Commit message: Names changed
Parts:
- added JP2: Jumper (Solder), FRANK:Jumper (solder), symbol Jumper:SolderJumper_2_Open
- added RP1: Rasberry Pi Pico, FRANK:Raspberry Pi Pico, symbol FRANK:Pico
Connections:
- new net: JP2.1 (A), RP1.36 (3V3)
- new net +3V3: JP2.2 (B)
- new net 5V_PICO: RP1.39 (VSYS)
- new net GND: RP1.13 (GND), RP1.18 (GND), RP1.23 (GND), RP1.28 (GND), RP1.3 (GND), RP1.33 (AGND), RP1.38 (GND), RP1.8 (GND)
- new net GPIO0: RP1.1 (GPIO0)
- new net GPIO1: RP1.2 (GPIO1)
- new net GPIO10: RP1.14 (GPIO10)
- new net GPIO11: RP1.15 (GPIO11)
- new net GPIO12: RP1.16 (GPIO12)
- new net GPIO13: RP1.17 (GPIO13)
- new net GPIO14: RP1.19 (GPIO14)
- new net GPIO15: RP1.20 (GPIO15)
- new net GPIO16: RP1.21 (GPIO16)
- new net GPIO17: RP1.22 (GPIO17)
- new net GPIO18: RP1.24 (GPIO18)
- new net GPIO19: RP1.25 (GPIO19)
- new net GPIO2: RP1.4 (GPIO2)
- new net GPIO20: RP1.26 (GPIO20)
- new net GPIO21: RP1.27 (GPIO21)
- new net GPIO22: RP1.29 (GPIO22)
- new net GPIO23: RP1.37 (3V3_EN)
- new net GPIO26: RP1.31 (GPIO26_ADC0)
- new net GPIO27: RP1.32 (GPIO27_ADC1)
- new net GPIO28: RP1.34 (GPIO28_ADC2)
- new net GPIO29: RP1.35 (ADC_VREF)
- new net GPIO3: RP1.5 (GPIO3)
- new net GPIO4: RP1.6 (GPIO4)
- new net GPIO5: RP1.7 (GPIO5)
- new net GPIO6: RP1.9 (GPIO6)
- new net GPIO7: RP1.10 (GPIO7)
- new net GPIO8: RP1.11 (GPIO8)
- new net GPIO9: RP1.12 (GPIO9)
- new net RUN: RP1.30 (RUN)
- new net VBUS: RP1.40 (VBUS)
Other:
- company: (none) -> Mikhail Matveev
- title: (none) -> FRANK

Commit message: FRANK M1 & M2 HW Revisions
Other:
- title: FRANK -> FRANK M2
Changed lines of the file:
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@@
 	(paper "A4")
 	(title_block
-		(title "FRANK")
-		(date "2025-02-18")
-		(rev "1.13")
+		(title "FRANK M2")
+		(date "2025-02-19")
+		(rev "2.1")
 		(company "Mikhail Matveev")
 		(comment 1 "https://github.com/xtremespb/frank")

Commit message: HW Rev 1.02 (M2)
Changed lines of the file:
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@@
 (kicad_sch
-	(version 20231120)
+	(version 20250114)
 	(generator "eeschema")
-	(generator_version "8.0")
+	(generator_version "9.0")
 	(paper "A4")
 	(title_block
 		(title "FRANK M2")
-		(date "2025-02-19")
-		(rev "2.1")
+		(date "2025-03-04")
+		(rev "1.02")
 		(company "Mikhail Matveev")
 		(comment 1 "https://github.com/xtremespb/frank")
@@
 		(shape input)
 		(at 105.41 69.85 0)
-		(fields_autoplaced yes)
 		(effects
 			(font
@@
 		(shape input)
 		(at 105.41 59.69 0)
-		(fields_autoplaced yes)
 		(effects
 			(font
@@
 		(shape input)
 		(at 44.45 57.15 180)
-		(fields_autoplaced yes)
 		(effects
 			(font
@@
 		(shape input)
 		(at 44.45 77.47 180)
-		(fields_autoplaced yes)
 		(effects
 			(font
@@
 		(shape input)
 		(at 105.41 80.01 0)
-		(fields_autoplaced yes)
 		(effects
 			(font
@@
 		(shape input)
 		(at 105.41 34.29 0)
-		(fields_autoplaced yes)
 		(effects
 			(font
@@
 		(shape input)
 		(at 44.45 39.37 180)
-		(fields_autoplaced yes)
 		(effects
 			(font
@@
 		(shape input)
 		(at 44.45 72.39 180)
-		(fields_autoplaced yes)
 		(effects
 			(font
@@
 		(shape input)
 		(at 105.41 44.45 0)
-		(fields_autoplaced yes)
 		(effects
 			(font
@@
 		(shape input)
 		(at 105.41 46.99 0)
-		(fields_autoplaced yes)
 		(effects
 			(font
@@
 		(shape input)
 		(at 105.41 54.61 0)
-		(fields_autoplaced yes)
 		(effects
 			(font
@@
 		(shape input)
 		(at 105.41 77.47 0)
-		(fields_autoplaced yes)
 		(effects
 			(font
@@
 		(shape input)
 		(at 44.45 69.85 180)
-		(fields_autoplaced yes)
 		(effects
 			(font
@@
 		(shape input)
 		(at 44.45 64.77 180)
-		(fields_autoplaced yes)
 		(effects
 			(font
@@
 		(shape input)
 		(at 44.45 34.29 180)
-		(fields_autoplaced yes)
 		(effects
 			(font
@@
 		(shape input)
 		(at 44.45 44.45 180)
-		(fields_autoplaced yes)
 		(effects
 			(font
@@
 		(shape input)
 		(at 105.41 64.77 0)
-		(fields_autoplaced yes)
 		(effects
 			(font
@@
 		(shape input)
 		(at 44.45 67.31 180)
-		(fields_autoplaced yes)
 		(effects
 			(font
@@
 		(shape input)
 		(at 44.45 52.07 180)
-		(fields_autoplaced yes)
 		(effects
 			(font
@@
 		(shape input)
 		(at 105.41 52.07 0)
-		(fields_autoplaced yes)
 		(effects
 			(font
@@
 		(shape input)
 		(at 44.45 31.75 180)
-		(fields_autoplaced yes)
 		(effects
 			(font
@@
 		(shape input)
 		(at 44.45 41.91 180)
-		(fields_autoplaced yes)
 		(effects
 			(font
@@
 		(shape input)
 		(at 44.45 54.61 180)
-		(fields_autoplaced yes)
 		(effects
 			(font
@@
 		(shape input)
 		(at 105.41 39.37 0)
-		(fields_autoplaced yes)
 		(effects
 			(font
@@
 		(shape input)
 		(at 105.41 67.31 0)
-		(fields_autoplaced yes)
 		(effects
 			(font
@@
 		(shape input)
 		(at 44.45 59.69 180)
-		(fields_autoplaced yes)
 		(effects
 			(font
@@
 		(shape input)
 		(at 44.45 46.99 180)
-		(fields_autoplaced yes)
 		(effects
 			(font
@@
 		(shape input)
 		(at 105.41 57.15 0)
-		(fields_autoplaced yes)
 		(effects
 			(font
@@
 		(shape input)
 		(at 44.45 80.01 180)
-		(fields_autoplaced yes)
 		(effects
 			(font
@@
 		(shape input)
 		(at 105.41 72.39 0)
-		(fields_autoplaced yes)
 		(effects
 			(font
@@
 		(dnp no)
 		(fields_autoplaced yes)
-		(property "Reference" "#PWR046"
+		(property "Reference" "#PWR064"
 			(at 38.1 74.93 0)
 			(effects
@@
 		(dnp no)
 		(fields_autoplaced yes)
-		(property "Reference" "#PWR042"
+		(property "Reference" "#PWR060"
 			(at 38.1 49.53 0)
 			(effects
@@
 		(dnp no)
 		(fields_autoplaced yes)
-		(property "Reference" "#PWR043"
+		(property "Reference" "#PWR061"
 			(at 111.76 49.53 0)
 			(effects
@@
 		(dnp no)
 		(fields_autoplaced yes)
-		(property "Reference" "#PWR041"
+		(property "Reference" "#PWR058"
 			(at 111.76 36.83 0)
 			(effects
@@
 		(dnp no)
 		(fields_autoplaced yes)
-		(property "Reference" "#PWR047"
+		(property "Reference" "#PWR065"
 			(at 111.76 74.93 0)
 			(effects
@@
 		(dnp no)
 		(fields_autoplaced yes)
-		(property "Reference" "#PWR040"
+		(property "Reference" "#PWR057"
 			(at 38.1 36.83 0)
 			(effects
@@
 		(dnp no)
 		(fields_autoplaced yes)
-		(property "Reference" "#PWR039"
+		(property "Reference" "#PWR056"
 			(at 101.6 31.75 0)
 			(effects
@@
 			)
 		)
-		(property "Datasheet" "https://cdn-shop.adafruit.com/product-files/4677/4677_esp-psram64_esp-psram64h_datasheet_en.pdf"
+		(property "Datasheet" "~"
 			(at 120.65 41.91 0)
 			(effects
@@
 			)
 		)
-		(property "Description" ""
+		(property "Description" "Solder Jumper, 2-pole, open"
 			(at 120.65 41.91 0)
 			(effects
@@
 		(dnp no)
 		(fields_autoplaced yes)
-		(property "Reference" "#PWR044"
+		(property "Reference" "#PWR062"
 			(at 38.1 62.23 0)
 			(effects
@@
 		(dnp no)
 		(fields_autoplaced yes)
-		(property "Reference" "#PWR045"
+		(property "Reference" "#PWR063"
 			(at 111.76 62.23 0)
 			(effects
