File: hardware/frank_m2/sd.kicad_sch (KiCad schematic)
At the start: 3 parts

Commit message: Names changed
Parts:
- SD1: value 47571-0001 -> 0475710001
- renumbered C43 to C4
Other:
- note added: "Short TF Card slot is used to save some space on the PCB."
- title: Frank M2 -> FRANK

Commit message: FRANK M1 & M2 HW Revisions
Other:
- title: FRANK -> FRANK M2
Changed lines of the file:
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@@
 	(paper "A4")
 	(title_block
-		(title "FRANK")
-		(date "2025-02-18")
-		(rev "1.13")
+		(title "FRANK M2")
+		(date "2025-02-19")
+		(rev "2.1")
 		(company "Mikhail Matveev")
 		(comment 1 "https://github.com/xtremespb/frank")
