File: hardware/frank_m2/tape.kicad_sch (KiCad schematic)
At the start: 11 parts, among them Q1 BC850, Q2 BC850

Commit message: Names changed
Parts:
- AJ1: value PJ-325C -> SJ1-353XNG
- Q1, Q2: AliExpress https://www.aliexpress.com/item/33017911878.html -> https://www.aliexpress.com/item/1005005008637286.html
- R2: AliExpress https://www.vishay.com/docs/28952/mcs0402at-mct0603at-mcu08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 -> https://www.aliexpress.com/item/1005005945735199.html
Other:
- note added: "This schematics is used to load data from external audio source, e.g. tape."
- title: Frank M2 -> FRANK
Changed lines of the file:
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@@
 	(paper "A4")
 	(title_block
-		(title "Frank M2")
-		(date "2025-02-02")
-		(rev "1.02")
+		(title "FRANK")
+		(date "2025-02-18")
+		(rev "1.13")
 		(company "Mikhail Matveev")
 		(comment 1 "https://github.com/xtremespb/frank")
@@
 			(width 0)
 			(type default)
+		)
+	)
+	(text "This schematics is used to load data from\nexternal audio source, e.g. tape."
+		(exclude_from_sim no)
+		(at 38.1 27.178 0)
+		(effects
+			(font
+				(size 1.27 1.27)
+			)
+			(justify left)
 		)
 	)
@@
 			)
 		)
-		(property "Datasheet" "https://www.vishay.com/docs/40002/293d.pdf"
+		(property "Datasheet" "https://www.vishay.com/docs/85748/1n4148w.pdf"
 			(at 93.98 64.77 0)
 			(effects
@@
 			)
 			(project ""
-				(path "/8c0b3d8b-46d3-4173-ab1e-a61765f77d61/49084664-1062-4a43-8f46-2816e4bba858"
-					(reference "D14")
+				(path "/8c0b3d8b-46d3-4173-ab1e-a61765f77d61/599e2208-d0f7-4f1d-beb8-3b4e6272cb10"
+					(reference "D7")
 					(unit 1)
 				)
@@
 			)
 			(project ""
-				(path "/8c0b3d8b-46d3-4173-ab1e-a61765f77d61/49084664-1062-4a43-8f46-2816e4bba858"
-					(reference "#PWR085")
+				(path "/8c0b3d8b-46d3-4173-ab1e-a61765f77d61/599e2208-d0f7-4f1d-beb8-3b4e6272cb10"
+					(reference "#PWR054")
 					(unit 1)
 				)
@@
 			)
 			(project "38NJU24"
-				(path "/8c0b3d8b-46d3-4173-ab1e-a61765f77d61/49084664-1062-4a43-8f46-2816e4bba858"
-					(reference "R65")
+				(path "/8c0b3d8b-46d3-4173-ab1e-a61765f77d61/599e2208-d0f7-4f1d-beb8-3b4e6272cb10"
+					(reference "R30")
 					(unit 1)
 				)
@@
 			)
 			(project ""
-				(path "/8c0b3d8b-46d3-4173-ab1e-a61765f77d61/49084664-1062-4a43-8f46-2816e4bba858"
-					(reference "#PWR084")
+				(path "/8c0b3d8b-46d3-4173-ab1e-a61765f77d61/599e2208-d0f7-4f1d-beb8-3b4e6272cb10"
+					(reference "#PWR053")
 					(unit 1)
 				)
@@
 			)
 		)
-		(property "AliExpress" "https://www.vishay.com/docs/28952/mcs0402at-mct0603at-mcu0805at-mca1206at.pdf"
+		(property "AliExpress" "https://www.aliexpress.com/item/1005005945735199.html"
 			(at 116.84 53.34 0)
 			(effects
@@
 			)
 			(project "38NJU24"
-				(path "/8c0b3d8b-46d3-4173-ab1e-a61765f77d61/49084664-1062-4a43-8f46-2816e4bba858"
-					(reference "R64")
+				(path "/8c0b3d8b-46d3-4173-ab1e-a61765f77d61/599e2208-d0f7-4f1d-beb8-3b4e6272cb10"
+					(reference "R29")
 					(unit 1)
 				)
@@
 			)
 		)
-		(property "Value" "PJ-325C"
+		(property "Value" "SJ1-353XNG"
 			(at 46.99 66.04 0)
 			(effects
@@
 			)
 			(project "38NJU24"
-				(path "/8c0b3d8b-46d3-4173-ab1e-a61765f77d61/49084664-1062-4a43-8f46-2816e4bba858"
-					(reference "AJ4")
+				(path "/8c0b3d8b-46d3-4173-ab1e-a61765f77d61/599e2208-d0f7-4f1d-beb8-3b4e6272cb10"
+					(reference "AJ2")
 					(unit 1)
 				)
@@
 			)
 		)
-		(property "Datasheet" "https://eu.mouser.com/datasheet/2/447/KEM_C1075_X7R_HT_SMD-3316221.pdf"
+		(property "Datasheet" "https://eu.mouser.com/datasheet/2/40/KGM_X7R-3223212.pdf"
 			(at 69.85 72.39 0)
 			(effects
@@
 			)
 			(project "38NJU24"
-				(path "/8c0b3d8b-46d3-4173-ab1e-a61765f77d61/49084664-1062-4a43-8f46-2816e4bba858"
-					(reference "C41")
+				(path "/8c0b3d8b-46d3-4173-ab1e-a61765f77d61/599e2208-d0f7-4f1d-beb8-3b4e6272cb10"
+					(reference "C13")
 					(unit 1)
 				)
@@
 			)
 			(project ""
-				(path "/8c0b3d8b-46d3-4173-ab1e-a61765f77d61/49084664-1062-4a43-8f46-2816e4bba858"
-					(reference "#PWR083")
+				(path "/8c0b3d8b-46d3-4173-ab1e-a61765f77d61/599e2208-d0f7-4f1d-beb8-3b4e6272cb10"
+					(reference "#PWR052")
 					(unit 1)
 				)
@@
 			)
 			(project "38NJU24"
-				(path "/8c0b3d8b-46d3-4173-ab1e-a61765f77d61/49084664-1062-4a43-8f46-2816e4bba858"
-					(reference "R66")
+				(path "/8c0b3d8b-46d3-4173-ab1e-a61765f77d61/599e2208-d0f7-4f1d-beb8-3b4e6272cb10"
+					(reference "R31")
 					(unit 1)
 				)
@@
 			)
 			(project ""
-				(path "/8c0b3d8b-46d3-4173-ab1e-a61765f77d61/49084664-1062-4a43-8f46-2816e4bba858"
-					(reference "#PWR082")
+				(path "/8c0b3d8b-46d3-4173-ab1e-a61765f77d61/599e2208-d0f7-4f1d-beb8-3b4e6272cb10"
+					(reference "#PWR051")
 					(unit 1)
 				)
@@
 			)
 			(project ""
-				(path "/8c0b3d8b-46d3-4173-ab1e-a61765f77d61/49084664-1062-4a43-8f46-2816e4bba858"
-					(reference "#PWR086")
+				(path "/8c0b3d8b-46d3-4173-ab1e-a61765f77d61/599e2208-d0f7-4f1d-beb8-3b4e6272cb10"
+					(reference "#PWR055")
 					(unit 1)
 				)
@@
 			)
 			(project ""
-				(path "/8c0b3d8b-46d3-4173-ab1e-a61765f77d61/49084664-1062-4a43-8f46-2816e4bba858"
-					(reference "#PWR081")
+				(path "/8c0b3d8b-46d3-4173-ab1e-a61765f77d61/599e2208-d0f7-4f1d-beb8-3b4e6272cb10"
+					(reference "#PWR050")
 					(unit 1)
 				)
@@
 			)
 		)
-		(property "Datasheet" "https://eu.mouser.com/datasheet/2/447/KEM_C1075_X7R_HT_SMD-3316221.pdf"
+		(property "Datasheet" "https://eu.mouser.com/datasheet/2/40/KGM_X7R-3223212.pdf"
 			(at 132.08 50.8 0)
 			(effects
@@
 			)
 			(project "38NJU24"
-				(path "/8c0b3d8b-46d3-4173-ab1e-a61765f77d61/49084664-1062-4a43-8f46-2816e4bba858"
-					(reference "C40")
+				(path "/8c0b3d8b-46d3-4173-ab1e-a61765f77d61/599e2208-d0f7-4f1d-beb8-3b4e6272cb10"
+					(reference "C12")
 					(unit 1)
 				)
@@
 			)
 			(project "38NJU24"
-				(path "/8c0b3d8b-46d3-4173-ab1e-a61765f77d61/49084664-1062-4a43-8f46-2816e4bba858"
-					(reference "R67")
+				(path "/8c0b3d8b-46d3-4173-ab1e-a61765f77d61/599e2208-d0f7-4f1d-beb8-3b4e6272cb10"
+					(reference "R32")
 					(unit 1)
 				)
@@
 			)
 		)
-		(property "Datasheet" "http://www.infineon.com/dgdl/Infineon-BC847SERIES_BC848SERIES_BC849SERIES_BC850SERIES-DS-v01_01-en.pdf?fileId=db3a304314dca389011541d4630a1657"
+		(property "Datasheet" "https://assets.nexperia.com/documents/data-sheet/BC849_BC850.pdf"
 			(at 96.52 72.39 0)
 			(effects
@@
 			)
 		)
-		(property "AliExpress" "https://www.aliexpress.com/item/33017911878.html"
+		(property "AliExpress" "https://www.aliexpress.com/item/1005005008637286.html"
 			(at 96.52 72.39 0)
 			(effects
@@
 			)
 			(project "38NJU24"
-				(path "/8c0b3d8b-46d3-4173-ab1e-a61765f77d61/49084664-1062-4a43-8f46-2816e4bba858"
-					(reference "Q6")
+				(path "/8c0b3d8b-46d3-4173-ab1e-a61765f77d61/599e2208-d0f7-4f1d-beb8-3b4e6272cb10"
+					(reference "Q2")
 					(unit 1)
 				)
@@
 			)
 			(project "38NJU24"
-				(path "/8c0b3d8b-46d3-4173-ab1e-a61765f77d61/49084664-1062-4a43-8f46-2816e4bba858"
-					(reference "R63")
+				(path "/8c0b3d8b-46d3-4173-ab1e-a61765f77d61/599e2208-d0f7-4f1d-beb8-3b4e6272cb10"
+					(reference "R28")
 					(unit 1)
 				)
@@
 			)
 		)
-		(property "Datasheet" "http://www.infineon.com/dgdl/Infineon-BC847SERIES_BC848SERIES_BC849SERIES_BC850SERIES-DS-v01_01-en.pdf?fileId=db3a304314dca389011541d4630a1657"
+		(property "Datasheet" "https://assets.nexperia.com/documents/data-sheet/BC849_BC850.pdf"
 			(at 114.3 64.77 0)
 			(effects
@@
 			)
 		)
-		(property "AliExpress" "https://www.aliexpress.com/item/33017911878.html"
+		(property "AliExpress" "https://www.aliexpress.com/item/1005005008637286.html"
 			(at 114.3 64.77 0)
 			(effects
@@
 			)
 			(project "38NJU24"
-				(path "/8c0b3d8b-46d3-4173-ab1e-a61765f77d61/49084664-1062-4a43-8f46-2816e4bba858"
-					(reference "Q5")
-					(unit 1)
-				)
+				(path "/8c0b3d8b-46d3-4173-ab1e-a61765f77d61/599e2208-d0f7-4f1d-beb8-3b4e6272cb10"
+					(reference "Q1")
+					(unit 1)
+				)

Commit message: FRANK M1 & M2 HW Revisions
Other:
- title: FRANK -> FRANK M2
Changed lines of the file:
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@@
 	(paper "A4")
 	(title_block
-		(title "FRANK")
-		(date "2025-02-18")
-		(rev "1.13")
+		(title "FRANK M2")
+		(date "2025-02-19")
+		(rev "2.1")
 		(company "Mikhail Matveev")
 		(comment 1 "https://github.com/xtremespb/frank")

Commit message: HW Rev 1.02 (M2)
Parts:
- renumbered AJ1 to AJ2, C1 to C12, C2 to C13, D1 to D7, R1 to R28, R2 to R29, R3 to R30, R4 to R31, R5 to R32
Changed lines of the file:
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@@
 (kicad_sch
-	(version 20231120)
+	(version 20250114)
 	(generator "eeschema")
-	(generator_version "8.0")
+	(generator_version "9.0")
 	(paper "A4")
 	(title_block
 		(title "FRANK M2")
-		(date "2025-02-19")
-		(rev "2.1")
+		(date "2025-03-04")
+		(rev "1.02")
 		(company "Mikhail Matveev")
 		(comment 1 "https://github.com/xtremespb/frank")
+	)
+	(text "This schematics is used to load data from\nexternal audio source, e.g. tape."
+		(exclude_from_sim no)
+		(at 38.1 27.178 0)
+		(effects
+			(font
+				(size 1.27 1.27)
+			)
+			(justify left)
+		)
 	)
 	(junction
@@
 		)
 	)
-	(text "This schematics is used to load data from\nexternal audio source, e.g. tape."
-		(exclude_from_sim no)
-		(at 38.1 27.178 0)
+	(label "LOAD_IN"
+		(at 49.53 72.39 0)
 		(effects
 			(font
 				(size 1.27 1.27)
 			)
-			(justify left)
-		)
-	)
-	(label "LOAD_IN"
-		(at 49.53 72.39 0)
-		(fields_autoplaced yes)
-		(effects
-			(font
-				(size 1.27 1.27)
-			)
 			(justify left bottom)
 		)
@@
 		(shape input)
 		(at 138.43 66.04 0)
-		(fields_autoplaced yes)
 		(effects
 			(font
@@
 		(dnp no)
 		(fields_autoplaced yes)
-		(property "Reference" "D1"
+		(property "Reference" "D7"
 			(at 93.98 58.42 0)
 			(effects
@@
 		(dnp no)
 		(fields_autoplaced yes)
-		(property "Reference" "#PWR07"
+		(property "Reference" "#PWR054"
 			(at 99.06 93.98 0)
 			(effects
@@
 		(dnp no)
 		(fields_autoplaced yes)
-		(property "Reference" "R3"
+		(property "Reference" "R30"
 			(at 105.41 58.42 90)
 			(effects
@@
 		(dnp no)
 		(fields_autoplaced yes)
-		(property "Reference" "#PWR06"
+		(property "Reference" "#PWR053"
 			(at 66.04 93.98 0)
 			(effects
@@
 		(dnp no)
 		(fields_autoplaced yes)
-		(property "Reference" "R2"
+		(property "Reference" "R29"
 			(at 119.38 52.0699 0)
 			(effects
@@
 		(on_board yes)
 		(dnp no)
-		(property "Reference" "AJ1"
+		(property "Reference" "AJ2"
 			(at 37.3381 73.4603 0)
 			(effects
@@
 		(on_board yes)
 		(dnp no)
-		(property "Reference" "C2"
+		(property "Reference" "C13"
 			(at 71.12 68.58 90)
 			(effects
@@
 		(dnp no)
 		(fields_autoplaced yes)
-		(property "Reference" "#PWR05"
+		(property "Reference" "#PWR052"
 			(at 55.88 80.01 0)
 			(effects
@@
 		(dnp no)
 		(fields_autoplaced yes)
-		(property "Reference" "R4"
+		(property "Reference" "R31"
 			(at 81.28 66.04 90)
 			(effects
@@
 		(dnp no)
 		(fields_autoplaced yes)
-		(property "Reference" "#PWR04"
+		(property "Reference" "#PWR051"
 			(at 138.43 58.42 0)
 			(effects
@@
 		(dnp no)
 		(fields_autoplaced yes)
-		(property "Reference" "#PWR08"
+		(property "Reference" "#PWR055"
 			(at 116.84 93.98 0)
 			(effects
@@
 		(dnp no)
 		(fields_autoplaced yes)
-		(property "Reference" "#PWR03"
+		(property "Reference" "#PWR050"
 			(at 121.92 43.18 0)
 			(effects
@@
 		(on_board yes)
 		(dnp no)
-		(property "Reference" "C1"
+		(property "Reference" "C12"
 			(at 135.001 49.6316 0)
 			(effects
@@
 		(dnp no)
 		(fields_autoplaced yes)
-		(property "Reference" "R5"
+		(property "Reference" "R32"
 			(at 67.818 82.6078 0)
 			(effects
@@
 	)
 	(symbol
+		(lib_name "BC850_1")
 		(lib_id "Transistor_BJT:BC850")
 		(at 96.52 72.39 0)
@@
 			)
 		)
-		(property "Datasheet" "https://assets.nexperia.com/documents/data-sheet/BC849_BC850.pdf"
+		(property "Datasheet" "http://www.infineon.com/dgdl/Infineon-BC847SERIES_BC848SERIES_BC849SERIES_BC850SERIES-DS-v01_01-en.pdf?fileId=db3a304314dca389011541d4630a1657"
 			(at 96.52 72.39 0)
 			(effects
@@
 			)
 		)
-		(property "Description" ""
+		(property "Description" "0.1A Ic, 45V Vce, NPN Transistor, SOT-23"
 			(at 96.52 72.39 0)
 			(effects
@@
 		(dnp no)
 		(fields_autoplaced yes)
-		(property "Reference" "R1"
+		(property "Reference" "R28"
 			(at 101.6 52.0699 0)
 			(effects
@@
 			)
 		)
-		(property "Datasheet" "https://assets.nexperia.com/documents/data-sheet/BC849_BC850.pdf"
+		(property "Datasheet" "http://www.infineon.com/dgdl/Infineon-BC847SERIES_BC848SERIES_BC849SERIES_BC850SERIES-DS-v01_01-en.pdf?fileId=db3a304314dca389011541d4630a1657"
 			(at 114.3 64.77 0)
 			(effects
@@
 			)
 		)
-		(property "Description" ""
+		(property "Description" "0.1A Ic, 45V Vce, NPN Transistor, SOT-23"
 			(at 114.3 64.77 0)
 			(effects
