File: hardware/frank_m2/vga.kicad_sch (KiCad schematic)
At the start: 0 parts

Commit message: Names changed
Parts:
- added R37, R38, R39: 330R, FRANK:Resistor (0805), symbol Device:R
- added R40, R41, R42: 1K, FRANK:Resistor (0805), symbol Device:R
- added R43, R44: 100R, FRANK:Resistor (0805), symbol Device:R
- added VGA1: D-SUB 15 Female, FRANK:D-SUB (15 pin, female), symbol FRANK:VGA
Connections:
- new net: R39.2, R42.2, VGA1.3
- new net: R44.1, VGA1.14
- new net: R37.2, R40.2, VGA1.1
- new net: R43.1, VGA1.13
- new net: R38.2, R41.2, VGA1.2
- new net GND: VGA1.0, VGA1.10, VGA1.5, VGA1.6, VGA1.7, VGA1.8
- new net VGA_B: R42.1
- new net VGA_BH: R39.1
- new net VGA_G: R41.1
- new net VGA_GH: R38.1
- new net VGA_HS: R43.2
- new net VGA_R: R40.1
- new net VGA_RH: R37.1
- new net VGA_VS: R44.2
- no-connect marks 0 -> 5
Other:
- company: (none) -> Mikhail Matveev
- title: (none) -> FRANK

Commit message: FRANK M1 & M2 HW Revisions
Other:
- title: FRANK -> FRANK M2
Changed lines of the file:
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@@
 	(paper "A4")
 	(title_block
-		(title "FRANK")
-		(date "2025-02-18")
-		(rev "1.13")
+		(title "FRANK M2")
+		(date "2025-02-19")
+		(rev "2.1")
 		(company "Mikhail Matveev")
 		(comment 1 "https://github.com/xtremespb/frank")
@@
 			)
 		)
-		(property "Datasheet" "~"
+		(property "Datasheet" "https://gr.mouser.com/datasheet/2/418/8/ENG_CD_2301844_H-2497630.pdf"
 			(at 80.01 46.99 0)
 			(effects
