File: hardware/versa/usba.kicad_sch (KiCad schematic)
At the start: 2 parts, among them J1 676430910

Commit message: HW Rev 2.01
Parts:
- USB2: renamed from J1; footprint Connector_USB:USB_A_Molex_67643_Horizontal -> FRANK:USB Type A (single)
Changed lines of the file:
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@@
 	(title_block
 		(title "VersaTerm")
-		(date "2025-01-29")
-		(rev "2.0")
+		(date "2025-02-03")
+		(rev "2.01")
 		(company "Mikhail Matveev")
 		(comment 1 "https://github.com/xtremespb/frank")
@@
 		(dnp no)
 		(fields_autoplaced yes)
-		(property "Reference" "J1"
+		(property "Reference" "USB2"
 			(at 39.37 29.21 0)
 			(effects
@@
 			)
 		)
-		(property "Footprint" "Connector_USB:USB_A_Molex_67643_Horizontal"
+		(property "Footprint" "FRANK:USB Type A (single)"
 			(at 43.18 43.18 0)
 			(effects
@@
 			(project ""
 				(path "/8c0b3d8b-46d3-4173-ab1e-a61765f77d61/f7082aa6-6a82-45dd-9ad2-9a491cd5702e"
-					(reference "J1")
+					(reference "USB2")
 					(unit 1)
 				)
