File: hardware/versa/versa.kicad_pcb (KiCad board)
At the start: 2 copper layers, 52.2 x 54.4 mm, 69 parts, among them SW1 Flash Button, SW2 Button, SW4 Reset Button, U1 NCP1117-3.3_SOT223, Y1 12 MHz

Commit message: WIP
Parts:
- removed G***: LOGO, LIBS:RS232_LOGO
- removed KB1: PS/2, LIBS:Connector_Mini-DIN_Female_6Pin_2rows
- removed SW4: Reset Button, LIBS:Button_SMD_3x3x2
- added C24: 10u, FRANK:Capacitor (0805), F.Cu at (92.9, 34.6)
- added J1: 676430910, Connector_USB:USB_A_Molex_67643_Horizontal, F.Cu at (96.1, 19.1)
- added J2: Pin Header (1x04), FRANK:Pin Header (1x04), F.Cu at (81.0, 93.9)
- added SW3: KLS7-TS3302, FRANK:Button (SMD, 3x3mm), F.Cu at (99.8, 38.9)
- C1, C10, C14, C16, C17, C2, C4, C6, C7, C8, C9: footprint LIBS:Medved_C_0805 -> FRANK:Capacitor (0805)
- C11, C12: value 100n -> 1u; footprint LIBS:Medved_C_0805 -> FRANK:Capacitor (0805)
- C13: value 15p -> 100n; footprint LIBS:Medved_C_0805 -> FRANK:Capacitor (0805)
- C15: value 100n -> 15p; footprint LIBS:Medved_C_0805 -> FRANK:Capacitor (0805)
- C18, C23: value 0.1u -> 100n; footprint LIBS:Medved_C_0805 -> FRANK:Capacitor (0805)
- C19, C20, C21, C22: footprint LIBS:Medved_CP_Radial_D5.0mm_P2.50mm -> FRANK:Capacitor (0805)
- C3, C5: value 1u -> 100n; footprint LIBS:Medved_C_0805 -> FRANK:Capacitor (0805)
- COM1: value RS232 -> D-SUB 9 Male; footprint LIBS:DSUB-9 -> FRANK:D-SUB (9 pin, male, top mount)
- D1, D2, D3, D4: footprint LIBS:Medved_D_0805 -> FRANK:Diode (SOD-323)
- FL1: value W25Q128JVS -> W25Q128JVSIQ; footprint LIBS:Medved_SOIC-8_5.23x5.23mm_P1.27mm -> FRANK:SOIC-8
- HDMI1: value HDMI -> DC3RX19JA2; footprint LIBS:HDMI -> FRANK:HDMI (female)
- JP1: footprint LIBS:Medved_Jumper_Solder -> FRANK:Jumper (solder)
- L1: value LED -> Blue; footprint LIBS:Medved_L_0805 -> FRANK:LED (0805)
- L2: value GREEN -> Green; footprint LIBS:Medved_L_0805 -> FRANK:LED (0805)
- MAX1: footprint LIBS:SOIC127P600X175-16N -> FRANK:SOIC127P600X175-16N
- R1: value 27 -> 27R; footprint LIBS:Medved_R_0805 -> FRANK:Resistor (0805)
- R10: value 1k -> 100R; footprint LIBS:Medved_R_0805 -> FRANK:Resistor (0805)
- R11, R13, R14, R15, R16, R17, R18, R19, R20, R21, R22, R4, R6, R7, R8: footprint LIBS:Medved_R_0805 -> FRANK:Resistor (0805)
- R12: value 100R -> 1K; footprint LIBS:Medved_R_0805 -> FRANK:Resistor (0805)
- R2: value 27 -> 1K; footprint LIBS:Medved_R_0805 -> FRANK:Resistor (0805)
- R3: value 1k -> 27R; footprint LIBS:Medved_R_0805 -> FRANK:Resistor (0805)
- R5, R9: value 1k -> 1K; footprint LIBS:Medved_R_0805 -> FRANK:Resistor (0805)
- RP1: footprint LIBS:RP2040-QFN-56 -> FRANK:QFN 56
- SW1: footprint LIBS:Button_SMD_3x3x2 -> FRANK:Button (SMD, 3x3mm)
- SW2: value Button -> KLS7-TS3302; footprint LIBS:Button_SMD_3x3x2 -> FRANK:Button (SMD, 3x3mm)
- U1: value NCP1117-3.3_SOT223 -> NCP1117 3.3; footprint LIBS:Medved_SOT-223-3_TabPin2 -> FRANK:SOT-223
- USB1: value USB Type C -> USB4215; footprint LIBS:USB-TYPE-C-31-M-12_lib2 -> FRANK:USB Type C
- Y1: footprint LIBS:Medved_CRYSTAL_3225 -> FRANK:Crystal (3225)
- moved H2 151.3 mm to (85.0, 26.2)
- moved C19 135.4 mm to (124.9, 167.6)
- moved H3 131.8 mm to (85.0, 33.2)
- moved SW2 129.5 mm to (91.8, 38.9), turned to 0 degrees
- moved C20 127.6 mm to (124.9, 170.6)
- moved C18 124.8 mm to (90.4, 99.0)
- moved C21 124.1 mm to (124.9, 173.6)
- moved R14 121.0 mm to (138.2, 170.5), turned to 0 degrees
- moved C22 120.6 mm to (124.9, 176.6)
- moved MAX1 118.7 mm to (131.6, 171.9), turned to 0 degrees
- moved H1 118.6 mm to (85.0, 19.3)
- moved D4 117.4 mm to (143.2, 170.5), turned to 0 degrees
- moved R13 116.4 mm to (138.2, 167.6), turned to 0 degrees
- moved R9 116.0 mm to (85.6, 93.0), turned to 0 degrees
- moved R11 114.3 mm to (85.6, 99.0), turned to 0 degrees
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Connections:
- net /BTN_DEF renamed /GPIO14
- net /CTS_PICO renamed /GPIO18
- net /HDMI_D0P renamed /GPIO9
- net /HDMI_D1N renamed /GPIO10
- net /JMP_HDMI renamed /GPIO15
- net /RTS_PICO renamed /GPIO19
- net /RX_PICO renamed /GPIO17
- net /TX_PICO renamed /GPIO16
- C11 pad 1: +3V3 -> Net-(RP1-VREG_VOUT)
- C13 pad 1: /RP2040/XIN -> +3V3
- C15 pad 1: +3V3 -> /RP2040/XIN
- C19 pad 1: /RS232/C2+ -> /RS232/V+
- C19 pad 2: /RS232/C2- -> VBUS
- C20 pad 1: GND -> /RS232/C1-
- C20 pad 2: /RS232/V- -> /RS232/C1+
- C21 pad 1: /RS232/C1+ -> /RS232/C2-
- C21 pad 2: /RS232/C1- -> /RS232/C2+
- C22 pad 1: /RS232/V+ -> /RS232/V-
- C22 pad 2: VBUS -> GND
- C3 pad 1: Net-(RP1-VREG_VOUT) -> +3V3
- D1 pad 1: /PS2_CLK -> /GPIO0
- D2 pad 1: /PS2_DATA -> /GPIO1
- R10 pad 1: VBUS -> Net-(J2-Pin_3)
- R10 pad 2: Net-(KB1-Pad1) -> /GPIO0
- R11 pad 1: Net-(KB1-Pad5) -> Net-(J2-Pin_2)
- R11 pad 2: /PS2_CLK -> /GPIO1
- R12 pad 1: Net-(KB1-Pad1) -> VBUS
- R12 pad 2: /PS2_DATA -> Net-(J2-Pin_2)
- R15 pad 1: Net-(HDMI1-D0N) -> Net-(HDMI1-CLKN)
- R15 pad 2: /HDMI_D0N -> /GPIO6
- R16 pad 1: Net-(HDMI1-D2N) -> Net-(HDMI1-CLKP)
- R16 pad 2: /HDMI_D2N -> /GPIO7
- R17 pad 1: Net-(HDMI1-CLKN) -> Net-(HDMI1-D0N)
- R17 pad 2: /HDMI_CLKN -> /GPIO8
- R2 pad 1: /D- -> /RP2040/QSPI_SS
- R2 pad 2: Net-(RP1-USB_DM) -> /RP2040/~{USB_BOOT}
- R20 pad 1: Net-(HDMI1-D2P) -> Net-(HDMI1-D1P)
- R20 pad 2: /HDMI_D2P -> /GPIO11
- R21 pad 1: Net-(HDMI1-CLKP) -> Net-(HDMI1-D2N)
- R21 pad 2: /HDMI_CLKP -> /GPIO12
- R22 pad 1: Net-(HDMI1-D1P) -> Net-(HDMI1-D2P)
- R22 pad 2: /HDMI_D1P -> /GPIO13
- R3 pad 1: /RP2040/QSPI_SS -> /D-
- R3 pad 2: /RP2040/~{USB_BOOT} -> Net-(RP1-USB_DM)
- R4 pad 1: Net-(L1-A) -> /RP2040/XOUT
- R4 pad 2: /RP2040/GPIO25 -> Net-(C14-Pad1)
- R5 pad 1: /RP2040/XOUT -> Net-(L1-A)
- R5 pad 2: Net-(C14-Pad1) -> /RP2040/GPIO25
- R9 pad 2: Net-(KB1-Pad5) -> Net-(J2-Pin_3)
- RP1 pad 11: /HDMI_D0N -> /GPIO8
- RP1 pad 14: /HDMI_D1P -> /GPIO11
- RP1 pad 15: /HDMI_D2N -> /GPIO12
- RP1 pad 16: /HDMI_D2P -> /GPIO13
- RP1 pad 2: /PS2_CLK -> /GPIO0
- RP1 pad 3: /PS2_DATA -> /GPIO1
- RP1 pad 8: /HDMI_CLKN -> /GPIO6
- RP1 pad 9: /HDMI_CLKP -> /GPIO7
Routing:
- net VBUS: track 202.2 -> 0.00 mm, vias 2 -> 0
- net +3V3: track 151.8 -> 0.00 mm
- net /GPIO14: track 42.5 -> 0.00 mm, vias 2 -> 0
- net /RUN: track 37.2 -> 0.00 mm, vias 4 -> 0
- net /RS232/CTS_IN: track 34.9 -> 0.00 mm, vias 3 -> 0
- net /RS232/RTS_IN: track 29.1 -> 0.00 mm, vias 1 -> 0
- net /PS2_CLK: track 28.9 -> 0.00 mm, vias 2 -> 0
- net /RP2040/~{USB_BOOT}: track 27.4 -> 0.00 mm
- net Net-(RP1-VREG_VOUT): track 25.4 -> 0.00 mm
- net /RS232/C2-: track 24.0 -> 0.00 mm, vias 1 -> 0
- net /GPIO17: track 23.8 -> 0.00 mm, vias 4 -> 0
- net /RP2040/QSPI_SS: track 23.7 -> 0.00 mm, vias 2 -> 0
- net /PS2_DATA: track 22.7 -> 0.00 mm, vias 2 -> 0
- net /RS232/RX_IN: track 22.4 -> 0.00 mm, vias 2 -> 0
- net /RS232/TX_IN: track 22.0 -> 0.00 mm, vias 2 -> 0
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- removed copper zone on B.Cu, net GND
- removed copper zone on F.Cu, net GND
Other:
- board outline removed
- board text removed: "BOOT"
- board text removed: "DEFAULTS"
- board text removed: "HW REV 1.0"
- board text removed: "RESET"
- board text removed: "RH1.DEV"

Commit message: HW Rev 2.01
Parts:
- removed J1: 676430910, Connector_USB:USB_A_Molex_67643_Horizontal
- removed J2: Pin Header (1x04), FRANK:Pin Header (1x04)
- added KB1: PS/2, FRANK:MiniDIN (6 Pin, female), F.Cu at (175.4, 99.0)
- added USB2: 676430910, FRANK:USB Type A (single), F.Cu at (198.0, 99.8)
- R10: value 100R -> 1k
- R12: value 1K -> 100R
- moved H4 150.8 mm to (205.3, 131.1)
- moved H2 137.7 mm to (205.3, 93.3)
- moved SW2 134.2 mm to (191.8, 128.4), turned to -90 degrees
- moved SW3 131.5 mm to (196.1, 128.4), turned to -90 degrees
- moved C24 130.0 mm to (205.6, 99.5), turned to -90 degrees
- moved H3 112.6 mm to (140.6, 131.1)
- moved SW1 102.7 mm to (197.1, 131.7), turned to 90 degrees
- moved JP1 99.6 mm to (162.8, 115.3)
- moved C7 98.9 mm to (173.8, 129.9), turned to -90 degrees
- moved C13 94.6 mm to (198.9, 121.5)
- moved R22 93.4 mm to (151.0, 104.1), turned to -90 degrees
- moved R2 93.3 mm to (198.9, 124.5)
- moved Y1 93.3 mm to (167.2, 129.2), turned to 90 degrees
- moved C14 92.9 mm to (162.5, 127.0), turned to 180 degrees
- moved C10 92.8 mm to (182.3, 131.7)
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Connections:
- R10 pad 1: Net-(J2-Pin_3) -> VBUS
- R10 pad 2: /GPIO0 -> Net-(KB1-Pad1)
- R11 pad 1: Net-(J2-Pin_2) -> Net-(KB1-Pad5)
- R11 pad 2: /GPIO1 -> /GPIO0
- R12 pad 1: VBUS -> Net-(KB1-Pad1)
- R12 pad 2: Net-(J2-Pin_2) -> /GPIO1
- R9 pad 2: Net-(J2-Pin_3) -> Net-(KB1-Pad5)
Routing:
- net +3V3: track 0.00 -> 228.7 mm, vias 0 -> 2
- net VBUS: track 0.00 -> 180.7 mm
- net /D-: track 0.00 -> 51.5 mm, vias 0 -> 2
- net /D+: track 0.00 -> 40.4 mm, vias 0 -> 2
- net /GPIO14: track 0.00 -> 40.2 mm, vias 0 -> 4
- net /RP2040/GPIO25: track 0.00 -> 37.1 mm, vias 0 -> 2
- net Net-(RP1-VREG_VOUT): track 0.00 -> 36.1 mm, vias 0 -> 4
- net /RUN: track 0.00 -> 31.3 mm, vias 0 -> 2
- net /GPIO19: track 0.00 -> 30.9 mm, vias 0 -> 2
- net /GPIO13: track 0.00 -> 30.8 mm, vias 0 -> 2
- net /RP2040/QSPI_SS: track 0.00 -> 27.0 mm
- net /GPIO10: track 0.00 -> 23.8 mm, vias 0 -> 2
- net /RP2040/QSPI_SD0: track 0.00 -> 23.5 mm, vias 0 -> 2
- net /GPIO12: track 0.00 -> 23.4 mm, vias 0 -> 2
- net /RP2040/QSPI_SCLK: track 0.00 -> 23.1 mm
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- added copper zone on B.Cu, net GND
- added copper zone on F.Cu, net GND
Other:
- board outline added: 70.3 x 43.4 mm
- board text added: "Boot"
- board text added: "Defaults"
- board text added: "HW REV 2.01"
- board text added: "Reset"
- board text added: "Versa"
- board text added: "https://rh1.dev"
