File: hardware/frank_m2u/rp2040.kicad_sch (KiCad schematic)
At the start: 21 parts, among them SW3 Boot, U3 W25Q128JVSIQ, U4 RP2040

Commit message: WIP
Other:
- title: Valera-2350A -> Frank M2U
Changed lines of the file:
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@@
 	(paper "A4")
 	(title_block
-		(title "Valera-2350A")
-		(date "2025-01-30")
-		(rev "1.0")
+		(title "Frank M2U")
+		(date "2025-02-06")
+		(rev "1.00")
 		(company "Mikhail Matveev")
 		(comment 1 "https://github.com/xtremespb/frank")

Commit message: FRANK M2U HW Rev 1.00
Other:
- title: Frank M2U -> FRANK M2U
