File: hardware/frank_m1/CMZJ2.kicad_pcb (KiCad board)
At the start: 2 copper layers, 99 x 93.2 mm, 122 parts, among them CON1 Pin Header 1x03, CON2 Pin Header 1x03, CON3 Pin Header 1x08, J1 Pin Header 2x18, Q1 BC850, Q2 BC850, SW1 KLS7-TS3302, U1 NCP1117 3.3

Commit message: FRANK M1 & M2 HW Revisions
Routing:
- net /RS232_CTS: track 35.1 -> 44.7 mm
- net /RS232_RTS: track 33.6 -> 37.6 mm
- net /GPIO18: track 87.8 -> 89.4 mm
- net /GPIO10: track 61.7 -> 60.6 mm
- net /GPIO21: track 45.4 -> 46.5 mm
- net /GPIO15: track 106.8 -> 107.6 mm
- net /GPIO2: track 41.5 -> 42.1 mm
- net /KB_DATA: track 39.2 -> 39.8 mm
- net /GPIO6: track 72.7 -> 73.2 mm
- net /GPIO13: track 51.6 -> 52.1 mm
- net /GPIO26: track 39.9 -> 40.5 mm
- net GND: vias 84 -> 91
