File: hardware/frank_m1/CMZJ2.kicad_sch (KiCad schematic)
At the start: 7 parts, among them CON1 Pin Header 1x03, CON2 Pin Header 1x03, J1 Pin Header 2x18

Commit message: FRANK M1 & M2 HW Revisions
Other:
- title: FRANK -> FRANK M1
Changed lines of the file:
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@@
 	(paper "A4")
 	(title_block
-		(title "FRANK")
+		(title "FRANK M1")
 		(date "2025-02-18")
 		(rev "1.13")
