File: hardware/frank_m1/display.kicad_sch (KiCad schematic)
At the start: 1 part, among them CON3 Pin Header 1x08

Commit message: FRANK M1 & M2 HW Revisions
Other:
- title: FRANK -> FRANK M1
Changed lines of the file:
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@@
 	(paper "A4")
 	(title_block
-		(title "FRANK")
+		(title "FRANK M1")
 		(date "2025-02-18")
 		(rev "1.13")
