File: hardware/frank_m1/ps2.kicad_sch (KiCad schematic)
At the start: 14 parts

Commit message: FRANK M1 & M2 HW Revisions
Other:
- title: FRANK -> FRANK M1
Changed lines of the file:
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@@
 	(paper "A4")
 	(title_block
-		(title "FRANK")
+		(title "FRANK M1")
 		(date "2025-02-18")
 		(rev "1.13")

Commit message: HW Rev 1.14
Changed lines of the file:
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@@
 (kicad_sch
-	(version 20231120)
+	(version 20250114)
 	(generator "eeschema")
-	(generator_version "8.0")
+	(generator_version "9.0")
 	(paper "A4")
 	(title_block
 		(title "FRANK M1")
-		(date "2025-02-18")
-		(rev "1.13")
+		(date "2025-03-03")
+		(rev "1.14")
 		(company "Mikhail Matveev")
 		(comment 1 "https://github.com/xtremespb/frank")
@@
 		(shape input)
 		(at 62.23 144.78 270)
-		(fields_autoplaced yes)
 		(effects
 			(font
@@
 		(shape input)
 		(at 63.5 111.76 90)
-		(fields_autoplaced yes)
 		(effects
 			(font
@@
 		(shape input)
 		(at 74.93 45.72 180)
-		(fields_autoplaced yes)
 		(effects
 			(font
@@
 		(shape input)
 		(at 107.95 52.07 0)
-		(fields_autoplaced yes)
 		(effects
 			(font
@@
 		(shape input)
 		(at 57.15 144.78 270)
-		(fields_autoplaced yes)
 		(effects
 			(font
@@
 		(shape input)
 		(at 55.88 111.76 90)
-		(fields_autoplaced yes)
 		(effects
 			(font
@@
 		(shape input)
 		(at 107.95 46.99 0)
-		(fields_autoplaced yes)
 		(effects
 			(font
@@
 		(shape input)
 		(at 74.93 53.34 180)
-		(fields_autoplaced yes)
 		(effects
 			(font
@@
 			)
 		)
-		(property "Description" ""
+		(property "Description" "6-pin Mini-DIN connector"
 			(at 45.72 49.53 0)
 			(effects
