File: hardware/frank_m1/psram.kicad_sch (KiCad schematic)
At the start: 3 parts

Commit message: Work-in-progress
Parts:
- PSR1: footprint FRANK:SOIC-8 -> FRANK:SO-8
Changed lines of the file:
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@@
 			)
 		)
-		(property "Footprint" "FRANK:SOIC-8"
+		(property "Footprint" "FRANK:SO-8"
 			(at 69.85 73.66 0)
 			(effects

Commit message: FRANK M1 HW Rev 1.00
Parts:
- JP1: AliExpress https://www.aliexpress.com/item/1005006454399822.html -> (none)
Other:
- title: MiniFRANK -> FRANK M1
Changed lines of the file:
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@@
 	(paper "A4")
 	(title_block
-		(title "MiniFRANK")
-		(date "2025-01-14")
-		(rev "2.0")
+		(title "FRANK M1")
+		(date "2025-02-04")
+		(rev "1.00")
 		(company "Mikhail Matveev")
 		(comment 1 "https://github.com/xtremespb/frank")
@@
 			)
 		)
-		(property "Datasheet" "https://cdn-shop.adafruit.com/product-files/4677/4677_esp-psram64_esp-psram64h_datasheet_en.pdf"
+		(property "Datasheet" ""
 			(at 96.52 67.31 0)
 			(effects
@@
 			)
 		)
-		(property "AliExpress" "https://www.aliexpress.com/item/1005006454399822.html"
+		(property "AliExpress" ""
 			(at 96.52 67.31 0)
 			(effects

Commit message: Names changed
Parts:
- JP1: value Jumper PSRAM (2.54) -> Jumper (Solder); AliExpress (none) -> https://www.aliexpress.com/item/1005006454399822.html
- PSR1: footprint FRANK:SO-8 -> FRANK:SOIC-8
- renumbered C39 to C6
Other:
- note added: "As PSRAM is optional, you need to solder the jumper if you are going to use it."
- note removed: "As PSRAM is optional, you need to solder JP1 if you are going to use it."
- title: FRANK M1 -> FRANK
Changed lines of the file:
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@@
 	(paper "A4")
 	(title_block
-		(title "FRANK M1")
-		(date "2025-02-04")
-		(rev "1.00")
+		(title "FRANK")
+		(date "2025-02-18")
+		(rev "1.13")
 		(company "Mikhail Matveev")
 		(comment 1 "https://github.com/xtremespb/frank")
@@
 		)
 	)
-	(text "As PSRAM is optional, you need to solder JP1\nif you are going to use it."
+	(text "As PSRAM is optional, you need to solder the jumper\nif you are going to use it."
 		(exclude_from_sim no)
 		(at 44.196 24.892 0)
@@
 		(on_board yes)
 		(dnp no)
-		(property "Reference" "#PWR060"
+		(property "Reference" "#PWR043"
 			(at 67.31 77.47 0)
 			(effects
@@
 		(instances
 			(project "frank2"
-				(path "/8c0b3d8b-46d3-4173-ab1e-a61765f77d61/d087f9c7-614e-4819-a9d1-c2f8eb5efb4e"
-					(reference "#PWR060")
+				(path "/8c0b3d8b-46d3-4173-ab1e-a61765f77d61/c6465a8b-a48e-459c-b6f3-7a504929a2d8"
+					(reference "#PWR043")
 					(unit 1)
 				)
@@
 		(dnp no)
 		(fields_autoplaced yes)
-		(property "Reference" "#PWR058"
+		(property "Reference" "#PWR041"
 			(at 77.47 49.53 0)
 			(effects
@@
 		(instances
 			(project ""
-				(path "/8c0b3d8b-46d3-4173-ab1e-a61765f77d61/d087f9c7-614e-4819-a9d1-c2f8eb5efb4e"
-					(reference "#PWR058")
+				(path "/8c0b3d8b-46d3-4173-ab1e-a61765f77d61/c6465a8b-a48e-459c-b6f3-7a504929a2d8"
+					(reference "#PWR041")
 					(unit 1)
 				)
@@
 			)
 		)
-		(property "Footprint" "FRANK:SO-8"
+		(property "Footprint" "FRANK:SOIC-8"
 			(at 69.85 73.66 0)
 			(effects
@@
 		(instances
 			(project "frank2"
-				(path "/8c0b3d8b-46d3-4173-ab1e-a61765f77d61/d087f9c7-614e-4819-a9d1-c2f8eb5efb4e"
+				(path "/8c0b3d8b-46d3-4173-ab1e-a61765f77d61/c6465a8b-a48e-459c-b6f3-7a504929a2d8"
 					(reference "PSR1")
 					(unit 1)
@@
 		(on_board yes)
 		(dnp no)
-		(property "Reference" "C39"
+		(property "Reference" "C6"
 			(at 49.911 52.1716 0)
 			(effects
@@
 			)
 		)
-		(property "Datasheet" "https://eu.mouser.com/datasheet/2/447/KEM_C1075_X7R_HT_SMD-3316221.pdf"
+		(property "Datasheet" "https://eu.mouser.com/datasheet/2/40/KGM_X7R-3223212.pdf"
 			(at 46.99 53.34 0)
 			(effects
@@
 		(instances
 			(project "frank2"
-				(path "/8c0b3d8b-46d3-4173-ab1e-a61765f77d61/d087f9c7-614e-4819-a9d1-c2f8eb5efb4e"
-					(reference "C39")
+				(path "/8c0b3d8b-46d3-4173-ab1e-a61765f77d61/c6465a8b-a48e-459c-b6f3-7a504929a2d8"
+					(reference "C6")
 					(unit 1)
 				)
@@
 			)
 		)
-		(property "Value" "Jumper PSRAM (2.54)"
+		(property "Value" "Jumper (Solder)"
 			(at 97.028 69.85 0)
 			(effects
@@
 			)
 		)
-		(property "Datasheet" ""
+		(property "Datasheet" "https://cdn-shop.adafruit.com/product-files/4677/4677_esp-psram64_esp-psram64h_datasheet_en.pdf"
 			(at 96.52 67.31 0)
 			(effects
@@
 			)
 		)
-		(property "AliExpress" ""
+		(property "AliExpress" "https://www.aliexpress.com/item/1005006454399822.html"
 			(at 96.52 67.31 0)
 			(effects
@@
 		(instances
 			(project "frank2"
-				(path "/8c0b3d8b-46d3-4173-ab1e-a61765f77d61/d087f9c7-614e-4819-a9d1-c2f8eb5efb4e"
+				(path "/8c0b3d8b-46d3-4173-ab1e-a61765f77d61/c6465a8b-a48e-459c-b6f3-7a504929a2d8"
 					(reference "JP1")
 					(unit 1)
@@
 		(on_board yes)
 		(dnp no)
-		(property "Reference" "#PWR059"
+		(property "Reference" "#PWR042"
 			(at 46.99 67.31 0)
 			(effects
@@
 		(instances
 			(project "frank2"
-				(path "/8c0b3d8b-46d3-4173-ab1e-a61765f77d61/d087f9c7-614e-4819-a9d1-c2f8eb5efb4e"
-					(reference "#PWR059")
+				(path "/8c0b3d8b-46d3-4173-ab1e-a61765f77d61/c6465a8b-a48e-459c-b6f3-7a504929a2d8"
+					(reference "#PWR042")
 					(unit 1)
 				)

Commit message: FRANK M1 & M2 HW Revisions
Other:
- title: FRANK -> FRANK M1
Changed lines of the file:
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@@
 	(paper "A4")
 	(title_block
-		(title "FRANK")
+		(title "FRANK M1")
 		(date "2025-02-18")
 		(rev "1.13")

Commit message: HW Rev 1.14
Changed lines of the file:
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@@
 (kicad_sch
-	(version 20231120)
+	(version 20250114)
 	(generator "eeschema")
-	(generator_version "8.0")
+	(generator_version "9.0")
 	(paper "A4")
 	(title_block
 		(title "FRANK M1")
-		(date "2025-02-18")
-		(rev "1.13")
+		(date "2025-03-03")
+		(rev "1.14")
 		(company "Mikhail Matveev")
 		(comment 1 "https://github.com/xtremespb/frank")
-	)
-	(junction
-		(at 67.31 45.72)
-		(diameter 0)
-		(color 0 0 0 0)
-	)
-	(no_connect
-		(at 80.01 55.88)
-	)
-	(no_connect
-		(at 80.01 58.42)
-	)
-	(wire
-		(pts
-			(xy 80.01 50.8) (xy 110.49 50.8)
-		)
-		(stroke
-			(width 0)
-			(type default)
-		)
-	)
-	(wire
-		(pts
-			(xy 91.44 67.31) (xy 91.44 63.5)
-		)
-		(stroke
-			(width 0)
-			(type default)
-		)
-	)
-	(wire
-		(pts
-			(xy 91.44 67.31) (xy 92.71 67.31)
-		)
-		(stroke
-			(width 0)
-			(type default)
-		)
-	)
-	(wire
-		(pts
-			(xy 46.99 45.72) (xy 46.99 49.53)
-		)
-		(stroke
-			(width 0)
-			(type default)
-		)
-	)
-	(wire
-		(pts
-			(xy 80.01 53.34) (xy 110.49 53.34)
-		)
-		(stroke
-			(width 0)
-			(type default)
-		)
-	)
-	(wire
-		(pts
-			(xy 46.99 45.72) (xy 67.31 45.72)
-		)
-		(stroke
-			(width 0)
-			(type default)
-		)
-	)
-	(wire
-		(pts
-			(xy 67.31 45.72) (xy 77.47 45.72)
-		)
-		(stroke
-			(width 0)
-			(type default)
-		)
-	)
-	(wire
-		(pts
-			(xy 46.99 57.15) (xy 46.99 60.96)
-		)
-		(stroke
-			(width 0)
-			(type default)
-		)
-	)
-	(wire
-		(pts
-			(xy 80.01 60.96) (xy 110.49 60.96)
-		)
-		(stroke
-			(width 0)
-			(type default)
-		)
-	)
-	(wire
-		(pts
-			(xy 102.87 67.31) (xy 102.87 63.5)
-		)
-		(stroke
-			(width 0)
-			(type default)
-		)
-	)
-	(wire
-		(pts
-			(xy 102.87 63.5) (xy 110.49 63.5)
-		)
-		(stroke
-			(width 0)
-			(type default)
-		)
-	)
-	(wire
-		(pts
-			(xy 100.33 67.31) (xy 102.87 67.31)
-		)
-		(stroke
-			(width 0)
-			(type default)
-		)
-	)
-	(wire
-		(pts
-			(xy 91.44 63.5) (xy 80.01 63.5)
-		)
-		(stroke
-			(width 0)
-			(type default)
-		)
 	)
 	(text "As PSRAM is optional, you need to solder the jumper\nif you are going to use it."
@@
 		)
 	)
+	(junction
+		(at 67.31 45.72)
+		(diameter 0)
+		(color 0 0 0 0)
+	)
+	(no_connect
+		(at 80.01 55.88)
+	)
+	(no_connect
+		(at 80.01 58.42)
+	)
+	(wire
+		(pts
+			(xy 80.01 50.8) (xy 110.49 50.8)
+		)
+		(stroke
+			(width 0)
+			(type default)
+		)
+	)
+	(wire
+		(pts
+			(xy 91.44 67.31) (xy 91.44 63.5)
+		)
+		(stroke
+			(width 0)
+			(type default)
+		)
+	)
+	(wire
+		(pts
+			(xy 91.44 67.31) (xy 92.71 67.31)
+		)
+		(stroke
+			(width 0)
+			(type default)
+		)
+	)
+	(wire
+		(pts
+			(xy 46.99 45.72) (xy 46.99 49.53)
+		)
+		(stroke
+			(width 0)
+			(type default)
+		)
+	)
+	(wire
+		(pts
+			(xy 80.01 53.34) (xy 110.49 53.34)
+		)
+		(stroke
+			(width 0)
+			(type default)
+		)
+	)
+	(wire
+		(pts
+			(xy 46.99 45.72) (xy 67.31 45.72)
+		)
+		(stroke
+			(width 0)
+			(type default)
+		)
+	)
+	(wire
+		(pts
+			(xy 67.31 45.72) (xy 77.47 45.72)
+		)
+		(stroke
+			(width 0)
+			(type default)
+		)
+	)
+	(wire
+		(pts
+			(xy 46.99 57.15) (xy 46.99 60.96)
+		)
+		(stroke
+			(width 0)
+			(type default)
+		)
+	)
+	(wire
+		(pts
+			(xy 80.01 60.96) (xy 110.49 60.96)
+		)
+		(stroke
+			(width 0)
+			(type default)
+		)
+	)
+	(wire
+		(pts
+			(xy 102.87 67.31) (xy 102.87 63.5)
+		)
+		(stroke
+			(width 0)
+			(type default)
+		)
+	)
+	(wire
+		(pts
+			(xy 102.87 63.5) (xy 110.49 63.5)
+		)
+		(stroke
+			(width 0)
+			(type default)
+		)
+	)
+	(wire
+		(pts
+			(xy 100.33 67.31) (xy 102.87 67.31)
+		)
+		(stroke
+			(width 0)
+			(type default)
+		)
+	)
+	(wire
+		(pts
+			(xy 91.44 63.5) (xy 80.01 63.5)
+		)
+		(stroke
+			(width 0)
+			(type default)
+		)
+	)
 	(hierarchical_label "SISIO"
 		(shape input)
 		(at 110.49 60.96 0)
-		(fields_autoplaced yes)
 		(effects
 			(font
@@
 		(shape input)
 		(at 110.49 50.8 0)
-		(fields_autoplaced yes)
 		(effects
 			(font
@@
 		(shape input)
 		(at 110.49 53.34 0)
-		(fields_autoplaced yes)
 		(effects
 			(font
@@
 		(shape input)
 		(at 110.49 63.5 0)
-		(fields_autoplaced yes)
 		(effects
 			(font
@@
 			)
 		)
-		(property "Datasheet" "https://cdn-shop.adafruit.com/product-files/4677/4677_esp-psram64_esp-psram64h_datasheet_en.pdf"
+		(property "Datasheet" "~"
 			(at 96.52 67.31 0)
 			(effects
@@
 			)
 		)
-		(property "Description" ""
+		(property "Description" "Solder Jumper, 2-pole, open"
 			(at 96.52 67.31 0)
 			(effects
