File: hardware/frank_m1/usbstack.kicad_sch (KiCad schematic)
At the start: 7 parts

Commit message: FRANK M1 HW Rev 1.00
Other:
- title: TurboFRANK -> FRANK M1
Changed lines of the file:
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@@
 	(paper "A4")
 	(title_block
-		(title "TurboFRANK")
-		(date "2025-02-02")
-		(rev "1.01")
+		(title "FRANK M1")
+		(date "2025-02-04")
+		(rev "1.00")
 		(company "Mikhail Matveev")
 		(comment 1 "https://github.com/xtremespb/frank")

Commit message: Names changed
Parts:
- renumbered C40 to C14, C41 to C15, R28 to R33, R29 to R34, R30 to R35, R31 to R36
Other:
- title: FRANK M1 -> FRANK
Changed lines of the file:
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@@
 	(paper "A4")
 	(title_block
-		(title "FRANK M1")
-		(date "2025-02-04")
-		(rev "1.00")
+		(title "FRANK")
+		(date "2025-02-18")
+		(rev "1.13")
 		(company "Mikhail Matveev")
 		(comment 1 "https://github.com/xtremespb/frank")
@@
 		(instances
 			(project "usb2ps2"
-				(path "/8c0b3d8b-46d3-4173-ab1e-a61765f77d61/d5538ca7-dbbf-439a-a301-785764ff07ba"
+				(path "/8c0b3d8b-46d3-4173-ab1e-a61765f77d61/b237c830-8b62-42ca-9271-338aede27b72"
 					(reference "USB2")
 					(unit 1)
@@
 		(on_board yes)
 		(dnp no)
-		(property "Reference" "C40"
+		(property "Reference" "C14"
 			(at 84.201 44.5516 0)
 			(effects
@@
 		(instances
 			(project "usb2ps2"
-				(path "/8c0b3d8b-46d3-4173-ab1e-a61765f77d61/d5538ca7-dbbf-439a-a301-785764ff07ba"
-					(reference "C40")
+				(path "/8c0b3d8b-46d3-4173-ab1e-a61765f77d61/b237c830-8b62-42ca-9271-338aede27b72"
+					(reference "C14")
 					(unit 1)
 				)
@@
 		(on_board yes)
 		(dnp no)
-		(property "Reference" "R30"
+		(property "Reference" "R35"
 			(at 61.722 66.04 90)
 			(effects
@@
 		(instances
 			(project "usb2ps2"
-				(path "/8c0b3d8b-46d3-4173-ab1e-a61765f77d61/d5538ca7-dbbf-439a-a301-785764ff07ba"
-					(reference "R30")
+				(path "/8c0b3d8b-46d3-4173-ab1e-a61765f77d61/b237c830-8b62-42ca-9271-338aede27b72"
+					(reference "R35")
 					(unit 1)
 				)
@@
 		(on_board yes)
 		(dnp no)
-		(property "Reference" "C41"
+		(property "Reference" "C15"
 			(at 95.631 44.5516 0)
 			(effects
@@
 		(instances
 			(project "usb2ps2"
-				(path "/8c0b3d8b-46d3-4173-ab1e-a61765f77d61/d5538ca7-dbbf-439a-a301-785764ff07ba"
-					(reference "C41")
+				(path "/8c0b3d8b-46d3-4173-ab1e-a61765f77d61/b237c830-8b62-42ca-9271-338aede27b72"
+					(reference "C15")
 					(unit 1)
 				)
@@
 		(on_board yes)
 		(dnp no)
-		(property "Reference" "#PWR061"
+		(property "Reference" "#PWR067"
 			(at 52.07 40.64 0)
 			(effects
@@
 		(instances
 			(project "usb2ps2"
-				(path "/8c0b3d8b-46d3-4173-ab1e-a61765f77d61/d5538ca7-dbbf-439a-a301-785764ff07ba"
-					(reference "#PWR061")
+				(path "/8c0b3d8b-46d3-4173-ab1e-a61765f77d61/b237c830-8b62-42ca-9271-338aede27b72"
+					(reference "#PWR067")
 					(unit 1)
 				)
@@
 		(on_board yes)
 		(dnp no)
-		(property "Reference" "#PWR063"
+		(property "Reference" "#PWR069"
 			(at 81.28 57.15 0)
 			(effects
@@
 		(instances
 			(project "usb2ps2"
-				(path "/8c0b3d8b-46d3-4173-ab1e-a61765f77d61/d5538ca7-dbbf-439a-a301-785764ff07ba"
-					(reference "#PWR063")
+				(path "/8c0b3d8b-46d3-4173-ab1e-a61765f77d61/b237c830-8b62-42ca-9271-338aede27b72"
+					(reference "#PWR069")
 					(unit 1)
 				)
@@
 		(on_board yes)
 		(dnp no)
-		(property "Reference" "R29"
+		(property "Reference" "R34"
 			(at 70.612 64.77 90)
 			(effects
@@
 		(instances
 			(project "usb2ps2"
-				(path "/8c0b3d8b-46d3-4173-ab1e-a61765f77d61/d5538ca7-dbbf-439a-a301-785764ff07ba"
-					(reference "R29")
+				(path "/8c0b3d8b-46d3-4173-ab1e-a61765f77d61/b237c830-8b62-42ca-9271-338aede27b72"
+					(reference "R34")
 					(unit 1)
 				)
@@
 		(on_board yes)
 		(dnp no)
-		(property "Reference" "#PWR064"
+		(property "Reference" "#PWR070"
 			(at 92.71 57.15 0)
 			(effects
@@
 		(instances
 			(project "usb2ps2"
-				(path "/8c0b3d8b-46d3-4173-ab1e-a61765f77d61/d5538ca7-dbbf-439a-a301-785764ff07ba"
-					(reference "#PWR064")
+				(path "/8c0b3d8b-46d3-4173-ab1e-a61765f77d61/b237c830-8b62-42ca-9271-338aede27b72"
+					(reference "#PWR070")
 					(unit 1)
 				)
@@
 		(on_board yes)
 		(dnp no)
-		(property "Reference" "R28"
+		(property "Reference" "R33"
 			(at 57.912 59.69 90)
 			(effects
@@
 		(instances
 			(project "usb2ps2"
-				(path "/8c0b3d8b-46d3-4173-ab1e-a61765f77d61/d5538ca7-dbbf-439a-a301-785764ff07ba"
-					(reference "R28")
+				(path "/8c0b3d8b-46d3-4173-ab1e-a61765f77d61/b237c830-8b62-42ca-9271-338aede27b72"
+					(reference "R33")
 					(unit 1)
 				)
@@
 		(on_board yes)
 		(dnp no)
-		(property "Reference" "#PWR062"
+		(property "Reference" "#PWR068"
 			(at 58.42 40.64 0)
 			(effects
@@
 		(instances
 			(project "usb2ps2"
-				(path "/8c0b3d8b-46d3-4173-ab1e-a61765f77d61/d5538ca7-dbbf-439a-a301-785764ff07ba"
-					(reference "#PWR062")
+				(path "/8c0b3d8b-46d3-4173-ab1e-a61765f77d61/b237c830-8b62-42ca-9271-338aede27b72"
+					(reference "#PWR068")
 					(unit 1)
 				)
@@
 		(dnp no)
 		(fields_autoplaced yes)
-		(property "Reference" "#PWR065"
+		(property "Reference" "#PWR071"
 			(at 38.1 73.66 0)
 			(effects
@@
 		(instances
 			(project ""
-				(path "/8c0b3d8b-46d3-4173-ab1e-a61765f77d61/d5538ca7-dbbf-439a-a301-785764ff07ba"
-					(reference "#PWR065")
+				(path "/8c0b3d8b-46d3-4173-ab1e-a61765f77d61/b237c830-8b62-42ca-9271-338aede27b72"
+					(reference "#PWR071")
 					(unit 1)
 				)
@@
 		(on_board yes)
 		(dnp no)
-		(property "Reference" "R31"
+		(property "Reference" "R36"
 			(at 74.422 71.12 90)
 			(effects
@@
 		(instances
 			(project "usb2ps2"
-				(path "/8c0b3d8b-46d3-4173-ab1e-a61765f77d61/d5538ca7-dbbf-439a-a301-785764ff07ba"
-					(reference "R31")
+				(path "/8c0b3d8b-46d3-4173-ab1e-a61765f77d61/b237c830-8b62-42ca-9271-338aede27b72"
+					(reference "R36")
 					(unit 1)
 				)

Commit message: FRANK M1 & M2 HW Revisions
Other:
- title: FRANK -> FRANK M1
Changed lines of the file:
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@@
 	(paper "A4")
 	(title_block
-		(title "FRANK")
+		(title "FRANK M1")
 		(date "2025-02-18")
 		(rev "1.13")
