File: hardware/turbofrank/display.kicad_sch (KiCad schematic)
At the start: 1 part, among them CON1 Display

Commit message: HW Rev 1.0
Parts:
- CON3: renamed from CON1; value Display -> Pin Header 1x08; AliExpress (none) -> https://www.aliexpress.com/item/1005007039504981.html
Changed lines of the file:
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@@
 	(title_block
 		(title "TurboFRANK")
-		(date "2025-01-28")
+		(date "2025-01-29")
 		(rev "1.0")
 		(company "Mikhail Matveev")
@@
 		(dnp no)
 		(fields_autoplaced yes)
-		(property "Reference" "#PWR099"
+		(property "Reference" "#PWR0104"
 			(at 60.96 34.29 0)
 			(effects
@@
 			(project "turbofrank"
 				(path "/8c0b3d8b-46d3-4173-ab1e-a61765f77d61/05a34d6b-821f-4841-a010-fe0016ebb2f4"
-					(reference "#PWR099")
+					(reference "#PWR0104")
 					(unit 1)
 				)
@@
 		(dnp no)
 		(fields_autoplaced yes)
-		(property "Reference" "#PWR0100"
+		(property "Reference" "#PWR0105"
 			(at 50.8 36.83 0)
 			(effects
@@
 			(project ""
 				(path "/8c0b3d8b-46d3-4173-ab1e-a61765f77d61/05a34d6b-821f-4841-a010-fe0016ebb2f4"
-					(reference "#PWR0100")
+					(reference "#PWR0105")
 					(unit 1)
 				)
@@
 		(dnp no)
 		(fields_autoplaced yes)
-		(property "Reference" "CON1"
+		(property "Reference" "CON3"
 			(at 29.845 29.21 0)
 			(effects
@@
 			)
 		)
-		(property "Value" "Display"
+		(property "Value" "Pin Header 1x08"
 			(at 29.845 31.75 0)
 			(effects
@@
 		)
 		(property "Description" "Generic connector, single row, 01x08, script generated"
+			(at 29.21 41.91 0)
+			(effects
+				(font
+					(size 1.27 1.27)
+				)
+				(hide yes)
+			)
+		)
+		(property "AliExpress" "https://www.aliexpress.com/item/1005007039504981.html"
 			(at 29.21 41.91 0)
 			(effects
@@
 			(project "turbofrank"
 				(path "/8c0b3d8b-46d3-4173-ab1e-a61765f77d61/05a34d6b-821f-4841-a010-fe0016ebb2f4"
-					(reference "CON1")
+					(reference "CON3")
 					(unit 1)
 				)
