File: hardware/turbofrank/reset.kicad_sch (KiCad schematic)
At the start: 1 part, among them SW3 Reset Button (Pico)

Commit message: HW Rev 1.0
Parts:
- SW3: value Reset Button (Pico) -> KLS7-TS3302; AliExpress https://www.aliexpress.com/item/1005001629293584.html -> https://www.aliexpress.com/item/1005007359248990.html
Changed lines of the file:
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@@
 	(title_block
 		(title "TurboFRANK")
-		(date "2025-01-28")
+		(date "2025-01-29")
 		(rev "1.0")
 		(company "Mikhail Matveev")
@@
 			)
 		)
-		(property "Value" "Reset Button (Pico)"
+		(property "Value" "KLS7-TS3302"
 			(at 62.484 51.562 0)
 			(effects
@@
 			)
 		)
-		(property "AliExpress" "https://www.aliexpress.com/item/1005001629293584.html"
+		(property "AliExpress" "https://www.aliexpress.com/item/1005007359248990.html"
 			(at 48.26 59.69 0)
 			(effects
@@
 		(dnp no)
 		(fields_autoplaced yes)
-		(property "Reference" "#PWR063"
+		(property "Reference" "#PWR068"
 			(at 48.26 41.91 0)
 			(effects
@@
 			(project "frank2"
 				(path "/8c0b3d8b-46d3-4173-ab1e-a61765f77d61/44b0fc63-213a-4da4-a0e4-3ab9f837f02d"
-					(reference "#PWR063")
+					(reference "#PWR068")
 					(unit 1)
 				)
