File: hardware/turbofrank/rs232.kicad_sch (KiCad schematic)
At the start: 10 parts

Commit message: HW Rev 1.0
Parts:
- C33, C34, C35, C36: AliExpress (none) -> https://www.aliexpress.com/item/33008008276.html
- COM1: value RS232 -> D-SUB 9 Male; AliExpress (none) -> https://www.aliexpress.com/item/4001214300548.html
- D10: renamed from D12; AliExpress (none) -> https://www.aliexpress.com/item/1005005707644429.html
- D11: renamed from D13; AliExpress (none) -> https://www.aliexpress.com/item/1005005707644429.html
- MAX1: AliExpress (none) -> https://www.aliexpress.com/item/1005006286473801.html
- R108, R109: AliExpress (none) -> https://www.aliexpress.com/item/1005005945735199.html
Changed lines of the file:
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@@
 	(title_block
 		(title "TurboFRANK")
-		(date "2025-01-28")
+		(date "2025-01-29")
 		(rev "1.0")
 		(company "Mikhail Matveev")
@@
 			)
 		)
+		(property "AliExpress" "https://www.aliexpress.com/item/33008008276.html"
+			(at 59.69 68.58 0)
+			(effects
+				(font
+					(size 1.27 1.27)
+				)
+				(hide yes)
+			)
+		)
 		(pin "1"
 		)
@@
 		(dnp no)
 		(fields_autoplaced yes)
-		(property "Reference" "#PWR0103"
+		(property "Reference" "#PWR0108"
 			(at 99.06 36.83 0)
 			(effects
@@
 			(project ""
 				(path "/8c0b3d8b-46d3-4173-ab1e-a61765f77d61/960439d1-a657-47b6-aee7-897565b7d217"
-					(reference "#PWR0103")
+					(reference "#PWR0108")
 					(unit 1)
 				)
@@
 		(dnp no)
 		(fields_autoplaced yes)
-		(property "Reference" "#PWR0106"
+		(property "Reference" "#PWR0111"
 			(at 116.84 54.61 0)
 			(effects
@@
 			(project ""
 				(path "/8c0b3d8b-46d3-4173-ab1e-a61765f77d61/960439d1-a657-47b6-aee7-897565b7d217"
-					(reference "#PWR0106")
+					(reference "#PWR0111")
 					(unit 1)
 				)
@@
 			)
 		)
+		(property "AliExpress" "https://www.aliexpress.com/item/33008008276.html"
+			(at 48.26 73.66 0)
+			(effects
+				(font
+					(size 1.27 1.27)
+				)
+				(hide yes)
+			)
+		)
 		(pin "1"
 		)
@@
 			)
 		)
+		(property "AliExpress" "https://www.aliexpress.com/item/33008008276.html"
+			(at 106.68 57.15 0)
+			(effects
+				(font
+					(size 1.27 1.27)
+				)
+				(hide yes)
+			)
+		)
 		(pin "1"
 		)
@@
 		(dnp no)
 		(fields_autoplaced yes)
-		(property "Reference" "#PWR0104"
+		(property "Reference" "#PWR0109"
 			(at 146.05 36.83 0)
 			(effects
@@
 			(project "frank2"
 				(path "/8c0b3d8b-46d3-4173-ab1e-a61765f77d61/960439d1-a657-47b6-aee7-897565b7d217"
-					(reference "#PWR0104")
+					(reference "#PWR0109")
 					(unit 1)
 				)
@@
 			)
 		)
+		(property "AliExpress" "https://www.aliexpress.com/item/1005005945735199.html"
+			(at 142.24 41.91 0)
+			(effects
+				(font
+					(size 1.27 1.27)
+				)
+				(hide yes)
+			)
+		)
 		(pin "1"
 		)
@@
 			)
 		)
+		(property "AliExpress" "https://www.aliexpress.com/item/33008008276.html"
+			(at 46.99 83.82 0)
+			(effects
+				(font
+					(size 1.27 1.27)
+				)
+				(hide yes)
+			)
+		)
 		(pin "1"
 		)
@@
 		(dnp no)
 		(fields_autoplaced yes)
-		(property "Reference" "#PWR0105"
+		(property "Reference" "#PWR0110"
 			(at 187.96 53.34 0)
 			(effects
@@
 			(project "frank2"
 				(path "/8c0b3d8b-46d3-4173-ab1e-a61765f77d61/960439d1-a657-47b6-aee7-897565b7d217"
-					(reference "#PWR0105")
+					(reference "#PWR0110")
 					(unit 1)
 				)
@@
 		(dnp no)
 		(fields_autoplaced yes)
-		(property "Reference" "D13"
+		(property "Reference" "D11"
 			(at 132.08 40.64 0)
 			(effects
@@
 			)
 		)
-		(property "Datasheet" "https://assets.nexperia.com/documents/data-sheet/1N4148_1N4448.pdf"
+		(property "Datasheet" "https://www.vishay.com/docs/85748/1n4148w.pdf"
 			(at 132.08 46.99 0)
 			(effects
@@
 		)
 		(property "Sim.Pins" "1=K 2=A"
+			(at 132.08 46.99 0)
+			(effects
+				(font
+					(size 1.27 1.27)
+				)
+				(hide yes)
+			)
+		)
+		(property "AliExpress" "https://www.aliexpress.com/item/1005005707644429.html"
 			(at 132.08 46.99 0)
 			(effects
@@
 			(project "frank2"
 				(path "/8c0b3d8b-46d3-4173-ab1e-a61765f77d61/960439d1-a657-47b6-aee7-897565b7d217"
-					(reference "D13")
+					(reference "D11")
 					(unit 1)
 				)
@@
 				)
 				(justify left top)
+				(hide yes)
+			)
+		)
+		(property "AliExpress" "https://www.aliexpress.com/item/1005006286473801.html"
+			(at 81.28 68.58 0)
+			(effects
+				(font
+					(size 1.27 1.27)
+				)
 				(hide yes)
 			)
@@
 		(dnp no)
 		(fields_autoplaced yes)
-		(property "Reference" "#PWR0108"
+		(property "Reference" "#PWR0113"
 			(at 33.02 83.82 0)
 			(effects
@@
 			(project "frank2"
 				(path "/8c0b3d8b-46d3-4173-ab1e-a61765f77d61/960439d1-a657-47b6-aee7-897565b7d217"
-					(reference "#PWR0108")
+					(reference "#PWR0113")
 					(unit 1)
 				)
@@
 			)
 		)
+		(property "AliExpress" "https://www.aliexpress.com/item/1005005945735199.html"
+			(at 95.25 41.91 0)
+			(effects
+				(font
+					(size 1.27 1.27)
+				)
+				(hide yes)
+			)
+		)
 		(pin "1"
 		)
@@
 		(on_board yes)
 		(dnp no)
-		(property "Reference" "#PWR0107"
+		(property "Reference" "#PWR0112"
 			(at 118.11 71.12 0)
 			(effects
@@
 			(project "frank2"
 				(path "/8c0b3d8b-46d3-4173-ab1e-a61765f77d61/960439d1-a657-47b6-aee7-897565b7d217"
-					(reference "#PWR0107")
+					(reference "#PWR0112")
 					(unit 1)
 				)
@@
 		(dnp no)
 		(fields_autoplaced yes)
-		(property "Reference" "D12"
+		(property "Reference" "D10"
 			(at 85.09 40.64 0)
 			(effects
@@
 			)
 		)
-		(property "Datasheet" "https://assets.nexperia.com/documents/data-sheet/1N4148_1N4448.pdf"
+		(property "Datasheet" "https://www.vishay.com/docs/85748/1n4148w.pdf"
 			(at 85.09 46.99 0)
 			(effects
@@
 		)
 		(property "Sim.Pins" "1=K 2=A"
+			(at 85.09 46.99 0)
+			(effects
+				(font
+					(size 1.27 1.27)
+				)
+				(hide yes)
+			)
+		)
+		(property "AliExpress" "https://www.aliexpress.com/item/1005005707644429.html"
 			(at 85.09 46.99 0)
 			(effects
@@
 			(project "frank2"
 				(path "/8c0b3d8b-46d3-4173-ab1e-a61765f77d61/960439d1-a657-47b6-aee7-897565b7d217"
-					(reference "D12")
+					(reference "D10")
 					(unit 1)
 				)
@@
 			)
 		)
-		(property "Value" "RS232"
+		(property "Value" "D-SUB 9 Male"
 			(at 217.17 48.26 0)
 			(effects
@@
 			)
 		)
-		(property "Datasheet" "~"
+		(property "Datasheet" "https://eu.mouser.com/datasheet/2/578/original-3313093.pdf"
 			(at 219.71 63.5 0)
 			(effects
@@
 			(at 219.71 63.5 0)
 			(effects
+				(font
+					(size 1.27 1.27)
+				)
+				(hide yes)
+			)
+		)
+		(property "AliExpress" "https://www.aliexpress.com/item/4001214300548.html"
+			(at 219.71 63.5 0)
+			(effects

Commit message: HW Rev 1.02
Changed lines of the file:
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@@
 (kicad_sch
-	(version 20231120)
+	(version 20250114)
 	(generator "eeschema")
-	(generator_version "8.0")
+	(generator_version "9.0")
 	(paper "A4")
 	(title_block
 		(title "TurboFRANK")
-		(date "2025-02-02")
-		(rev "1.01")
+		(date "2025-03-03")
+		(rev "1.02")
 		(company "Mikhail Matveev")
 		(comment 1 "https://github.com/xtremespb/frank")
@@
 	(wire
 		(pts
+			(xy 63.5 83.82) (xy 81.28 83.82)
+		)
+		(stroke
+			(width 0)
+			(type default)
+		)
+	)
+	(wire
+		(pts
 			(xy 63.5 86.36) (xy 81.28 86.36)
 		)
@@
 	(wire
 		(pts
+			(xy 194.31 68.58) (xy 212.09 68.58)
+		)
+		(stroke
+			(width 0)
+			(type default)
+		)
+	)
+	(wire
+		(pts
 			(xy 115.57 54.61) (xy 120.65 54.61)
 		)
@@
 	(wire
 		(pts
-			(xy 63.5 83.82) (xy 81.28 83.82)
-		)
-		(stroke
-			(width 0)
-			(type default)
-		)
-	)
-	(wire
-		(pts
 			(xy 63.5 71.12) (xy 77.47 71.12)
 		)
@@
 		(pts
 			(xy 111.76 81.28) (xy 115.57 81.28)
-		)
-		(stroke
-			(width 0)
-			(type default)
-		)
-	)
-	(wire
-		(pts
-			(xy 194.31 68.58) (xy 212.09 68.58)
 		)
 		(stroke
@@
 	(label "CTS_MAX"
 		(at 115.57 86.36 0)
-		(fields_autoplaced yes)
 		(effects
 			(font
@@
 	(label "RX_IN"
 		(at 115.57 73.66 0)
-		(fields_autoplaced yes)
 		(effects
 			(font
@@
 	)
 	(label "CTS_IN"
-		(at 64.77 83.82 0)
-		(fields_autoplaced yes)
+		(at 63.5 83.82 0)
 		(effects
 			(font
@@
 	(label "CTS_MAX"
 		(at 69.85 46.99 0)
-		(fields_autoplaced yes)
 		(effects
 			(font
@@
 	(label "RX_MAX"
 		(at 116.84 46.99 0)
-		(fields_autoplaced yes)
 		(effects
 			(font
@@
 	)
 	(label "TX_IN"
-		(at 195.58 68.58 0)
-		(fields_autoplaced yes)
+		(at 194.31 68.58 0)
 		(effects
 			(font
@@
 	(label "C1-"
 		(at 64.77 73.66 0)
-		(fields_autoplaced yes)
 		(effects
 			(font
@@
 	(label "V-"
 		(at 64.77 81.28 0)
-		(fields_autoplaced yes)
 		(effects
 			(font
@@
 	)
 	(label "RTS_IN"
-		(at 195.58 60.96 0)
-		(fields_autoplaced yes)
+		(at 194.31 60.96 0)
 		(effects
 			(font
@@
 	(label "C2-"
 		(at 64.77 78.74 0)
-		(fields_autoplaced yes)
 		(effects
 			(font
@@
 	(label "RX_MAX"
 		(at 115.57 78.74 0)
-		(fields_autoplaced yes)
 		(effects
 			(font
@@
 	(label "C1+"
 		(at 64.77 68.58 0)
-		(fields_autoplaced yes)
 		(effects
 			(font
@@
 	)
 	(label "RTS_IN"
-		(at 64.77 86.36 0)
-		(fields_autoplaced yes)
+		(at 63.5 86.36 0)
 		(effects
 			(font
@@
 	(label "C2+"
 		(at 64.77 76.2 0)
-		(fields_autoplaced yes)
 		(effects
 			(font
@@
 	)
 	(label "CTS_IN"
-		(at 195.58 66.04 0)
-		(fields_autoplaced yes)
+		(at 194.31 66.04 0)
 		(effects
 			(font
@@
 	(label "TX_IN"
 		(at 115.57 76.2 0)
-		(fields_autoplaced yes)
 		(effects
 			(font
@@
 	)
 	(label "RX_IN"
-		(at 195.58 63.5 0)
-		(fields_autoplaced yes)
+		(at 194.31 63.5 0)
 		(effects
 			(font
@@
 	)
 	(label "V+"
-		(at 64.77 71.12 0)
-		(fields_autoplaced yes)
+		(at 63.5 71.12 0)
 		(effects
 			(font
@@
 		(shape input)
 		(at 149.86 46.99 0)
-		(fields_autoplaced yes)
 		(effects
 			(font
@@
 		(shape input)
 		(at 102.87 46.99 0)
-		(fields_autoplaced yes)
 		(effects
 			(font
@@
 		(shape input)
 		(at 115.57 83.82 0)
-		(fields_autoplaced yes)
 		(effects
 			(font
@@
 		(shape input)
 		(at 115.57 81.28 0)
-		(fields_autoplaced yes)
-		(effects
-			(font
+		(effects
+			(font
