File: hardware/turbofrank/sd.kicad_sch (KiCad schematic)
At the start: 3 parts

Commit message: HW Rev 1.0
Parts:
- SD1: value Micro SD (Short) -> 0475710001
- SD2: value Micro SD (Long) -> 104031-0811; AliExpress (none) -> https://www.aliexpress.com/item/1005004214252441.html
Changed lines of the file:
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@@
 	(title_block
 		(title "TurboFRANK")
-		(date "2025-01-28")
+		(date "2025-01-29")
 		(rev "1.0")
 		(company "Mikhail Matveev")
@@
 			)
 		)
-		(property "Datasheet" "https://eu.mouser.com/datasheet/2/447/KEM_C1075_X7R_HT_SMD-3316221.pdf"
+		(property "Datasheet" "https://eu.mouser.com/datasheet/2/40/KGM_X7R-3223212.pdf"
 			(at 138.43 53.34 0)
 			(effects
@@
 		(dnp no)
 		(fields_autoplaced yes)
-		(property "Reference" "#PWR053"
+		(property "Reference" "#PWR057"
 			(at 128.27 57.15 0)
 			(effects
@@
 			(project "core"
 				(path "/8c0b3d8b-46d3-4173-ab1e-a61765f77d61/2e81912e-397c-4129-8da5-abf37a4f2667"
-					(reference "#PWR053")
+					(reference "#PWR057")
 					(unit 1)
 				)
@@
 		(on_board yes)
 		(dnp no)
-		(property "Reference" "#PWR054"
+		(property "Reference" "#PWR058"
 			(at 148.59 53.34 0)
 			(effects
@@
 			(project "core"
 				(path "/8c0b3d8b-46d3-4173-ab1e-a61765f77d61/2e81912e-397c-4129-8da5-abf37a4f2667"
-					(reference "#PWR054")
+					(reference "#PWR058")
 					(unit 1)
 				)
@@
 		(dnp no)
 		(fields_autoplaced yes)
-		(property "Reference" "#PWR052"
+		(property "Reference" "#PWR056"
 			(at 55.88 53.34 0)
 			(effects
@@
 			(project "core"
 				(path "/8c0b3d8b-46d3-4173-ab1e-a61765f77d61/2e81912e-397c-4129-8da5-abf37a4f2667"
-					(reference "#PWR052")
+					(reference "#PWR056")
 					(unit 1)
 				)
@@
 			)
 		)
-		(property "Value" "Micro SD (Short)"
+		(property "Value" "0475710001"
 			(at 78.74 45.72 0)
 			(effects
@@
 		(dnp no)
 		(fields_autoplaced yes)
-		(property "Reference" "#PWR056"
+		(property "Reference" "#PWR060"
 			(at 101.6 58.42 0)
 			(effects
@@
 			(project "core"
 				(path "/8c0b3d8b-46d3-4173-ab1e-a61765f77d61/2e81912e-397c-4129-8da5-abf37a4f2667"
-					(reference "#PWR056")
+					(reference "#PWR060")
 					(unit 1)
 				)
@@
 		(dnp no)
 		(fields_autoplaced yes)
-		(property "Reference" "#PWR0111"
+		(property "Reference" "#PWR061"
 			(at 132.08 99.06 0)
 			(effects
@@
 			(project "turbofrank"
 				(path "/8c0b3d8b-46d3-4173-ab1e-a61765f77d61/2e81912e-397c-4129-8da5-abf37a4f2667"
-					(reference "#PWR0111")
+					(reference "#PWR061")
 					(unit 1)
 				)
@@
 			)
 		)
-		(property "Value" "Micro SD (Long)"
+		(property "Value" "104031-0811"
 			(at 161.925 77.47 0)
 			(effects
@@
 			)
 		)
-		(property "Datasheet" "http://katalog.we-online.de/em/datasheet/693072010801.pdf"
+		(property "Datasheet" "https://www.we-online.com/components/products/datasheet/693072010801.pdf"
 			(at 161.29 93.98 0)
 			(effects
@@
 			)
 		)
-		(property "Description" ""
+		(property "Description" "Micro SD Card Socket"
+			(at 161.29 93.98 0)
+			(effects
+				(font
+					(size 1.27 1.27)
+				)
+				(hide yes)
+			)
+		)
+		(property "AliExpress" "https://www.aliexpress.com/item/1005004214252441.html"
 			(at 161.29 93.98 0)
 			(effects
@@
 		(dnp no)
 		(fields_autoplaced yes)
-		(property "Reference" "#PWR055"
+		(property "Reference" "#PWR059"
 			(at 55.88 55.88 0)
 			(effects
@@
 			(project "core"
 				(path "/8c0b3d8b-46d3-4173-ab1e-a61765f77d61/2e81912e-397c-4129-8da5-abf37a4f2667"
-					(reference "#PWR055")
+					(reference "#PWR059")
 					(unit 1)
 				)
@@
 		(dnp no)
 		(fields_autoplaced yes)
-		(property "Reference" "#PWR051"
+		(property "Reference" "#PWR055"
 			(at 55.88 50.8 0)
 			(effects
@@
 			(project ""
 				(path "/8c0b3d8b-46d3-4173-ab1e-a61765f77d61/2e81912e-397c-4129-8da5-abf37a4f2667"
-					(reference "#PWR051")
+					(reference "#PWR055")
 					(unit 1)
 				)
