File: hardware/turbofrank/turbosound.kicad_sch (KiCad schematic)
At the start: 78 parts, among them Q1 BC850, SW1 Reset Button (Yamaha), SW2 Reset Button (Yamaha), U1 LM358, U2 YM2149, U3 YM2149, U4 74HC595, U5 74HC595, U6 74HC74, X1 3.58 MHz

Commit message: HW Rev 1.0
Parts:
- C1, C11, C12, C2, C8, C9: AliExpress (none) -> https://www.aliexpress.com/item/1005006870280809.html
- C10, C14, C15, C3, C4, C5, C6, C7: AliExpress (none) -> https://www.aliexpress.com/item/33008008276.html
- C13: value 0.1 -> 100n; AliExpress (none) -> https://www.aliexpress.com/item/33008008276.html
- D1: renamed from D2; value 1N4148W -> 1N4148; AliExpress (none) -> https://www.aliexpress.com/item/1005005707644429.html
- D2: renamed from D4; value 1N4148W -> 1N4148; AliExpress (none) -> https://www.aliexpress.com/item/1005005707644429.html
- L1: renamed from D1; value LED -> Orange; AliExpress (none) -> https://www.aliexpress.com/item/1005005975741298.html
- L2: renamed from D3; value LED -> Orange; AliExpress (none) -> https://www.aliexpress.com/item/1005005975741298.html
- Q1: AliExpress (none) -> https://www.aliexpress.com/item/1005005008637286.html
- R1, R10, R11, R12, R13, R14, R15, R16, R17, R18, R19, R2, R20, R21, R22, R23, R24, R25, R26, R27, R28, R29, R3, R30, R31, R32, R33, R34, R35, R36, R37, R38, R39, R4, R40, R41, R42, R43, R44, R45, R46, R47, R48, R49, R5, R6, R7, R8, R9: AliExpress (none) -> https://www.aliexpress.com/item/1005005945735199.html
- SW1, SW2: value Reset Button (Yamaha) -> KLS7-TS3302; AliExpress (none) -> https://www.aliexpress.com/item/1005007359248990.html
- U1: AliExpress (none) -> https://www.aliexpress.com/item/32533323519.html
- U2, U3: value YM2149 -> JFC95101; AliExpress (none) -> https://www.aliexpress.com/item/1005004784221287.html
- U4, U5: AliExpress (none) -> https://www.aliexpress.com/item/1005005723889972.html
- U6: AliExpress (none) -> https://www.aliexpress.com/item/1005006778848967.html
- X1: AliExpress (none) -> https://www.aliexpress.com/item/1005006783317100.html

Commit message: HW Rev 1.02
Parts:
- Q1: symbol PCM_Transistor_BJT_AKL:BC850 -> FRANK:PCM_Transistor_BJT_AKL_BC850
- X1: symbol PCM_Crystal_AKL:Crystal_Generic -> FRANK:Crystal_Generic
