File: hardware/minifrank_rm1/minifrank.kicad_pcb (KiCad board)
At the start: 2 copper layers, 66.5 x 48.3 mm, 94 parts, among them Q1 BC850, Q2 BC850, SW1 Flash Button, SW2 Reset Button, U1 NCP1117 3.3, Y1 12 MHz

Commit message: RM1 HW 2.01
Other:
- board text added: "HW RM1 2.01"
- board text added: "RST"
- board text added: "rh1.tech"
- board text removed: "HW REV 2.0"
- board text removed: "RESET"
- board text removed: "RH1.DEV"
