File: hardware/minifrank_rm1u/crystal_12mhz.kicad_sch (KiCad schematic)
At the start: 4 parts, among them Y1 12 MHz

Commit message: MiniFRANK updates
Other:
- title: FRANK M1 -> MiniFRANK RM1U
Changed lines of the file:
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@@
 (kicad_sch
-	(version 20231120)
+	(version 20250114)
 	(generator "eeschema")
-	(generator_version "8.0")
+	(generator_version "9.0")
 	(paper "A4")
 	(title_block
-		(title "FRANK M1")
-		(date "2025-02-04")
-		(rev "1.00")
+		(title "MiniFRANK RM1U")
+		(date "2025-03-04")
+		(rev "1.01")
 		(company "Mikhail Matveev")
 		(comment 1 "https://github.com/xtremespb/frank")
@@
 		(shape input)
 		(at 44.45 49.53 180)
-		(fields_autoplaced yes)
 		(effects
 			(font
@@
 		(shape input)
 		(at 44.45 39.37 180)
-		(fields_autoplaced yes)
 		(effects
 			(font
