File: hardware/minifrank_rm1u/frank_m1.kicad_pcb (KiCad board)
At the start: 2 copper layers, 81.4 x 58.4 mm, 121 parts, among them J1 Main Jumpers, J2 USB DP Jumper, J3 USB DM Jumper, J4 Gamepad, J5 Gamepad, J6 RP2 Reset, J7 UART, J8 +3.3V, Q1 BC850, Q2 BC850, SW1 KLS7-TS3302, SW2 KLS7-TS3302, SW3 KLS7-TS3302, U1 RP2040, U2 NCP1117 3.3, U3 RP2040, U4 TDA1387T, Y1 12 MHz

Commit message: MiniFRANK updates
Other:
- board text added: "HW RM1U 1.01"
- board text added: "KEYBOARD/MOUSE"
- board text added: "RST"
- board text added: "rh1.tech"
- board text removed: "KEYBOARD + MOUSE"
- board text removed: "M1P1 / REV 1.00"
- board text removed: "RESET"
- board text removed: "RH1.DEV"
