File: hardware/minifrank_rm1u/frank_m1.kicad_sch (KiCad schematic)
At the start: 10 parts, among them J1 Main Jumpers, J2 USB DP Jumper, J3 USB DM Jumper, J6 RP2 Reset, J7 UART, J8 +3.3V

Commit message: MiniFRANK updates
Other:
- title: FRANK M1 -> MiniFRANK RM1U
