File: hardware/minifrank_rm1u/gamepad.kicad_sch (KiCad schematic)
At the start: 4 parts, among them J5 Gamepad

Commit message: MiniFRANK updates
Parts:
- renumbered C36 to C16, D2 to D1, J5 to J4, R19 to R8
Other:
- title: FRANK M1 -> MiniFRANK RM1U
Changed lines of the file:
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@@
 (kicad_sch
-	(version 20231120)
+	(version 20250114)
 	(generator "eeschema")
-	(generator_version "8.0")
+	(generator_version "9.0")
 	(paper "A4")
 	(title_block
-		(title "FRANK M1")
-		(date "2025-02-04")
-		(rev "1.00")
+		(title "MiniFRANK RM1U")
+		(date "2025-03-04")
+		(rev "1.01")
 		(company "Mikhail Matveev")
 		(comment 1 "https://github.com/xtremespb/frank")
@@
 	(label "GND"
 		(at 68.58 40.64 0)
-		(fields_autoplaced yes)
 		(effects
 			(font
@@
 	(label "+5V"
 		(at 68.58 50.8 0)
-		(fields_autoplaced yes)
 		(effects
 			(font
@@
 	(label "J1_DATA"
 		(at 68.58 48.26 0)
-		(fields_autoplaced yes)
 		(effects
 			(font
@@
 		(shape input)
 		(at 68.58 38.1 180)
-		(fields_autoplaced yes)
 		(effects
 			(font
@@
 		(shape input)
 		(at 40.64 48.26 180)
-		(fields_autoplaced yes)
 		(effects
 			(font
@@
 		(shape input)
 		(at 68.58 43.18 180)
-		(fields_autoplaced yes)
 		(effects
 			(font
@@
 		(on_board yes)
 		(dnp no)
-		(property "Reference" "C36"
+		(property "Reference" "C16"
 			(at 58.801 53.4416 0)
 			(effects
@@
 		(on_board yes)
 		(dnp no)
-		(property "Reference" "R19"
+		(property "Reference" "R8"
 			(at 50.8 45.72 90)
 			(effects
@@
 		(dnp no)
 		(fields_autoplaced yes)
-		(property "Reference" "#PWR045"
+		(property "Reference" "#PWR024"
 			(at 48.26 64.77 0)
 			(effects
@@
 		(on_board yes)
 		(dnp no)
-		(property "Reference" "D2"
+		(property "Reference" "D1"
 			(at 45.72 53.34 0)
 			(effects
@@
 		(dnp no)
 		(fields_autoplaced yes)
-		(property "Reference" "#PWR046"
+		(property "Reference" "#PWR025"
 			(at 55.88 64.77 0)
 			(effects
@@
 		(on_board yes)
 		(dnp no)
-		(property "Reference" "J5"
+		(property "Reference" "J4"
 			(at 88.9 30.48 0)
 			(effects
