File: hardware/minifrank_rm2/audio_out_m1.kicad_sch (KiCad schematic)
At the start: 14 parts, among them U2 TDA1387T

Commit message: MiniFRANK RM2 HW 1.03
Other:
- title: Frank M2 -> Frank RM2
Changed lines of the file:
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@@
 	(paper "A4")
 	(title_block
-		(title "Frank M2")
-		(date "2025-02-02")
-		(rev "1.02")
+		(title "Frank RM2")
+		(date "2025-02-23")
+		(rev "1.03")
 		(company "Mikhail Matveev")
 		(comment 1 "https://github.com/xtremespb/frank")

Commit message: MiniFRANK updates
Other:
- title: Frank RM2 -> MiniFRANK RM2
Changed lines of the file:
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@@
 (kicad_sch
-	(version 20231120)
+	(version 20250114)
 	(generator "eeschema")
-	(generator_version "8.0")
+	(generator_version "9.0")
 	(paper "A4")
 	(title_block
-		(title "Frank RM2")
-		(date "2025-02-23")
-		(rev "1.03")
+		(title "MiniFRANK RM2")
+		(date "2025-03-04")
+		(rev "1.04")
 		(company "Mikhail Matveev")
 		(comment 1 "https://github.com/xtremespb/frank")
@@
 	(label "L"
 		(at 123.19 46.99 0)
-		(fields_autoplaced yes)
 		(effects
 			(font
@@
 	(label "R"
 		(at 123.19 68.58 0)
-		(fields_autoplaced yes)
 		(effects
 			(font
@@
 	(label "L*"
 		(at 115.57 60.96 0)
-		(fields_autoplaced yes)
 		(effects
 			(font
@@
 	(label "R*"
 		(at 115.57 66.04 0)
-		(fields_autoplaced yes)
 		(effects
 			(font
@@
 		(shape input)
 		(at 170.18 46.99 0)
-		(fields_autoplaced yes)
 		(effects
 			(font
@@
 		(shape input)
 		(at 170.18 60.96 0)
-		(fields_autoplaced yes)
 		(effects
 			(font
@@
 		(shape input)
 		(at 167.64 111.76 0)
-		(fields_autoplaced yes)
 		(effects
 			(font
@@
 		(shape input)
 		(at 102.87 106.68 180)
-		(fields_autoplaced yes)
 		(effects
 			(font
@@
 		(shape input)
 		(at 167.64 106.68 0)
-		(fields_autoplaced yes)
 		(effects
 			(font
@@
 		(shape input)
 		(at 102.87 109.22 180)
-		(fields_autoplaced yes)
 		(effects
 			(font
@@
 		(shape input)
 		(at 170.18 68.58 0)
-		(fields_autoplaced yes)
 		(effects
 			(font
@@
 		(shape input)
 		(at 102.87 111.76 180)
-		(fields_autoplaced yes)
-		(effects
-			(font
+		(effects
+			(font
