File: hardware/minifrank_rm2/rp2350a.kicad_sch (KiCad schematic)
At the start: 31 parts, among them SW2 SW_Push, U3 ESP-PSRAM32, U4 RP2350_60QFN, U5 W25Q128JVS, Y1 ABM8-272-T3

Commit message: MiniFRANK RM2 HW 1.03
Other:
- title: Frank M2 -> Frank RM2
Changed lines of the file:
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@@
 	(paper "A4")
 	(title_block
-		(title "Frank M2")
-		(date "2025-02-02")
-		(rev "1.02")
+		(title "Frank RM2")
+		(date "2025-02-23")
+		(rev "1.03")
 		(company "Mikhail Matveev")
 		(comment 1 "https://github.com/xtremespb/frank")

Commit message: MiniFRANK updates
Other:
- title: Frank RM2 -> MiniFRANK RM2
Changed lines of the file:
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@@
 (kicad_sch
-	(version 20231120)
+	(version 20250114)
 	(generator "eeschema")
-	(generator_version "8.0")
+	(generator_version "9.0")
 	(paper "A4")
 	(title_block
-		(title "Frank RM2")
-		(date "2025-02-23")
-		(rev "1.03")
+		(title "MiniFRANK RM2")
+		(date "2025-03-04")
+		(rev "1.04")
 		(company "Mikhail Matveev")
 		(comment 1 "https://github.com/xtremespb/frank")
 	)
+	(circle
+		(center 118.11 65.405)
+		(radius 0.635)
+		(stroke
+			(width 0)
+			(type default)
+			(color 132 0 0 1)
+		)
+		(fill
+			(type color)
+			(color 132 0 0 1)
+		)
+	)
+	(text "Make sure these are close to RP2350\n"
+		(exclude_from_sim no)
+		(at 237.49 59.69 0)
+		(effects
+			(font
+				(size 1.27 1.27)
+			)
+			(justify left bottom)
+		)
+	)
 	(junction
 		(at 92.71 54.61)
@@
 		)
 	)
-	(circle
-		(center 118.11 65.405)
-		(radius 0.635)
-		(stroke
-			(width 0)
-			(type default)
-			(color 132 0 0 1)
-		)
-		(fill
-			(type color)
-			(color 132 0 0 1)
-		)
-	)
-	(text "Make sure these are close to RP2350\n"
-		(exclude_from_sim no)
-		(at 237.49 59.69 0)
-		(effects
-			(font
-				(size 1.27 1.27)
-			)
-			(justify left bottom)
-		)
-	)
 	(label "QSPI_SD2"
 		(at 137.16 91.44 0)
-		(fields_autoplaced yes)
 		(effects
 			(font
@@
 	(label "VREG_AVDD"
 		(at 139.065 49.53 0)
-		(fields_autoplaced yes)
 		(effects
 			(font
@@
 	(label "XOUT"
 		(at 137.16 111.76 0)
-		(fields_autoplaced yes)
 		(effects
 			(font
@@
 	(label "XIN"
 		(at 76.2 176.53 180)
-		(fields_autoplaced yes)
 		(effects
 			(font
@@
 	(label "QSPI_SS"
 		(at 16.51 148.59 0)
-		(fields_autoplaced yes)
 		(effects
 			(font
@@
 	(label "QSPI_SD3"
 		(at 137.16 93.98 0)
-		(fields_autoplaced yes)
 		(effects
 			(font
@@
 	(label "QSPI_SD2"
 		(at 95.25 153.67 180)
-		(fields_autoplaced yes)
 		(effects
 			(font
@@
 	(label "QSPI_SS"
 		(at 137.795 82.55 0)
-		(fields_autoplaced yes)
 		(effects
 			(font
@@
 	(label "QSPI_SD0"
 		(at 74.93 100.33 0)
-		(fields_autoplaced yes)
 		(effects
 			(font
@@
 	(label "QSPI_SD3"
 		(at 74.93 95.25 0)
-		(fields_autoplaced yes)
 		(effects
 			(font
@@
 	(label "~{USB_BOOT}"
 		(at 111.76 82.55 0)
-		(fields_autoplaced yes)
 		(effects
 			(font
@@
 	(label "QSPI_SCLK"
 		(at 38.1 153.67 0)
-		(fields_autoplaced yes)
 		(effects
 			(font
@@
 	(label "QSPI_SD1"
 		(at 95.25 148.59 180)
-		(fields_autoplaced yes)
 		(effects
 			(font
@@
 	(label "QSPI_SD2"
 		(at 74.93 97.79 0)
-		(fields_autoplaced yes)
 		(effects
 			(font
@@
 	(label "XIN"
 		(at 137.16 106.68 0)
-		(fields_autoplaced yes)
 		(effects
 			(font
@@
 	(label "GPIO25"
 		(at 229.87 134.62 180)
-		(fields_autoplaced yes)
 		(effects
 			(font
@@
 	(label "QSPI_SD0"
 		(at 95.25 146.05 180)
-		(fields_autoplaced yes)
 		(effects
 			(font
@@
 	(label "GPIO8"
 		(at 74.93 90.17 0)
-		(fields_autoplaced yes)
 		(effects
 			(font
@@
 	(label "QSPI_SCLK"
 		(at 137.16 97.79 0)
-		(fields_autoplaced yes)
 		(effects
 			(font
@@
 	(label "QSPI_SD1"
 		(at 74.93 102.87 0)
-		(fields_autoplaced yes)
 		(effects
 			(font
@@
 	(label "XOUT"
 		(at 76.2 186.69 180)
-		(fields_autoplaced yes)
 		(effects
 			(font
@@
 	(label "QSPI_SD3"
 		(at 95.25 156.21 180)
-		(fields_autoplaced yes)
 		(effects
 			(font
@@
 	(label "QSPI_SD0"
 		(at 137.16 86.36 0)
-		(fields_autoplaced yes)
 		(effects
 			(font
@@
 	(label "FLASH_SS"
 		(at 38.735 148.59 0)
-		(fields_autoplaced yes)
 		(effects
 			(font
@@
 	(label "QSPI_SD1"
 		(at 137.16 88.9 0)
-		(fields_autoplaced yes)
 		(effects
 			(font
@@
 	(label "VREG_LX"
 		(at 137.16 72.39 0)
-		(fields_autoplaced yes)
 		(effects
 			(font
@@
 	(label "QSPI_SCLK"
 		(at 74.93 92.71 0)
-		(fields_autoplaced yes)
 		(effects
 			(font
@@
 		(shape input)
 		(at 229.87 139.7 0)
-		(fields_autoplaced yes)
 		(effects
 			(font
@@
 		(shape input)
 		(at 137.16 124.46 180)
-		(fields_autoplaced yes)
 		(effects
 			(font
@@
 		(shape input)
 		(at 229.87 91.44 0)
-		(fields_autoplaced yes)
 		(effects
 			(font
@@
 		(shape input)
 		(at 229.87 83.82 0)
-		(fields_autoplaced yes)
 		(effects
 			(font
@@
 		(shape input)
 		(at 229.87 119.38 0)
-		(fields_autoplaced yes)
 		(effects
 			(font
@@
 		(shape input)
 		(at 247.65 54.61 0)
-		(fields_autoplaced yes)
 		(effects
 			(font
@@
 		(shape input)
 		(at 229.87 88.9 0)
-		(fields_autoplaced yes)
 		(effects
 			(font
@@
 		(shape input)
 		(at 229.87 132.08 0)
-		(fields_autoplaced yes)
 		(effects
 			(font
@@
 		(shape input)
 		(at 229.87 73.66 0)
-		(fields_autoplaced yes)
 		(effects
 			(font
@@
 		(shape input)
 		(at 229.87 101.6 0)
-		(fields_autoplaced yes)
 		(effects
 			(font
@@
 		(shape input)
 		(at 247.65 63.5 0)
-		(fields_autoplaced yes)
 		(effects
 			(font
@@
 		(shape input)
 		(at 229.87 124.46 0)
-		(fields_autoplaced yes)
 		(effects
 			(font
@@
 		(shape input)
 		(at 229.87 106.68 0)
-		(fields_autoplaced yes)
 		(effects
 			(font
@@
 		(shape input)
 		(at 137.16 135.89 180)
-		(fields_autoplaced yes)
 		(effects
 			(font
@@
 		(shape input)
 		(at 229.87 114.3 0)
-		(fields_autoplaced yes)
 		(effects
 			(font
@@
 		(shape input)
 		(at 229.87 93.98 0)
-		(fields_autoplaced yes)
 		(effects
 			(font
@@
 		(shape input)
 		(at 229.87 127 0)
-		(fields_autoplaced yes)
 		(effects
 			(font
@@
 		(shape input)
 		(at 229.87 86.36 0)
-		(fields_autoplaced yes)
 		(effects
 			(font
@@
 		(shape input)
 		(at 229.87 76.2 0)
-		(fields_autoplaced yes)
 		(effects
 			(font
@@
 		(shape input)
 		(at 229.87 71.12 0)
-		(fields_autoplaced yes)
 		(effects
 			(font
@@
 		(shape input)
 		(at 229.87 81.28 0)
-		(fields_autoplaced yes)
 		(effects
 			(font
@@
 		(shape input)
 		(at 229.87 142.24 0)
-		(fields_autoplaced yes)
 		(effects
 			(font
@@
 		(shape input)
 		(at 229.87 147.32 0)
-		(fields_autoplaced yes)
 		(effects
 			(font
@@
 		(shape input)
 		(at 229.87 104.14 0)
-		(fields_autoplaced yes)
 		(effects
 			(font
@@
 		(shape input)
 		(at 229.87 109.22 0)
-		(fields_autoplaced yes)
 		(effects
 			(font
@@
 		(shape input)
 		(at 229.87 99.06 0)
-		(fields_autoplaced yes)
 		(effects
 			(font
@@
 		(shape input)
 		(at 229.87 96.52 0)
-		(fields_autoplaced yes)
 		(effects
 			(font
@@
 		(shape input)
 		(at 229.87 129.54 0)
-		(fields_autoplaced yes)
 		(effects
 			(font
@@
 		(shape input)
 		(at 229.87 121.92 0)
-		(fields_autoplaced yes)
 		(effects
 			(font
@@
 		(shape input)
 		(at 229.87 78.74 0)
-		(fields_autoplaced yes)
 		(effects
 			(font
@@
 		(shape input)
 		(at 137.16 138.43 180)
-		(fields_autoplaced yes)
 		(effects
 			(font
@@
 		(shape input)
 		(at 229.87 144.78 0)
-		(fields_autoplaced yes)
 		(effects
 			(font
@@
 		(shape input)
 		(at 229.87 116.84 0)
-		(fields_autoplaced yes)
 		(effects
 			(font
@@
 		(shape input)
 		(at 229.87 111.76 0)
-		(fields_autoplaced yes)
 		(effects
 			(font
@@
 			)
 		)
-		(property "Datasheet" "https://www.we-online.com/components/products/datasheet/15408085BA400.pdf"
+		(property "Datasheet" "~"
 			(at 139.7 182.88 0)
 			(effects
@@
 			(at 139.7 182.88 0)
 			(effects
+				(font
+					(size 1.27 1.27)
+				)
+				(hide yes)
+			)
+		)
+		(property "Sim.Pins" "1=K 2=A"
+			(at 139.7 182.88 0)
+			(effects
