File: hardware/minifrank_rm2e/hdmi.kicad_sch (KiCad schematic)
At the start: 10 parts

Commit message: Bugfixes
Other:
- title: MiniFRANK RM2 -> MiniFRANK RM2E
Changed lines of the file:
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@@
 	(paper "A4")
 	(title_block
-		(title "MiniFRANK RM2")
-		(date "2025-03-04")
-		(rev "1.04")
+		(title "MiniFRANK RM2E")
+		(date "2025-03-08")
+		(rev "1.00")
 		(company "Mikhail Matveev")
 		(comment 1 "https://github.com/xtremespb/frank")
