File: hardware/usb2ps2/ps2d.kicad_sch (KiCad schematic)
At the start: 10 parts, among them CN3 PS/2 Pins

Commit message: Structural updates
Parts:
- removed CN3: PS/2 Pins, LIBS:Medved_PinHeader_1x04, symbol Connector:Conn_01x04_Pin
- D1, D2, D3, D4: footprint LIBS:Medved_D_0805 -> FRANK:Diode (SOD-323)
- PS1: footprint LIBS:Connector_Mini-DIN_Female_6Pin_2rows -> FRANK:MiniDIN (6 Pin, female)
- R5: renamed from R13; footprint LIBS:Medved_R_0805 -> FRANK:Resistor (0805)
- R6: renamed from R14; footprint LIBS:Medved_R_0805 -> FRANK:Resistor (0805)
- R7: renamed from R15; footprint LIBS:Medved_R_0805 -> FRANK:Resistor (0805)
- R8: renamed from R16; footprint LIBS:Medved_R_0805 -> FRANK:Resistor (0805)
Changed lines of the file:
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@@
 (kicad_sch
-	(version 20231120)
+	(version 20250114)
 	(generator "eeschema")
-	(generator_version "8.0")
+	(generator_version "9.0")
 	(paper "A3")
 	(title_block
 		(title "USB to PS/2 Adapter")
-		(date "2024-12-07")
-		(rev "1.2")
+		(date "2025-03-04")
+		(rev "1.02")
 		(company "Mikhail Matveev")
+		(comment 1 "https://github.com/xtremespb/frank")
 	)
 	(junction
@@
 	(label "KB_DATA"
 		(at 102.87 92.71 0)
-		(fields_autoplaced yes)
 		(effects
 			(font
@@
 	(label "KB_CLK"
 		(at 104.14 87.63 0)
-		(fields_autoplaced yes)
 		(effects
 			(font
@@
 	(label "MS_DATA"
 		(at 74.93 92.71 0)
-		(fields_autoplaced yes)
 		(effects
 			(font
@@
 	(label "MS_CLK"
 		(at 74.93 87.63 0)
-		(fields_autoplaced yes)
 		(effects
 			(font
@@
 	(hierarchical_label "CLK1"
 		(shape input)
-		(at 156.21 82.55 0)
-		(fields_autoplaced yes)
+		(at 115.57 49.53 90)
 		(effects
 			(font
@@
 		)
 	)
-	(hierarchical_label "DATA1"
+	(hierarchical_label "CLK2"
 		(shape input)
-		(at 156.21 85.09 0)
-		(fields_autoplaced yes)
+		(at 67.31 49.53 90)
 		(effects
 			(font
@@
 		)
 	)
-	(hierarchical_label "DATA2"
+	(hierarchical_label "DATA1"
 		(shape input)
-		(at 156.21 90.17 0)
-		(fields_autoplaced yes)
+		(at 121.92 49.53 90)
 		(effects
 			(font
@@
 		)
 	)
-	(hierarchical_label "CLK2"
+	(hierarchical_label "DATA2"
 		(shape input)
-		(at 156.21 87.63 0)
-		(fields_autoplaced yes)
+		(at 60.96 49.53 90)
 		(effects
 			(font
@@
 		)
 	)
-	(hierarchical_label "CLK1"
-		(shape input)
-		(at 115.57 49.53 90)
-		(fields_autoplaced yes)
-		(effects
-			(font
-				(size 1.27 1.27)
-			)
-			(justify left)
-		)
-	)
-	(hierarchical_label "CLK2"
-		(shape input)
-		(at 67.31 49.53 90)
-		(fields_autoplaced yes)
-		(effects
-			(font
-				(size 1.27 1.27)
-			)
-			(justify left)
-		)
-	)
-	(hierarchical_label "DATA1"
-		(shape input)
-		(at 121.92 49.53 90)
-		(fields_autoplaced yes)
-		(effects
-			(font
-				(size 1.27 1.27)
-			)
-			(justify left)
-		)
-	)
-	(hierarchical_label "DATA2"
-		(shape input)
-		(at 60.96 49.53 90)
-		(fields_autoplaced yes)
-		(effects
-			(font
-				(size 1.27 1.27)
-			)
-			(justify left)
-		)
-	)
 	(symbol
 		(lib_id "power:GND")
@@
 		(on_board yes)
 		(dnp no)
-		(property "Reference" "#PWR040"
+		(property "Reference" "#PWR013"
 			(at 106.68 90.17 0)
 			(effects
@@
 			(project "usb2ps2"
 				(path "/8c0b3d8b-46d3-4173-ab1e-a61765f77d61/6c767f01-0461-4c4b-955a-2f0ac89894b4"
-					(reference "#PWR040")
+					(reference "#PWR013")
 					(unit 1)
 				)
@@
 			)
 		)
-		(property "Footprint" "LIBS:Medved_D_0805"
+		(property "Footprint" "FRANK:Diode (SOD-323)"
 			(at 52.07 52.07 90)
 			(effects
@@
 		(dnp no)
 		(fields_autoplaced yes)
-		(property "Reference" "#PWR039"
+		(property "Reference" "#PWR012"
 			(at 143.51 59.69 0)
 			(effects
@@
 			(project "usb2ps2"
 				(path "/8c0b3d8b-46d3-4173-ab1e-a61765f77d61/6c767f01-0461-4c4b-955a-2f0ac89894b4"
-					(reference "#PWR039")
+					(reference "#PWR012")
 					(unit 1)
 				)
@@
 			)
 		)
-		(property "Footprint" "LIBS:Connector_Mini-DIN_Female_6Pin_2rows"
+		(property "Footprint" "FRANK:MiniDIN (6 Pin, female)"
 			(at 92.71 90.17 0)
 			(effects
@@
 		(dnp no)
 		(fields_autoplaced yes)
-		(property "Reference" "#PWR041"
+		(property "Reference" "#PWR014"
 			(at 69.85 95.25 0)
 			(effects
@@
 			(project ""
 				(path "/8c0b3d8b-46d3-4173-ab1e-a61765f77d61/6c767f01-0461-4c4b-955a-2f0ac89894b4"
-					(reference "#PWR041")
+					(reference "#PWR014")
 					(unit 1)
 				)
@@
 			)
 		)
-		(property "Footprint" "LIBS:Medved_D_0805"
+		(property "Footprint" "FRANK:Diode (SOD-323)"
 			(at 52.07 59.69 90)
 			(effects
@@
 		(on_board yes)
 		(dnp no)
-		(property "Reference" "R13"
+		(property "Reference" "R5"
 			(at 60.452 72.39 90)
 			(effects
@@
 			)
 		)
-		(property "Footprint" "LIBS:Medved_R_0805"
+		(property "Footprint" "FRANK:Resistor (0805)"
 			(at 56.642 72.39 90)
 			(effects
@@
 			(project "usb2ps2"
 				(path "/8c0b3d8b-46d3-4173-ab1e-a61765f77d61/6c767f01-0461-4c4b-955a-2f0ac89894b4"
-					(reference "R13")
+					(reference "R5")
 					(unit 1)
 				)
@@
 		(dnp no)
 		(fields_autoplaced yes)
-		(property "Reference" "#PWR036"
+		(property "Reference" "#PWR09"
 			(at 39.37 52.07 0)
 			(effects
@@
 			(project "usb2ps2"
 				(path "/8c0b3d8b-46d3-4173-ab1e-a61765f77d61/6c767f01-0461-4c4b-955a-2f0ac89894b4"
-					(reference "#PWR036")
-					(unit 1)
-				)
-			)
-		)
-	)
-	(symbol
-		(lib_id "Connector:Conn_01x04_Pin")
-		(at 151.13 85.09 0)
-		(unit 1)
-		(exclude_from_sim no)
-		(in_bom yes)
-		(on_board yes)
-		(dnp no)
-		(fields_autoplaced yes)
-		(property "Reference" "CN3"
-			(at 151.765 77.47 0)
-			(effects
-				(font
-					(size 1.27 1.27)
-				)
-			)
-		)
-		(property "Value" "PS/2 Pins"
-			(at 151.765 80.01 0)
-			(effects
-				(font
-					(size 1.27 1.27)
-				)
-			)
-		)
-		(property "Footprint" "LIBS:Medved_PinHeader_1x04"
-			(at 151.13 85.09 0)
-			(effects
-				(font
-					(size 1.27 1.27)
-				)
-				(hide yes)
-			)
-		)
-		(property "Datasheet" "~"
-			(at 151.13 85.09 0)
-			(effects
-				(font
-					(size 1.27 1.27)
-				)
-				(hide yes)
-			)
-		)
-		(property "Description" "Generic connector, single row, 01x04, script generated"
-			(at 151.13 85.09 0)
-			(effects
-				(font
-					(size 1.27 1.27)
-				)
-				(hide yes)
-			)
-		)
-		(pin "3"
-		)
-		(pin "4"
-		)
-		(pin "2"
-		)
-		(pin "1"
-		)
-		(instances
-			(project ""
-				(path "/8c0b3d8b-46d3-4173-ab1e-a61765f77d61/6c767f01-0461-4c4b-955a-2f0ac89894b4"
-					(reference "CN3")
+					(reference "#PWR09")
 					(unit 1)
 				)
@@
 		(on_board yes)
 		(dnp no)
-		(property "Reference" "R16"
+		(property "Reference" "R8"
 			(at 122.428 72.39 90)
 			(effects
@@
 			)
 		)
-		(property "Footprint" "LIBS:Medved_R_0805"
+		(property "Footprint" "FRANK:Resistor (0805)"
 			(at 126.238 72.39 90)
 			(effects
@@
 			(project "usb2ps2"
 				(path "/8c0b3d8b-46d3-4173-ab1e-a61765f77d61/6c767f01-0461-4c4b-955a-2f0ac89894b4"
-					(reference "R16")
+					(reference "R8")
 					(unit 1)
 				)
@@
 		(dnp no)
 		(fields_autoplaced yes)
-		(property "Reference" "#PWR037"
+		(property "Reference" "#PWR010"
 			(at 143.51 52.07 0)
 			(effects
@@
 			(project "usb2ps2"
 				(path "/8c0b3d8b-46d3-4173-ab1e-a61765f77d61/6c767f01-0461-4c4b-955a-2f0ac89894b4"
-					(reference "#PWR037")
+					(reference "#PWR010")
 					(unit 1)
 				)
@@
 		(dnp no)
 		(fields_autoplaced yes)
-		(property "Reference" "#PWR038"
+		(property "Reference" "#PWR011"
 			(at 39.37 59.69 0)
 			(effects
@@
 			(project "usb2ps2"
 				(path "/8c0b3d8b-46d3-4173-ab1e-a61765f77d61/6c767f01-0461-4c4b-955a-2f0ac89894b4"
-					(reference "#PWR038")
+					(reference "#PWR011")
 					(unit 1)
 				)
@@
 		(on_board yes)
 		(dnp no)
-		(property "Reference" "R14"
+		(property "Reference" "R6"
 			(at 69.596 72.136 90)
 			(effects
@@
 			)
 		)
-		(property "Footprint" "LIBS:Medved_R_0805"
+		(property "Footprint" "FRANK:Resistor (0805)"
 			(at 65.532 72.39 90)
 			(effects
@@
 			(project "usb2ps2"
 				(path "/8c0b3d8b-46d3-4173-ab1e-a61765f77d61/6c767f01-0461-4c4b-955a-2f0ac89894b4"
-					(reference "R14")
+					(reference "R6")
 					(unit 1)
 				)
@@
 			)
 		)
-		(property "Footprint" "LIBS:Medved_D_0805"
+		(property "Footprint" "FRANK:Diode (SOD-323)"
 			(at 130.81 59.69 90)
 			(effects
@@
 		(on_board yes)
 		(dnp no)
-		(property "Reference" "R15"
+		(property "Reference" "R7"
 			(at 113.284 72.136 90)
 			(effects
@@
 			)
 		)
-		(property "Footprint" "LIBS:Medved_R_0805"
+		(property "Footprint" "FRANK:Resistor (0805)"
 			(at 117.348 72.39 90)
 			(effects
@@
 			(project "usb2ps2"
 				(path "/8c0b3d8b-46d3-4173-ab1e-a61765f77d61/6c767f01-0461-4c4b-955a-2f0ac89894b4"
-					(reference "R15")
+					(reference "R7")
 					(unit 1)
 				)
@@
 			)
 		)
-		(property "Footprint" "LIBS:Medved_D_0805"
+		(property "Footprint" "FRANK:Diode (SOD-323)"
 			(at 130.81 52.07 90)
 			(effects
