File: hardware/usb2ps2/uart.kicad_sch (KiCad schematic)
At the start: 1 part, among them CN2 UART

Commit message: Structural updates
Parts:
- CN2: footprint LIBS:Medved_UART_Pin3 -> FRANK:Pin Header (1x03)
Changed lines of the file:
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@@
 (kicad_sch
-	(version 20231120)
+	(version 20250114)
 	(generator "eeschema")
-	(generator_version "8.0")
+	(generator_version "9.0")
 	(paper "A3")
 	(title_block
 		(title "USB to PS/2 Adapter")
-		(date "2024-12-07")
-		(rev "1.2")
+		(date "2025-03-04")
+		(rev "1.02")
 		(company "Mikhail Matveev")
+		(comment 1 "https://github.com/xtremespb/frank")
 	)
 	(wire
@@
 		(shape input)
 		(at 50.8 36.83 0)
-		(fields_autoplaced yes)
 		(effects
 			(font
@@
 		(shape input)
 		(at 50.8 39.37 0)
-		(fields_autoplaced yes)
 		(effects
 			(font
@@
 			)
 		)
-		(property "Footprint" "LIBS:Medved_UART_Pin3"
+		(property "Footprint" "FRANK:Pin Header (1x03)"
 			(at 31.75 39.37 0)
 			(effects
@@
 		(dnp no)
 		(fields_autoplaced yes)
-		(property "Reference" "#PWR030"
+		(property "Reference" "#PWR03"
 			(at 50.8 48.26 0)
 			(effects
@@
 			(project "usb2ps2"
 				(path "/8c0b3d8b-46d3-4173-ab1e-a61765f77d61/806fcbb1-aec7-4a20-b8ef-b5e6440967de"
-					(reference "#PWR030")
+					(reference "#PWR03")
 					(unit 1)
 				)

Commit message: Minor updates
Parts:
- renumbered CN2 to CN1
Changed lines of the file:
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@@
 	(title_block
 		(title "USB to PS/2 Adapter")
-		(date "2025-03-04")
-		(rev "1.02")
+		(date "2025-03-09")
+		(rev "1.03")
 		(company "Mikhail Matveev")
 		(comment 1 "https://github.com/xtremespb/frank")
@@
 		(dnp no)
 		(fields_autoplaced yes)
-		(property "Reference" "CN2"
+		(property "Reference" "CN1"
 			(at 32.385 31.75 0)
 			(effects
@@
 			(project "usb2ps2"
 				(path "/8c0b3d8b-46d3-4173-ab1e-a61765f77d61/806fcbb1-aec7-4a20-b8ef-b5e6440967de"
-					(reference "CN2")
+					(reference "CN1")
 					(unit 1)
 				)
