File: hardware/usb2ps2/usb2ps2.kicad_pcb (KiCad board)
At the start: 2 copper layers, 54.4 x 33.1 mm, 55 parts, among them CN1 Conn_01x03_Pin, CN2 UART, CN3 PS/2 Pins, SW1 Flash Button, U1 NCP1117-3.3_SOT223, Y1 ABM8-272-T3

Commit message: Structural updates
Parts:
- removed C10, C3, C4, C5, C6, C7, C8, C9: 100n, LIBS:Medved_C_0805
- removed C11, C12: 1u, LIBS:Medved_C_0805
- removed C13, C14: 15p, LIBS:Medved_C_0805
- removed C15, C16: 10u, LIBS:Medved_C_0805
- removed C17, C18: 10u, LIBS:Medved_R_0805
- removed CN1: Conn_01x03_Pin, LIBS:Medved_PinHeader_1x03
- removed CN3: PS/2 Pins, LIBS:Medved_PinHeader_1x04
- removed FL1: W25Q128JVS, LIBS:Medved_SOIC-8_5.23x5.23mm_P1.27mm
- removed H1, H2, H3, H4: MountingHole, LIBS:MountingHole_2.1mm
- removed L1, L2: LED, LIBS:Medved_LED_0805
- removed R10, R11, R12, R9: 22R, LIBS:Medved_R_0805
- removed R13, R14, R15, R16: 100R, LIBS:Medved_R_0805
- removed SW1: Flash Button, LIBS:Button_SMD_3x3x2
- removed U1: NCP1117-3.3_SOT223, LIBS:Medved_SOT-223-3_TabPin2
- removed USB2: USB_A_Stacked, LIBS:Medved_USB_A_CUI_UJ2-ADH-TH_Horizontal_Stacked
- removed Y1: ABM8-272-T3, Crystal:Crystal_SMD_3225-4Pin_3.2x2.5mm
- C1, C2: value 100n -> 10u; footprint LIBS:Medved_C_0805 -> FRANK:Capacitor (0805); moved to B.Cu
- CN2: footprint LIBS:Medved_UART_Pin3 -> FRANK:Pin Header (1x03)
- D1, D2, D3, D4: footprint LIBS:Medved_D_0805 -> FRANK:Diode (SOD-323)
- PS1: footprint LIBS:Connector_Mini-DIN_Female_6Pin_2rows -> FRANK:MiniDIN (6 Pin, female)
- R1, R4: value 1k -> 22R; footprint LIBS:Medved_R_0805 -> FRANK:Resistor (0805); moved to B.Cu
- R2, R3: value 27 -> 22R; footprint LIBS:Medved_R_0805 -> FRANK:Resistor (0805); moved to B.Cu
- R5, R8: value 1K -> 100R; footprint LIBS:Medved_R_0805 -> FRANK:Resistor (0805); moved to B.Cu
- R6, R7: value 5.1K -> 100R; footprint LIBS:Medved_R_0805 -> FRANK:Resistor (0805); moved to B.Cu
- RP1: value RP2040 -> RP 2040 Zero; footprint LIBS:RP2040-QFN-56 -> FRANK:Raspberry Pi Zero (Outer pins); moved to B.Cu
- USB1: value USB Type C -> USB_A_Stacked; footprint LIBS:USB-TYPE-C-31-M-12_lib2 -> FRANK:USB Type A (stacked)
- moved C1 99.2 mm to (215.5, 118.0), turned to 0 degrees
- moved R8 94.7 mm to (204.2, 113.9)
- moved USB1 89.5 mm to (212.3, 118.4)
- moved C2 84.2 mm to (215.5, 115.9), turned to 0 degrees
- moved CN2 83.6 mm to (199.1, 108.5), turned to 90 degrees
- moved R1 82.1 mm to (199.1, 111.2), turned to 0 degrees
- moved R4 74.3 mm to (199.1, 117.5), turned to 0 degrees
- moved R7 73.4 mm to (204.2, 119.4), turned to -90 degrees
- moved R6 71.6 mm to (199.1, 121.7)
- moved RP1 69.9 mm to (195.0, 114.8), turned to -90 degrees
- moved R3 68.7 mm to (199.1, 115.4), turned to 0 degrees
- moved R5 68.1 mm to (199.1, 119.6), turned to 0 degrees
- moved R2 67.3 mm to (199.1, 113.3), turned to 0 degrees
- moved D3 61.6 mm to (201.3, 118.0)
- moved D1 60.7 mm to (201.3, 112.0)
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Connections:
- net /RP2040/GPIO6 renamed /RP Zero/GPIO7
- net /RP2040/GPIO7 renamed /RP Zero/GPIO8
- net /RP2040/GPIO8 renamed /RP Zero/GPIO10
- C1 pad 1: +3V3 -> VBUS
- C2 pad 1: Net-(RP1-VREG_VOUT) -> VBUS
- R1 pad 1: /RP2040/QSPI_SS -> /GPIO2
- R1 pad 2: /RP2040/~{USB_BOOT} -> Net-(USB1-D1+)
- R2 pad 1: /D+ -> /GPIO4
- R2 pad 2: Net-(RP1-USB_DP) -> Net-(USB1-D2+)
- R3 pad 1: /D- -> /GPIO3
- R3 pad 2: Net-(RP1-USB_DM) -> Net-(USB1-D1-)
- R4 pad 1: /RP2040/XOUT -> /GPIO5
- R4 pad 2: Net-(C14-Pad1) -> Net-(USB1-D2-)
- R5 pad 1: Net-(L1-A) -> /PS2 with Diodes/MS_DATA
- R5 pad 2: /RP2040/GPIO25 -> /GPIO14
- R6 pad 1: GND -> /PS2 with Diodes/MS_CLK
- R6 pad 2: Net-(USB1-CC1) -> /GPIO15
- R7 pad 1: GND -> /PS2 with Diodes/KB_CLK
- R7 pad 2: Net-(USB1-CC2) -> /GPIO12
- R8 pad 1: Net-(L2-A) -> /PS2 with Diodes/KB_DATA
- R8 pad 2: +3V3 -> /GPIO11
- RP1 pad 1: +3V3 -> /GPIO0
- RP1 pad 10: +3V3 -> /RP Zero/GPIO9
- RP1 pad 12: /RP2040/GPIO9 -> /GPIO11
- RP1 pad 13: /RP2040/GPIO10 -> /GPIO12
- RP1 pad 14: /GPIO11 -> /RP Zero/GPIO13
- RP1 pad 15: /GPIO12 -> /GPIO14
- RP1 pad 16: /RP2040/GPIO13 -> /GPIO15
- RP1 pad 17: /GPIO14 -> /RP Zero/GPIO26
- RP1 pad 18: /GPIO15 -> /RP Zero/GPIO27
- RP1 pad 19: GND -> /RP Zero/GPIO28
- RP1 pad 2: /GPIO0 -> /GPIO1
- RP1 pad 20: /RP2040/XIN -> /RP Zero/GPIO29
- RP1 pad 21: /RP2040/XOUT -> /RP Zero/3V3
- RP1 pad 22: +3V3 -> GND
- RP1 pad 23: Net-(RP1-VREG_VOUT) -> VBUS
- RP1 pad 3: /GPIO1 -> /GPIO2
- RP1 pad 4: /GPIO2 -> /GPIO3
- RP1 pad 5: /GPIO3 -> /GPIO4
- RP1 pad 6: /GPIO4 -> /GPIO5
- RP1 pad 7: /GPIO5 -> /RP Zero/GPIO6
- USB1 pad 1: GND -> VBUS
- USB1 pad 2: VBUS -> Net-(USB1-D1-)
- USB1 pad 3: unconnected-(USB1-SBU2-Pad3) -> Net-(USB1-D1+)
- USB1 pad 4: Net-(USB1-CC1) -> GND
- USB1 pad 5: /D- -> VBUS
- USB1 pad 6: /D+ -> Net-(USB1-D2-)
- USB1 pad 7: /D- -> Net-(USB1-D2+)
- USB1 pad 8: /D+ -> GND
- USB1 pad 9: unconnected-(USB1-SBU1-Pad9) -> GND
Routing:
- net +3V3: track 143.9 -> 0.00 mm, vias 4 -> 0
- net /GPIO11: track 69.5 -> 9.72 mm, vias 1 -> 0
- net VBUS: track 122.6 -> 64.3 mm, vias 4 -> 0
- net /GPIO12: track 67.1 -> 16.2 mm, vias 3 -> 1
- net /GPIO14: track 63.8 -> 19.7 mm, vias 3 -> 1
- net /GPIO15: track 55.9 -> 24.2 mm, vias 3 -> 1
- net Net-(RP1-VREG_VOUT): track 27.7 -> 0.00 mm
- net Net-(USB2-D1-): track 25.9 -> 0.00 mm, vias 1 -> 0
- net /RP2040/~{USB_BOOT}: track 18.0 -> 0.00 mm
- net /GPIO5: track 26.5 -> 8.61 mm, vias 2 -> 0
- net Net-(USB1-CC2): track 17.5 -> 0.00 mm
- net /RP2040/QSPI_SS: track 16.7 -> 0.00 mm
- net /RP2040/QSPI_SD1: track 16.7 -> 0.00 mm
- net Net-(USB2-D1+): track 16.1 -> 0.00 mm
- net Net-(USB2-D2-): track 15.9 -> 0.00 mm
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Other:
- board size 54.4 x 33.1 mm -> 40.2 x 20.4 mm
- board text added: "HW Rev 1.02"
- board text added: "rh1.tech"
- board text removed: "HW Rev 1.2"
- board text removed: "USB>PS/2"
- board text removed: "rh1.dev"

Commit message: Minor updates
Parts:
- removed CN2: UART, FRANK:Pin Header (1x03)
- added CN1: UART, FRANK:Pin Header (1x03), F.Cu at (137.5, 56.3)
- added H1: MountingHole, FRANK:Mounting Hole (2.7mm), F.Cu at (130.7, 32.1)
- added H2: MountingHole, FRANK:Mounting Hole (2.7mm), F.Cu at (130.7, 56.1)
- added H3: MountingHole, FRANK:Mounting Hole (2.7mm), F.Cu at (178.7, 32.1)
- added H4: MountingHole, FRANK:Mounting Hole (2.7mm), F.Cu at (178.7, 56.1)
- C1, C2, R1, R2, R3, R4, R5, R6, R7, R8: moved to F.Cu
- RP1: footprint FRANK:Raspberry Pi Zero (Outer pins) -> FRANK:Raspberry Pi Zero (on board); moved to F.Cu
- moved C2 114.7 mm to (137.5, 31.8), turned to 180 degrees
- moved C1 113.4 mm to (141.8, 31.8)
- moved USB1 107.9 mm to (137.5, 40.7), turned to 0 degrees
- moved R4 89.3 mm to (173.6, 32.0), turned to 90 degrees
- moved R3 87.9 mm to (171.5, 32.0), turned to 90 degrees
- moved R2 86.6 mm to (169.4, 32.0), turned to 90 degrees
- moved R1 85.4 mm to (167.3, 32.0), turned to 90 degrees
- moved RP1 84.1 mm to (155.1, 40.8), turned to 0 degrees
- moved D3 82.1 mm to (148.3, 55.3)
- moved D4 79.1 mm to (157.3, 55.3)
- moved PS1 75.4 mm to (173.1, 42.7), turned to 90 degrees
- moved D1 74.6 mm to (152.8, 55.3)
- moved R7 72.2 mm to (169.4, 56.2)
- moved D2 71.6 mm to (161.9, 55.3)
- moved R6 70.3 mm to (173.6, 56.2), turned to -90 degrees
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Routing:
- net Net-(USB1-D1-): track 13.3 -> 68.5 mm, vias 1 -> 3
- net VBUS: track 64.3 -> 114.9 mm, vias 0 -> 1
- net Net-(USB1-D2-): track 11.1 -> 61.6 mm, vias 1 -> 3
- net Net-(USB1-D2+): track 11.6 -> 56.1 mm, vias 0 -> 3
- net Net-(USB1-D1+): track 14.5 -> 55.9 mm, vias 1 -> 3
- net /GPIO0: track 26.4 -> 53.3 mm, vias 0 -> 1
- net /GPIO1: track 27.6 -> 49.6 mm, vias 0 -> 1
- net /PS2 with Diodes/MS_DATA: track 14.1 -> 28.3 mm, vias 3 -> 0
- net /GPIO15: track 24.2 -> 36.6 mm, vias 1 -> 0
- net /GPIO2: track 16.7 -> 5.24 mm
- net /GPIO14: track 19.7 -> 29.7 mm, vias 1 -> 0
- net /GPIO5: track 8.61 -> 18.3 mm
- net /PS2 with Diodes/KB_CLK: track 12.1 -> 20.6 mm, vias 1 -> 0
- net /GPIO3: track 18.2 -> 11.6 mm, vias 0 -> 2
- net /GPIO11: track 9.72 -> 14.0 mm
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Other:
- board size 40.2 x 20.4 mm -> 54 x 30 mm
- board text added: "+5V/1"
- board text added: "+5V/4"
- board text added: "+5V/5"
- board text added: "1.03"
- board text added: "D1+/3"
- board text added: "D1-/2"
- board text added: "D2+/2"
- board text added: "D2-/2"
- board text added: "GND"
- board text added: "GND/3"
- board text added: "GND/4"
- board text added: "GND/8"
- board text added: "GP0"
- board text added: "GP1"
- board text added: "KBC/5"
- board text added: "KBD/1"
- board text added: "MSC/6"
- board text added: "MSD/2"
- board text added: "PS/2"
- board text added: "USB"
- board text added: "USB > PS/2"
- board text removed: "HW Rev 1.02"
