File: hardware/usb2ps2/zero.kicad_sch (KiCad schematic)
At the start: 1 part

Commit message: Minor updates
Parts:
- RP1: footprint FRANK:Raspberry Pi Zero (Outer pins) -> FRANK:Raspberry Pi Zero (on board)
Changed lines of the file:
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@@
 	(title_block
 		(title "USB to PS/2 Adapter")
-		(date "2025-03-04")
-		(rev "1.02")
+		(date "2025-03-09")
+		(rev "1.03")
 		(company "Mikhail Matveev")
 		(comment 1 "https://github.com/xtremespb/frank")
@@
 			)
 		)
-		(property "Footprint" "FRANK:Raspberry Pi Zero (Outer pins)"
+		(property "Footprint" "FRANK:Raspberry Pi Zero (on board)"
 			(at 71.12 54.61 0)
 			(effects
