File: hardware/minifrank_rm2f/frank_rm2f.kicad_pcb (KiCad board)
At the start: 2 copper layers, 78.4 x 50 mm, 93 parts, among them J1 Pin Header 2x18, SW1 Reset, SW2 SW_Push, U1 NCP1117 3.3, U2 TDA1387T, U3 RP2350_60QFN, U4 ESP-PSRAM32, U5 W25Q128JVS, Y1 ASE-xxxMHz

Commit message: RM24 WIP
Routing:
- net /D+: track 89.5 -> 86.6 mm
Changed lines of the file:
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@@
+	)
+	(segment
+		(start 248.625028 48.374972)
+		(end 249.2 47.8)
+		(width 0.5)
+		(layer "B.Cu")
+		(net 29)
+	)
+	(segment
+		(start 249.2 47.8)
+		(end 254.3 47.8)
+		(width 0.5)
+		(layer "B.Cu")
+		(net 29)
+	)
+	(segment
+		(start 256.5465 81.289628)
+		(end 256.9 81.643128)
+		(width 0.5)
+		(layer "B.Cu")
+		(net 29)
+	)
+	(segment
+		(start 255.75 49.25)
+		(end 256.243 49.25)
+		(width 0.5)
+		(layer "B.Cu")
+		(net 29)
+	)
+	(segment
+		(start 248 48.374972)
+		(end 248.625028 48.374972)
+		(width 0.5)
+		(layer "B.Cu")
+		(net 29)
+	)
+	(segment
+		(start 256.243 49.25)
+		(end 256.5465 49.5535)
+		(width 0.5)
+		(layer "B.Cu")
+		(net 29)
 	)
 	(segment
@@
 	)
 	(segment
-		(start 257.1 49.1)
-		(end 259.2 51.2)
-		(width 0.5)
-		(layer "B.Cu")
-		(net 29)
-	)
-	(segment
-		(start 249.2 47.8)
-		(end 254.3 47.8)
-		(width 0.5)
-		(layer "B.Cu")
-		(net 29)
-	)
-	(segment
-		(start 259.2 51.2)
-		(end 256.5465 53.8535)
+		(start 230.6 92.4)
+		(end 230.5 92.5)
 		(width 0.5)
 		(layer "B.Cu")
@@
 	(segment
 		(start 254.3 47.8)
-		(end 255.526 49.026)
-		(width 0.5)
-		(layer "B.Cu")
-		(net 29)
-	)
-	(segment
-		(start 257.1 49.026)
-		(end 257.1 49.1)
+		(end 255.75 49.25)
 		(width 0.5)
 		(layer "B.Cu")
@@
 	)
 	(segment
-		(start 230.6 92.4)
-		(end 230.5 92.5)
-		(width 0.5)
-		(layer "B.Cu")
-		(net 29)
-	)
-	(segment
-		(start 248 48.374972)
-		(end 248.625028 48.374972)
-		(width 0.5)
-		(layer "B.Cu")
-		(net 29)
-	)
-	(segment
-		(start 248.625028 48.374972)
-		(end 249.2 47.8)
-		(width 0.5)
-		(layer "B.Cu")
-		(net 29)
-	)
-	(segment
-		(start 256.5465 81.289628)
-		(end 256.9 81.643128)
-		(width 0.5)
-		(layer "B.Cu")
-		(net 29)
-	)
-	(segment
-		(start 256.5465 53.8535)
+		(start 256.5465 49.5535)
 		(end 256.5465 81.289628)
 		(width 0.5)
@@
 	)
 	(segment
-		(start 255.526 49.026)
-		(end 257.1 49.026)
-		(width 0.5)
-		(layer "B.Cu")
-		(net 29)
+		(start 256.624 84.676)
+		(end 258.6485 84.676)
+		(width 0.5)
+		(layer "F.Cu")
+		(net 30)
+	)
+	(segment
+		(start 248.701 48.299)
+		(end 248.701 48.665336)
+		(width 0.5)
+		(layer "F.Cu")
+		(net 30)
+	)
+	(segment
+		(start 248.701 48.665336)
+		(end 248.356 49.010336)
+		(width 0.5)
+		(layer "F.Cu")
+		(net 30)
+	)
+	(segment
+		(start 248.199 49.645)
+		(end 248.305 49.751)
+		(width 0.3)
+		(layer "F.Cu")
+		(net 30)
+	)
+	(segment
+		(start 226.2 90.6)
+		(end 225.1 91.7)
+		(width 0.5)
+		(layer "F.Cu")
+		(net 30)
+	)
+	(segment
+		(start 259.199 51.48392)
+		(end 256.74108 49.026)
+		(width 0.5)
+		(layer "F.Cu")
+		(net 30)
+	)
+	(segment
+		(start 252.970206 49.026)
+		(end 251.744206 47.8)
+		(width 0.5)
+		(layer "F.Cu")
+		(net 30)
+	)
+	(segment
+		(start 246.87149 93.7)
+		(end 250.97249 89.599)
+		(width 0.5)
+		(layer "F.Cu")
+		(net 30)
+	)
+	(segment
+		(start 256.74108 49.026)
+		(end 252.970206 49.026)
+		(width 0.5)
+		(layer "F.Cu")
+		(net 30)
+	)
+	(segment
+		(start 248.305 49.751)
+		(end 248.305 50.67)
+		(width 0.3)
+		(layer "F.Cu")
+		(net 30)
+	)
+	(segment
+		(start 259.199 84.1255)
+		(end 259.199 51.48392)
+		(width 0.5)
+		(layer "F.Cu")
+		(net 30)
+	)
+	(segment
+		(start 249.2 47.8)
+		(end 248.701 48.299)
+		(width 0.5)
+		(layer "F.Cu")
+		(net 30)
+	)
+	(segment
+		(start 247.305 49.645)
+		(end 248.199 49.645)
+		(width 0.3)
+		(layer "F.Cu")
+		(net 30)
 	)
 	(segment
@@
 	)
 	(segment
-		(start 259.199 84.1255)
-		(end 259.199 51.48392)
-		(width 0.5)
-		(layer "F.Cu")
-		(net 30)
-	)
-	(segment
-		(start 255.69842 49.026)
-		(end 254.47242 47.8)
-		(width 0.5)
-		(layer "F.Cu")
-		(net 30)
-	)
-	(segment
-		(start 248.199 49.645)
-		(end 248.305 49.751)
-		(width 0.3)
-		(layer "F.Cu")
-		(net 30)
-	)
-	(segment
-		(start 256.624 84.676)
-		(end 258.6485 84.676)
-		(width 0.5)
+		(start 226.2 88.8)
+		(end 226.2 90.6)
+		(width 0.5)
+		(layer "F.Cu")
+		(net 30)
+	)
+	(segment
+		(start 247.305 50.67)
+		(end 247.305 49.645)
+		(width 0.3)
 		(layer "F.Cu")
 		(net 30)
@@
 	)
 	(segment
-		(start 226.2 90.6)
-		(end 225.1 91.7)
-		(width 0.5)
-		(layer "F.Cu")
-		(net 30)
-	)
-	(segment
-		(start 248.701 48.299)
-		(end 248.701 48.665336)
-		(width 0.5)
-		(layer "F.Cu")
-		(net 30)
-	)
-	(segment
-		(start 248.305 49.751)
-		(end 248.305 50.67)
-		(width 0.3)
+		(start 248.356 49.010336)
+		(end 248.356 49.644)
+		(width 0.5)
 		(layer "F.Cu")
 		(net 30)
@@
 	)
 	(segment
+		(start 251.744206 47.8)
+		(end 249.2 47.8)
+		(width 0.5)
+		(layer "F.Cu")
+		(net 30)
+	)
+	(segment
+		(start 225.1 91.7)
+		(end 225.1 93.22758)
+		(width 0.5)
+		(layer "F.Cu")
+		(net 30)
+	)
+	(segment
 		(start 251.701 89.599)
 		(end 256.624 84.676)
 		(width 0.5)
 		(layer "F.Cu")
-		(net 30)
-	)
-	(segment
-		(start 259.199 51.48392)
-		(end 256.74108 49.026)
-		(width 0.5)
-		(layer "F.Cu")
-		(net 30)
-	)
-	(segment
-		(start 225.1 91.7)
-		(end 225.1 93.22758)
-		(width 0.5)
-		(layer "F.Cu")
-		(net 30)
-	)
-	(segment
-		(start 248.701 48.665336)
-		(end 248.356 49.010336)
-		(width 0.5)
-		(layer "F.Cu")
-		(net 30)
-	)
-	(segment
-		(start 247.305 49.645)
-		(end 248.199 49.645)
-		(width 0.3)
-		(layer "F.Cu")
-		(net 30)
-	)
-	(segment
-		(start 254.47242 47.8)
-		(end 249.2 47.8)
-		(width 0.5)
-		(layer "F.Cu")
-		(net 30)
-	)
-	(segment
-		(start 249.2 47.8)
-		(end 248.701 48.299)
-		(width 0.5)
-		(layer "F.Cu")
-		(net 30)
-	)
-	(segment
-		(start 226.2 88.8)
-		(end 226.2 90.6)
-		(width 0.5)
-		(layer "F.Cu")
-		(net 30)
-	)
-	(segment
-		(start 247.305 50.67)
-		(end 247.305 49.645)
-		(width 0.3)
-		(layer "F.Cu")
-		(net 30)
-	)
-	(segment
-		(start 248.356 49.010336)
-		(end 248.356 49.644)
-		(width 0.5)
-		(layer "F.Cu")
-		(net 30)
-	)
-	(segment
-		(start 256.74108 49.026)
-		(end 255.69842 49.026)
-		(width 0.5)
-		(layer "F.Cu")
-		(net 30)
-	)
-	(segment
-		(start 246.87149 93.7)
-		(end 250.97249 89.599)
-		(width 0.5)
-		(layer "F.Cu")
