File: hardware/minifrank_rm24/ps2.kicad_sch (KiCad schematic)
At the start: 14 parts

Commit message: MiniFRANK RM24 added
Other:
- title: MiniFRANK RM2F -> MiniFRANK RM24
Changed lines of the file:
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@@
 	(paper "A4")
 	(title_block
-		(title "MiniFRANK RM2F")
-		(date "2025-03-13")
+		(title "MiniFRANK RM24")
+		(date "2025-03-14")
 		(rev "1.00")
 		(company "Mikhail Matveev")
